File: CAD/BT832A.sch (EAGLE design)
At the start: 41 parts, among them IC1 CP2102, U1 MCP73831T-3ACI/OT, U2 BT832, U3 LP5907MFX-3.3/NOPB, U4 LP5907MFX-3.3/NOPB, U5 ADS131M08IPBS, U6 BCM857BS, X1 ABM3B-8.000MHZ-B2-T, X2 FC-12M

Commit message: edits
Connections:
- net +5V: no longer C7.1, U4.EN, U4.IN
- net VIN: now also C7.1, U4.EN, U4.IN
Changed lines of the file:
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@@
 <grid distance="10" unitdist="mil" unit="mil" style="lines" multiple="1" display="no" altdistance="0.01" altunitdist="inch" altunit="inch"/>
 <layers>
-<layer number="1" name="Top" color="4" fill="1" visible="yes" active="no"/>
-<layer number="2" name="Route2" color="16" fill="1" visible="yes" active="no"/>
-<layer number="3" name="Route3" color="17" fill="1" visible="yes" active="no"/>
-<layer number="4" name="Route4" color="18" fill="1" visible="yes" active="no"/>
-<layer number="5" name="Route5" color="19" fill="1" visible="yes" active="no"/>
-<layer number="6" name="Route6" color="25" fill="1" visible="yes" active="no"/>
-<layer number="7" name="Route7" color="26" fill="1" visible="yes" active="no"/>
-<layer number="8" name="Route8" color="27" fill="1" visible="yes" active="no"/>
-<layer number="9" name="Route9" color="28" fill="1" visible="yes" active="no"/>
-<layer number="10" name="Route10" color="29" fill="1" visible="yes" active="no"/>
-<layer number="11" name="Route11" color="30" fill="1" visible="yes" active="no"/>
-<layer number="12" name="Route12" color="20" fill="1" visible="yes" active="no"/>
-<layer number="13" name="Route13" color="21" fill="1" visible="yes" active="no"/>
-<layer number="14" name="Route14" color="22" fill="1" visible="yes" active="no"/>
-<layer number="15" name="Route15" color="23" fill="1" visible="yes" active="no"/>
-<layer number="16" name="Bottom" color="1" fill="1" visible="yes" active="no"/>
-<layer number="17" name="Pads" color="2" fill="1" visible="yes" active="no"/>
-<layer number="18" name="Vias" color="2" fill="1" visible="yes" active="no"/>
-<layer number="19" name="Unrouted" color="6" fill="1" visible="yes" active="no"/>
-<layer number="20" name="Dimension" color="24" fill="1" visible="yes" active="no"/>
-<layer number="21" name="tPlace" color="7" fill="1" visible="yes" active="no"/>
-<layer number="22" name="bPlace" color="7" fill="1" visible="yes" active="no"/>
-<layer number="23" name="tOrigins" color="15" fill="1" visible="yes" active="no"/>
-<layer number="24" name="bOrigins" color="15" fill="1" visible="yes" active="no"/>
-<layer number="25" name="tNames" color="7" fill="1" visible="yes" active="no"/>
-<layer number="26" name="bNames" color="7" fill="1" visible="yes" active="no"/>
-<layer number="27" name="tValues" color="7" fill="1" visible="yes" active="no"/>
-<layer number="28" name="bValues" color="7" fill="1" visible="yes" active="no"/>
+<layer number="1" name="Top" color="4" fill="1" visible="no" active="no"/>
+<layer number="2" name="Route2" color="16" fill="1" visible="no" active="no"/>
+<layer number="3" name="Route3" color="17" fill="1" visible="no" active="no"/>
+<layer number="4" name="Route4" color="18" fill="1" visible="no" active="no"/>
+<layer number="5" name="Route5" color="19" fill="1" visible="no" active="no"/>
+<layer number="6" name="Route6" color="25" fill="1" visible="no" active="no"/>
+<layer number="7" name="Route7" color="26" fill="1" visible="no" active="no"/>
+<layer number="8" name="Route8" color="27" fill="1" visible="no" active="no"/>
+<layer number="9" name="Route9" color="28" fill="1" visible="no" active="no"/>
+<layer number="10" name="Route10" color="29" fill="1" visible="no" active="no"/>
+<layer number="11" name="Route11" color="30" fill="1" visible="no" active="no"/>
+<layer number="12" name="Route12" color="20" fill="1" visible="no" active="no"/>
+<layer number="13" name="Route13" color="21" fill="1" visible="no" active="no"/>
+<layer number="14" name="Route14" color="22" fill="1" visible="no" active="no"/>
+<layer number="15" name="Route15" color="23" fill="1" visible="no" active="no"/>
+<layer number="16" name="Bottom" color="1" fill="1" visible="no" active="no"/>
+<layer number="17" name="Pads" color="2" fill="1" visible="no" active="no"/>
+<layer number="18" name="Vias" color="2" fill="1" visible="no" active="no"/>
+<layer number="19" name="Unrouted" color="6" fill="1" visible="no" active="no"/>
+<layer number="20" name="Dimension" color="24" fill="1" visible="no" active="no"/>
+<layer number="21" name="tPlace" color="7" fill="1" visible="no" active="no"/>
+<layer number="22" name="bPlace" color="7" fill="1" visible="no" active="no"/>
+<layer number="23" name="tOrigins" color="15" fill="1" visible="no" active="no"/>
+<layer number="24" name="bOrigins" color="15" fill="1" visible="no" active="no"/>
+<layer number="25" name="tNames" color="7" fill="1" visible="no" active="no"/>
+<layer number="26" name="bNames" color="7" fill="1" visible="no" active="no"/>
+<layer number="27" name="tValues" color="7" fill="1" visible="no" active="no"/>
+<layer number="28" name="bValues" color="7" fill="1" visible="no" active="no"/>
 <layer number="29" name="tStop" color="7" fill="3" visible="no" active="no"/>
 <layer number="30" name="bStop" color="7" fill="6" visible="no" active="no"/>
@@
 <layer number="35" name="tGlue" color="7" fill="4" visible="no" active="no"/>
 <layer number="36" name="bGlue" color="7" fill="5" visible="no" active="no"/>
-<layer number="37" name="tTest" color="7" fill="1" visible="yes" active="no"/>
-<layer number="38" name="bTest" color="7" fill="1" visible="yes" active="no"/>
+<layer number="37" name="tTest" color="7" fill="1" visible="no" active="no"/>
+<layer number="38" name="bTest" color="7" fill="1" visible="no" active="no"/>
 <layer number="39" name="tKeepout" color="4" fill="11" visible="no" active="no"/>
 <layer number="40" name="bKeepout" color="1" fill="11" visible="no" active="no"/>
@@
 <layer number="44" name="Drills" color="7" fill="1" visible="no" active="no"/>
 <layer number="45" name="Holes" color="7" fill="1" visible="no" active="no"/>
-<layer number="46" name="Milling" color="3" fill="1" visible="yes" active="no"/>
-<layer number="47" name="Measures" color="7" fill="1" visible="yes" active="no"/>
-<layer number="48" name="Document" color="7" fill="1" visible="yes" active="no"/>
-<layer number="49" name="Reference" color="7" fill="1" visible="yes" active="no"/>
-<layer number="50" name="dxf" color="7" fill="1" visible="yes" active="no"/>
-<layer number="51" name="tDocu" color="7" fill="1" visible="yes" active="no"/>
-<layer number="52" name="bDocu" color="7" fill="1" visible="yes" active="no"/>
-<layer number="53" name="tGND_GNDA" color="7" fill="9" visible="yes" active="no"/>
-<layer number="54" name="bGND_GNDA" color="1" fill="9" visible="yes" active="no"/>
-<layer number="56" name="wert" color="7" fill="1" visible="yes" active="no"/>
-<layer number="57" name="tCAD" color="7" fill="1" visible="yes" active="no"/>
-<layer number="59" name="tCarbon" color="7" fill="1" visible="yes" active="no"/>
-<layer number="60" name="bCarbon" color="7" fill="1" visible="yes" active="no"/>
+<layer number="46" name="Milling" color="3" fill="1" visible="no" active="no"/>
+<layer number="47" name="Measures" color="7" fill="1" visible="no" active="no"/>
+<layer number="48" name="Document" color="7" fill="1" visible="no" active="no"/>
+<layer number="49" name="Reference" color="7" fill="1" visible="no" active="no"/>
+<layer number="50" name="dxf" color="7" fill="1" visible="no" active="no"/>
+<layer number="51" name="tDocu" color="7" fill="1" visible="no" active="no"/>
+<layer number="52" name="bDocu" color="7" fill="1" visible="no" active="no"/>
+<layer number="53" name="tGND_GNDA" color="7" fill="9" visible="no" active="no"/>
+<layer number="54" name="bGND_GNDA" color="1" fill="9" visible="no" active="no"/>
+<layer number="56" name="wert" color="7" fill="1" visible="no" active="no"/>
+<layer number="57" name="tCAD" color="7" fill="1" visible="no" active="no"/>
+<layer number="59" name="tCarbon" color="7" fill="1" visible="no" active="no"/>
+<layer number="60" name="bCarbon" color="7" fill="1" visible="no" active="no"/>
 <layer number="88" name="SimResults" color="9" fill="1" visible="yes" active="yes"/>
 <layer number="89" name="SimProbes" color="9" fill="1" visible="yes" active="yes"/>
@@
 </segment>
 <segment>
-<pinref part="U4" gate="G$1" pin="EN"/>
-<wire x1="-50.292" y1="143.256" x2="-47.752" y2="143.256" width="0.1524" layer="91"/>
-<label x="-46.99" y="144.526" size="1.778" layer="95"/>
-</segment>
-<segment>
-<pinref part="U4" gate="G$1" pin="IN"/>
-<wire x1="-50.292" y1="138.176" x2="-48.006" y2="138.176" width="0.1524" layer="91"/>
-<label x="-46.99" y="138.43" size="1.778" layer="95"/>
-</segment>
-<segment>
-<pinref part="C7" gate="G$1" pin="1"/>
-<wire x1="-34.29" y1="140.97" x2="-34.29" y2="139.7" width="0.1524" layer="91"/>
-<label x="-34.036" y="136.652" size="1.778" layer="95"/>
-</segment>
-<segment>
 <pinref part="D2" gate="G$1" pin="AA"/>
 <wire x1="54.356" y1="42.164" x2="54.356" y2="38.1" width="0.1524" layer="91"/>
@@
 <label x="54.102" y="121.92" size="1.778" layer="95"/>
 </segment>
-</net>
+<segment>
+<pinref part="U4" gate="G$1" pin="EN"/>
+<wire x1="-50.292" y1="143.256" x2="-47.752" y2="143.256" width="0.1524" layer="91"/>
+<label x="-46.99" y="144.526" size="1.778" layer="95"/>
+</segment>
+<segment>
+<pinref part="U4" gate="G$1" pin="IN"/>
+<wire x1="-50.292" y1="138.176" x2="-48.006" y2="138.176" width="0.1524" layer="91"/>
+<label x="-46.99" y="138.43" size="1.778" layer="95"/>
+</segment>
+<segment>
+<pinref part="C7" gate="G$1" pin="1"/>
+<wire x1="-34.29" y1="140.97" x2="-34.29" y2="139.7" width="0.1524" layer="91"/>
+<label x="-34.036" y="136.652" size="1.778" layer="95"/>
+</segment>
+</net>

Commit message: edits
Connections:
- net VDD: now also IC1.VDD
Other:
- moved on the sheet: C12, C13, U3
Changed lines of the file:
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@@
 <attribute name="VALUE" x="162.5377" y="91.3917" size="1.7806" layer="96"/>
 </instance>
-<instance part="U3" gate="G$1" x="81.28" y="114.3" smashed="yes">
-<attribute name="NAME" x="68.58" y="122.92" size="2.0828" layer="95" ratio="10" rot="SR0"/>
-<attribute name="VALUE" x="68.58" y="102.68" size="2.0828" layer="96" ratio="10" rot="SR0"/>
+<instance part="U3" gate="G$1" x="73.66" y="127.508" smashed="yes">
+<attribute name="NAME" x="60.96" y="136.128" size="2.0828" layer="95" ratio="10" rot="SR0"/>
+<attribute name="VALUE" x="57.404" y="114.11" size="2.0828" layer="96" ratio="10" rot="SR0"/>
 </instance>
 <instance part="X2" gate="G$1" x="142.24" y="147.32" smashed="yes" rot="R90">
@@
 </instance>
 <instance part="P+3" gate="1" x="154.94" y="66.04" smashed="yes" rot="R90">
-<attribute name="VALUE" x="160.02" y="63.5" size="1.778" layer="96" rot="R180"/>
+<attribute name="VALUE" x="160.02" y="64.77" size="1.778" layer="96" rot="R180"/>
 </instance>
 <instance part="R1" gate="G$1" x="203.2" y="76.2" smashed="yes" rot="R90">
@@
 <attribute name="VALUE" x="206.502" y="72.39" size="1.778" layer="96" rot="R90"/>
 </instance>
-<instance part="C12" gate="G$1" x="105.41" y="113.03" smashed="yes" rot="R180">
-<attribute name="NAME" x="104.394" y="112.395" size="1.778" layer="95" rot="R180"/>
-<attribute name="VALUE" x="104.394" y="117.221" size="1.778" layer="96" rot="R180"/>
-</instance>
-<instance part="C13" gate="G$1" x="55.88" y="113.792" smashed="yes" rot="R180">
-<attribute name="NAME" x="54.864" y="113.157" size="1.778" layer="95" rot="R180"/>
-<attribute name="VALUE" x="54.864" y="117.983" size="1.778" layer="96" rot="R180"/>
+<instance part="C12" gate="G$1" x="97.79" y="126.238" smashed="yes" rot="R180">
+<attribute name="NAME" x="96.774" y="125.603" size="1.778" layer="95" rot="R180"/>
+<attribute name="VALUE" x="96.774" y="130.429" size="1.778" layer="96" rot="R180"/>
+</instance>
+<instance part="C13" gate="G$1" x="48.26" y="127" smashed="yes" rot="R180">
+<attribute name="NAME" x="47.244" y="126.365" size="1.778" layer="95" rot="R180"/>
+<attribute name="VALUE" x="47.244" y="131.191" size="1.778" layer="96" rot="R180"/>
 </instance>
 <instance part="SUPPLY4" gate="GND" x="148.59" y="51.816" smashed="yes">
@@
 <segment>
 <pinref part="C13" gate="G$1" pin="1"/>
-<wire x1="55.88" y1="111.252" x2="55.88" y2="108.712" width="0.1524" layer="91"/>
-<label x="56.134" y="106.934" size="1.778" layer="95"/>
+<wire x1="48.26" y1="124.46" x2="48.26" y2="121.92" width="0.1524" layer="91"/>
+<label x="48.514" y="120.142" size="1.778" layer="95"/>
 </segment>
 <segment>
 <pinref part="C12" gate="G$1" pin="1"/>
-<wire x1="105.41" y1="110.49" x2="105.41" y2="107.95" width="0.1524" layer="91"/>
-<label x="105.664" y="106.426" size="1.778" layer="95"/>
+<wire x1="97.79" y1="123.698" x2="97.79" y2="121.158" width="0.1524" layer="91"/>
+<label x="98.044" y="119.634" size="1.778" layer="95"/>
 </segment>
 <segment>
@@
 <segment>
 <pinref part="U3" gate="G$1" pin="OUT"/>
-<wire x1="96.52" y1="119.38" x2="98.806" y2="119.38" width="0.1524" layer="91"/>
-<label x="97.79" y="119.38" size="1.778" layer="95"/>
+<wire x1="88.9" y1="132.588" x2="91.186" y2="132.588" width="0.1524" layer="91"/>
+<label x="90.17" y="132.588" size="1.778" layer="95"/>
 </segment>
 <segment>
 <pinref part="C12" gate="G$1" pin="2"/>
-<wire x1="105.41" y1="118.11" x2="105.41" y2="120.904" width="0.1524" layer="91"/>
-<label x="105.918" y="121.158" size="1.778" layer="95"/>
+<wire x1="97.79" y1="131.318" x2="97.79" y2="134.112" width="0.1524" layer="91"/>
+<label x="98.298" y="134.366" size="1.778" layer="95"/>
 </segment>
 <segment>
@@
 <label x="203.454" y="83.566" size="1.778" layer="95"/>
 </segment>
+<segment>
+<pinref part="IC1" gate="G$1" pin="VDD"/>
+<wire x1="162.56" y1="60.96" x2="160.274" y2="60.96" width="0.1524" layer="91"/>
+<label x="156.21" y="58.928" size="1.778" layer="95"/>
+</segment>
 </net>
 <net name="N$8" class="0">
 <segment>
 <pinref part="U3" gate="G$1" pin="GND"/>
-<wire x1="96.52" y1="109.22" x2="98.552" y2="109.22" width="0.1524" layer="91"/>
+<wire x1="88.9" y1="122.428" x2="90.932" y2="122.428" width="0.1524" layer="91"/>
 </segment>
 </net>
@@
 <segment>
 <pinref part="U3" gate="G$1" pin="IN"/>
-<wire x1="66.04" y1="119.38" x2="63.754" y2="119.38" width="0.1524" layer="91"/>
-<label x="60.452" y="119.634" size="1.778" layer="95"/>
+<wire x1="58.42" y1="132.588" x2="56.134" y2="132.588" width="0.1524" layer="91"/>
+<label x="52.832" y="132.842" size="1.778" layer="95"/>
 </segment>
 <segment>
 <pinref part="U3" gate="G$1" pin="EN"/>
-<wire x1="66.04" y1="114.3" x2="63.754" y2="114.3" width="0.1524" layer="91"/>
-<label x="60.452" y="115.062" size="1.778" layer="95"/>
+<wire x1="58.42" y1="127.508" x2="56.134" y2="127.508" width="0.1524" layer="91"/>
+<label x="52.832" y="128.27" size="1.778" layer="95"/>
 </segment>
 <segment>
@@
 <segment>
 <pinref part="C13" gate="G$1" pin="2"/>
-<wire x1="55.88" y1="118.872" x2="55.88" y2="121.158" width="0.1524" layer="91"/>
-<label x="54.102" y="121.92" size="1.778" layer="95"/>
-</segment>
-<segment>
+<wire x1="48.26" y1="132.08" x2="48.26" y2="134.366" width="0.1524" layer="91"/>
+<label x="46.482" y="135.128" size="1.778" layer="95"/>
+</segment>
+<segment>

Commit message: edits
Parts:
- removed R1: 4.7kΩ, adafruit:R-US_R0402
Connections:
- net B+: now also U1.VBAT
- net CPRST: no longer R1.1
- net GND: now also U1.VSS
- net VDD: no longer R1.2
Other:
- moved on the sheet: R4
Changed lines of the file:
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@@
 <part name="P+2" library="supply1" library_urn="urn:adsk.eagle:library:371" deviceset="+5V" device=""/>
 <part name="P+3" library="supply1" library_urn="urn:adsk.eagle:library:371" deviceset="+5V" device=""/>
-<part name="R1" library="adafruit" library_urn="urn:adsk.eagle:library:420" deviceset="R-US_" device="R0402" package3d_urn="urn:adsk.eagle:package:6240564/1" value="4.7kΩ"/>
 <part name="C12" library="adafruit" deviceset="C-US" device="C0402" value="1uF"/>
 <part name="C13" library="adafruit" deviceset="C-US" device="C0402" value="1uF"/>
@@
 <part name="P+5" library="supply1" library_urn="urn:adsk.eagle:library:371" deviceset="+5V" device=""/>
 <part name="S1" library="CL-SB-12B-01T" deviceset="CL-SB-12B-01T" device=""/>
+<part name="SUPPLY10" library="supply2" library_urn="urn:adsk.eagle:library:372" deviceset="GND" device=""/>
 </parts>
 <sheets>
@@
 <attribute name="VALUE" x="160.02" y="64.77" size="1.778" layer="96" rot="R180"/>
 </instance>
-<instance part="R1" gate="G$1" x="203.2" y="76.2" smashed="yes" rot="R90">
-<attribute name="NAME" x="201.7014" y="72.39" size="1.778" layer="95" rot="R90"/>
-<attribute name="VALUE" x="206.502" y="72.39" size="1.778" layer="96" rot="R90"/>
-</instance>
 <instance part="C12" gate="G$1" x="97.79" y="126.238" smashed="yes" rot="R180">
 <attribute name="NAME" x="96.774" y="125.603" size="1.778" layer="95" rot="R180"/>
@@
 <attribute name="VALUE" x="219.456" y="144.272" size="1.778" layer="96" rot="R90"/>
 </instance>
-<instance part="R4" gate="G$1" x="102.87" y="58.166" smashed="yes" rot="R90">
-<attribute name="NAME" x="101.3714" y="54.356" size="1.778" layer="95" rot="R90"/>
-<attribute name="VALUE" x="106.172" y="54.356" size="1.778" layer="96" rot="R90"/>
+<instance part="R4" gate="G$1" x="108.712" y="58.166" smashed="yes" rot="R90">
+<attribute name="NAME" x="107.2134" y="54.356" size="1.778" layer="95" rot="R90"/>
+<attribute name="VALUE" x="112.014" y="54.356" size="1.778" layer="96" rot="R90"/>
 </instance>
 <instance part="R5" gate="G$1" x="44.704" y="55.372" smashed="yes" rot="R270">
@@
 <attribute name="VALUE" x="42.799" y="42.291" size="1.778" layer="96"/>
 </instance>
-<instance part="SUPPLY9" gate="GND" x="102.87" y="48.006" smashed="yes">
-<attribute name="VALUE" x="100.965" y="44.831" size="1.778" layer="96"/>
+<instance part="SUPPLY9" gate="GND" x="108.712" y="47.498" smashed="yes">
+<attribute name="VALUE" x="106.807" y="44.323" size="1.778" layer="96"/>
 </instance>
 <instance part="P+5" gate="1" x="49.022" y="71.628" smashed="yes">
@@
 <attribute name="NAME" x="90.66451875" y="85.36085" size="1.27336875" layer="95" ratio="10"/>
 <attribute name="VALUE" x="90.66936875" y="72.633209375" size="1.27215" layer="96" ratio="10"/>
+</instance>
+<instance part="SUPPLY10" gate="GND" x="66.802" y="26.924" smashed="yes">
+<attribute name="VALUE" x="64.897" y="23.749" size="1.778" layer="96"/>
 </instance>
 </instances>
@@
 <segment>
 <pinref part="R4" gate="G$1" pin="1"/>
-<wire x1="102.87" y1="53.086" x2="102.87" y2="50.546" width="0.1524" layer="91"/>
+<wire x1="108.712" y1="53.086" x2="108.712" y2="50.038" width="0.1524" layer="91"/>
 <pinref part="SUPPLY9" gate="GND" pin="GND"/>
+</segment>
+<segment>
+<pinref part="U1" gate="A" pin="VSS"/>
+<wire x1="68.834" y1="34.544" x2="66.802" y2="34.544" width="0.1524" layer="91"/>
+<wire x1="66.802" y1="34.544" x2="66.802" y2="29.464" width="0.1524" layer="91"/>
+<pinref part="SUPPLY10" gate="GND" pin="GND"/>
 </segment>
 </net>
@@
 <segment>
 <pinref part="IC1" gate="G$1" pin="!RST"/>
-<wire x1="200.66" y1="68.58" x2="203.2" y2="68.58" width="0.1524" layer="91"/>
 <label x="205.74" y="68.58" size="1.778" layer="95"/>
-<pinref part="R1" gate="G$1" pin="1"/>
-<wire x1="203.2" y1="68.58" x2="205.74" y2="68.58" width="0.1524" layer="91"/>
-<wire x1="203.2" y1="68.58" x2="203.2" y2="71.12" width="0.1524" layer="91"/>
-<junction x="203.2" y="68.58"/>
+<wire x1="200.66" y1="68.58" x2="205.74" y2="68.58" width="0.1524" layer="91"/>
 </segment>
 <segment>
@@
 <wire x1="97.79" y1="131.318" x2="97.79" y2="134.112" width="0.1524" layer="91"/>
 <label x="98.298" y="134.366" size="1.778" layer="95"/>
-</segment>
-<segment>
-<pinref part="R1" gate="G$1" pin="2"/>
-<wire x1="203.2" y1="81.28" x2="203.2" y2="83.82" width="0.1524" layer="91"/>
-<label x="203.454" y="83.566" size="1.778" layer="95"/>
 </segment>
 <segment>
@@
 <junction x="98.552" y="65.786"/>
 <pinref part="R4" gate="G$1" pin="2"/>
-<wire x1="102.87" y1="63.246" x2="102.87" y2="65.786" width="0.1524" layer="91"/>
-<wire x1="98.552" y1="65.786" x2="102.87" y2="65.786" width="0.1524" layer="91"/>
+<wire x1="108.712" y1="63.246" x2="108.712" y2="65.786" width="0.1524" layer="91"/>
+<wire x1="98.552" y1="65.786" x2="108.712" y2="65.786" width="0.1524" layer="91"/>
 <label x="100.33" y="66.548" size="1.778" layer="95"/>
 </segment>
@@
 <label x="81.534" y="78.994" size="1.778" layer="95"/>
 </segment>
-</net>
+<segment>
+<pinref part="U1" gate="A" pin="VBAT"/>
+<wire x1="96.774" y1="44.704" x2="98.552" y2="44.704" width="0.1524" layer="91"/>
+<label x="99.314" y="43.942" size="1.778" layer="95"/>
+</segment>
+</net>
