File: CAD/BT832A.sch (EAGLE design)
At the start: 40 parts, among them IC1 CP2102, U1 MCP73831T-3ACI/OT, U2 BT832, U3 LP5907MFX-3.3/NOPB, U4 LP5907MFX-3.3/NOPB, U5 ADS131M08IPBS, U6 BCM857BS, X1 ABM3B-8.000MHZ-B2-T, X2 FC-12M

Commit message: edits
Connections:
- removed net N$3: LED2.C
- removed net N$4: U2.VDD
- removed net N$5: R3.2
- net GND: now also LED2.C
- net VDD: now also R3.2, U2.VDD
Changed lines of the file:
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@@
 <pinref part="SUPPLY10" gate="GND" pin="GND"/>
+</segment>
+<segment>
+<pinref part="LED2" gate="G$1" pin="C"/>
+<wire x1="216.154" y1="133.858" x2="216.154" y2="130.81" width="0.1524" layer="91"/>
+<label x="213.36" y="128.016" size="1.778" layer="95"/>
 </segment>
 </net>
@@
 <label x="156.21" y="58.928" size="1.778" layer="95"/>
 </segment>
+<segment>
+<pinref part="U2" gate="G$1" pin="VDD"/>
+<wire x1="198.12" y1="152.4" x2="202.438" y2="152.4" width="0.1524" layer="91"/>
+<label x="202.438" y="153.416" size="1.778" layer="95"/>
+</segment>
+<segment>
+<pinref part="R3" gate="G$1" pin="2"/>
+<wire x1="216.154" y1="153.162" x2="216.154" y2="156.21" width="0.1524" layer="91"/>
+<label x="216.662" y="157.226" size="1.778" layer="95"/>
+</segment>
 </net>
 <net name="N$8" class="0">
@@
 </segment>
 </net>
-<net name="N$3" class="0">
-<segment>
-<pinref part="LED2" gate="G$1" pin="C"/>
-<wire x1="216.154" y1="133.858" x2="216.154" y2="130.81" width="0.1524" layer="91"/>
-</segment>
-</net>
-<net name="N$4" class="0">
-<segment>
-<pinref part="U2" gate="G$1" pin="VDD"/>
-<wire x1="198.12" y1="152.4" x2="202.438" y2="152.4" width="0.1524" layer="91"/>
-</segment>
-</net>
-<net name="N$5" class="0">
-<segment>
-<pinref part="R3" gate="G$1" pin="2"/>
-<wire x1="216.154" y1="153.162" x2="216.154" y2="156.21" width="0.1524" layer="91"/>
-</segment>
-</net>

Commit message: edityedits
Connections:
- removed net N$8: U3.GND
- net GND: now also U3.GND
Changed lines of the file:
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@@
 <part name="S1" library="CL-SB-12B-01T" deviceset="CL-SB-12B-01T" device=""/>
 <part name="SUPPLY10" library="supply2" library_urn="urn:adsk.eagle:library:372" deviceset="GND" device=""/>
+<part name="SUPPLY11" library="supply2" library_urn="urn:adsk.eagle:library:372" deviceset="GND" device=""/>
 </parts>
 <sheets>
@@
 <attribute name="VALUE" x="64.897" y="23.749" size="1.778" layer="96"/>
 </instance>
+<instance part="SUPPLY11" gate="GND" x="90.932" y="116.586" smashed="yes">
+<attribute name="VALUE" x="89.027" y="113.411" size="1.778" layer="96"/>
+</instance>
 </instances>
 <busses>
@@
 <label x="213.36" y="128.016" size="1.778" layer="95"/>
 </segment>
+<segment>
+<pinref part="U3" gate="G$1" pin="GND"/>
+<wire x1="88.9" y1="122.428" x2="90.932" y2="122.428" width="0.1524" layer="91"/>
+<wire x1="90.932" y1="122.428" x2="90.932" y2="119.126" width="0.1524" layer="91"/>
+<pinref part="SUPPLY11" gate="GND" pin="GND"/>
+</segment>
 </net>
 <net name="XTAL2_2" class="0">
@@
 </segment>
 </net>
-<net name="N$8" class="0">
-<segment>
-<pinref part="U3" gate="G$1" pin="GND"/>
-<wire x1="88.9" y1="122.428" x2="90.932" y2="122.428" width="0.1524" layer="91"/>
-</segment>
-</net>

Commit message: changes
Parts:
- R7: device adafruit:R-US_R0603 -> adafruit:R-US_R0402
Changed lines of the file:
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@@
 <grid distance="10" unitdist="mil" unit="mil" style="lines" multiple="1" display="no" altdistance="0.01" altunitdist="inch" altunit="inch"/>
 <layers>
-<layer number="1" name="Top" color="4" fill="1" visible="no" active="no"/>
-<layer number="2" name="Route2" color="16" fill="1" visible="no" active="no"/>
-<layer number="3" name="Route3" color="17" fill="1" visible="no" active="no"/>
-<layer number="4" name="Route4" color="18" fill="1" visible="no" active="no"/>
-<layer number="5" name="Route5" color="19" fill="1" visible="no" active="no"/>
-<layer number="6" name="Route6" color="25" fill="1" visible="no" active="no"/>
-<layer number="7" name="Route7" color="26" fill="1" visible="no" active="no"/>
-<layer number="8" name="Route8" color="27" fill="1" visible="no" active="no"/>
-<layer number="9" name="Route9" color="28" fill="1" visible="no" active="no"/>
-<layer number="10" name="Route10" color="29" fill="1" visible="no" active="no"/>
-<layer number="11" name="Route11" color="30" fill="1" visible="no" active="no"/>
-<layer number="12" name="Route12" color="20" fill="1" visible="no" active="no"/>
-<layer number="13" name="Route13" color="21" fill="1" visible="no" active="no"/>
-<layer number="14" name="Route14" color="22" fill="1" visible="no" active="no"/>
-<layer number="15" name="Route15" color="23" fill="1" visible="no" active="no"/>
-<layer number="16" name="Bottom" color="1" fill="1" visible="no" active="no"/>
-<layer number="17" name="Pads" color="2" fill="1" visible="no" active="no"/>
-<layer number="18" name="Vias" color="2" fill="1" visible="no" active="no"/>
-<layer number="19" name="Unrouted" color="6" fill="1" visible="no" active="no"/>
-<layer number="20" name="Dimension" color="24" fill="1" visible="no" active="no"/>
-<layer number="21" name="tPlace" color="7" fill="1" visible="no" active="no"/>
-<layer number="22" name="bPlace" color="7" fill="1" visible="no" active="no"/>
-<layer number="23" name="tOrigins" color="15" fill="1" visible="no" active="no"/>
-<layer number="24" name="bOrigins" color="15" fill="1" visible="no" active="no"/>
-<layer number="25" name="tNames" color="7" fill="1" visible="no" active="no"/>
-<layer number="26" name="bNames" color="7" fill="1" visible="no" active="no"/>
-<layer number="27" name="tValues" color="7" fill="1" visible="no" active="no"/>
-<layer number="28" name="bValues" color="7" fill="1" visible="no" active="no"/>
+<layer number="1" name="Top" color="4" fill="1" visible="yes" active="no"/>
+<layer number="2" name="Route2" color="16" fill="1" visible="yes" active="no"/>
+<layer number="3" name="Route3" color="17" fill="1" visible="yes" active="no"/>
+<layer number="4" name="Route4" color="18" fill="1" visible="yes" active="no"/>
+<layer number="5" name="Route5" color="19" fill="1" visible="yes" active="no"/>
+<layer number="6" name="Route6" color="25" fill="1" visible="yes" active="no"/>
+<layer number="7" name="Route7" color="26" fill="1" visible="yes" active="no"/>
+<layer number="8" name="Route8" color="27" fill="1" visible="yes" active="no"/>
+<layer number="9" name="Route9" color="28" fill="1" visible="yes" active="no"/>
+<layer number="10" name="Route10" color="29" fill="1" visible="yes" active="no"/>
+<layer number="11" name="Route11" color="30" fill="1" visible="yes" active="no"/>
+<layer number="12" name="Route12" color="20" fill="1" visible="yes" active="no"/>
+<layer number="13" name="Route13" color="21" fill="1" visible="yes" active="no"/>
+<layer number="14" name="Route14" color="22" fill="1" visible="yes" active="no"/>
+<layer number="15" name="Route15" color="23" fill="1" visible="yes" active="no"/>
+<layer number="16" name="Bottom" color="1" fill="1" visible="yes" active="no"/>
+<layer number="17" name="Pads" color="2" fill="1" visible="yes" active="no"/>
+<layer number="18" name="Vias" color="2" fill="1" visible="yes" active="no"/>
+<layer number="19" name="Unrouted" color="6" fill="1" visible="yes" active="no"/>
+<layer number="20" name="Dimension" color="24" fill="1" visible="yes" active="no"/>
+<layer number="21" name="tPlace" color="7" fill="1" visible="yes" active="no"/>
+<layer number="22" name="bPlace" color="7" fill="1" visible="yes" active="no"/>
+<layer number="23" name="tOrigins" color="15" fill="1" visible="yes" active="no"/>
+<layer number="24" name="bOrigins" color="15" fill="1" visible="yes" active="no"/>
+<layer number="25" name="tNames" color="7" fill="1" visible="yes" active="no"/>
+<layer number="26" name="bNames" color="7" fill="1" visible="yes" active="no"/>
+<layer number="27" name="tValues" color="7" fill="1" visible="yes" active="no"/>
+<layer number="28" name="bValues" color="7" fill="1" visible="yes" active="no"/>
 <layer number="29" name="tStop" color="7" fill="3" visible="no" active="no"/>
 <layer number="30" name="bStop" color="7" fill="6" visible="no" active="no"/>
@@
 <layer number="35" name="tGlue" color="7" fill="4" visible="no" active="no"/>
 <layer number="36" name="bGlue" color="7" fill="5" visible="no" active="no"/>
-<layer number="37" name="tTest" color="7" fill="1" visible="no" active="no"/>
-<layer number="38" name="bTest" color="7" fill="1" visible="no" active="no"/>
+<layer number="37" name="tTest" color="7" fill="1" visible="yes" active="no"/>
+<layer number="38" name="bTest" color="7" fill="1" visible="yes" active="no"/>
 <layer number="39" name="tKeepout" color="4" fill="11" visible="no" active="no"/>
 <layer number="40" name="bKeepout" color="1" fill="11" visible="no" active="no"/>
@@
 <layer number="44" name="Drills" color="7" fill="1" visible="no" active="no"/>
 <layer number="45" name="Holes" color="7" fill="1" visible="no" active="no"/>
-<layer number="46" name="Milling" color="3" fill="1" visible="no" active="no"/>
-<layer number="47" name="Measures" color="7" fill="1" visible="no" active="no"/>
-<layer number="48" name="Document" color="7" fill="1" visible="no" active="no"/>
-<layer number="49" name="Reference" color="7" fill="1" visible="no" active="no"/>
-<layer number="50" name="dxf" color="7" fill="1" visible="no" active="no"/>
-<layer number="51" name="tDocu" color="7" fill="1" visible="no" active="no"/>
-<layer number="52" name="bDocu" color="7" fill="1" visible="no" active="no"/>
-<layer number="53" name="tGND_GNDA" color="7" fill="9" visible="no" active="no"/>
-<layer number="54" name="bGND_GNDA" color="1" fill="9" visible="no" active="no"/>
-<layer number="56" name="wert" color="7" fill="1" visible="no" active="no"/>
-<layer number="57" name="tCAD" color="7" fill="1" visible="no" active="no"/>
-<layer number="59" name="tCarbon" color="7" fill="1" visible="no" active="no"/>
-<layer number="60" name="bCarbon" color="7" fill="1" visible="no" active="no"/>
+<layer number="46" name="Milling" color="3" fill="1" visible="yes" active="no"/>
+<layer number="47" name="Measures" color="7" fill="1" visible="yes" active="no"/>
+<layer number="48" name="Document" color="7" fill="1" visible="yes" active="no"/>
+<layer number="49" name="Reference" color="7" fill="1" visible="yes" active="no"/>
+<layer number="50" name="dxf" color="7" fill="1" visible="yes" active="no"/>
+<layer number="51" name="tDocu" color="7" fill="1" visible="yes" active="no"/>
+<layer number="52" name="bDocu" color="7" fill="1" visible="yes" active="no"/>
+<layer number="53" name="tGND_GNDA" color="7" fill="9" visible="yes" active="no"/>
+<layer number="54" name="bGND_GNDA" color="1" fill="9" visible="yes" active="no"/>
+<layer number="56" name="wert" color="7" fill="1" visible="yes" active="no"/>
+<layer number="57" name="tCAD" color="7" fill="1" visible="yes" active="no"/>
+<layer number="59" name="tCarbon" color="7" fill="1" visible="yes" active="no"/>
+<layer number="60" name="bCarbon" color="7" fill="1" visible="yes" active="no"/>
 <layer number="88" name="SimResults" color="9" fill="1" visible="yes" active="yes"/>
 <layer number="89" name="SimProbes" color="9" fill="1" visible="yes" active="yes"/>
@@
 <part name="P+4" library="supply1" library_urn="urn:adsk.eagle:library:371" deviceset="+5V" device=""/>
 <part name="SUPPLY5" library="supply2" library_urn="urn:adsk.eagle:library:372" deviceset="GND" device=""/>
-<part name="R7" library="adafruit" library_urn="urn:adsk.eagle:library:420" deviceset="R-US_" device="R0603" package3d_urn="urn:adsk.eagle:package:6240565/1" value="10kΩ"/>
+<part name="R7" library="adafruit" library_urn="urn:adsk.eagle:library:420" deviceset="R-US_" device="R0402" package3d_urn="urn:adsk.eagle:package:6240564/1" value="10kΩ"/>
 <part name="SUPPLY6" library="supply2" library_urn="urn:adsk.eagle:library:372" deviceset="GND" device=""/>
 <part name="SUPPLY7" library="supply2" library_urn="urn:adsk.eagle:library:372" deviceset="GND" device=""/>

Commit message: almost there
Parts:
- removed SJ1: (no value), jumper:SJ
- removed U$2: PINHD-1X10, adafruit:PINHD-1X10
- added JP2, JP3: (no value), adafruit:PINHD-1X8CLEANBIG
- JP1: device adafruit:PINHD-1X1 -> adafruit:PINHD-1X8CLEANBIG
Connections:
- removed net REFIN_CAP: C9.2, SJ1.2
- new net N$10: U2.P30
- new net N$12: U2.P31
- new net N$13: U2.P03/AIN1
- new net N$15: U2.P02/AIN0
- new net N$16: U2.P16
- new net N$17: U2.P17
- new net N$19: U2.P18
- new net N$20: U2.P19
- new net N$21: U2.P20
- new net N$22: U2.P22
- new net N$23: U2.P23
- new net N$24: U2.P24
- new net N$25: U2.P26/SDA
- new net N$26: U2.P27/SCL
- new net N$3: U2.P15
- new net N$4: U2.P14
- new net N$5: U2.P13
- new net N$6: U2.P010/NFC2
- new net N$7: U2.P009/NFC1
- new net N$8: U2.P06
- net 3V3: no longer U$2.1
- net CS: now also U2.P05; no longer U$2.9
- net DIN: now also U2.P25; no longer U$2.5
- net DOUT: now also U2.P28; no longer U$2.6
- net DRDY: now also U2.P04; no longer U$2.8
- net GND: no longer U$2.2
- net REFIN: now also C9.2; no longer JP1.1, SJ1.1
- net SCLK: now also U2.P29; no longer U$2.7
- net SYNC/RESET: now also U2.P07; no longer U$2.10

Commit message: moarrrr
Connections:
- net N$13 renamed 6
- net N$15 renamed 5
- net N$17 renamed C3
- net N$19 renamed 12
- net N$2 renamed 14
- net N$20 renamed D2
- net N$21 renamed 13
- net N$22 renamed C2
- net N$23 renamed D1
- net N$24 renamed C1
- net N$25 renamed SDA
- net N$26 renamed SCL
- net N$4 renamed D4
- net N$5 renamed 11
- net N$6 renamed NFC2
- net N$7 renamed NFC1
- removed net N$10: U2.P30
- removed net N$12: U2.P31
- removed net N$16: U2.P16
- removed net N$3: U2.P15
- removed net N$8: U2.P06
- new net N$27: JP2.8
- new net N$28: JP2.7
- new net N$29: JP2.6
- new net N$30: JP2.5
- new net N$31: JP2.4
- new net N$32: JP2.3
- new net N$33: JP2.2
- new net N$34: JP2.1
- new net N$35: JP1.1
- new net N$36: JP1.2
- new net N$37: JP1.3
- new net N$38: JP1.4
- new net N$43: JP3.1
- new net N$44: JP3.2
- new net N$45: JP3.3
- new net N$46: JP3.4
- new net N$47: JP3.5
- new net N$48: JP3.6
- new net N$49: JP3.7
- new net N$50: JP3.8
- net D3: now also U2.P16
- net GND: now also JP1.5
- net RXD: now also JP1.7
- net TXD: now also JP1.8
- net VDD: now also JP1.6

Commit message: draft
Connections:
- removed net N$27: JP2.8
- removed net N$28: JP2.7
- removed net N$29: JP2.6
- removed net N$30: JP2.5
- removed net N$31: JP2.4
- removed net N$32: JP2.3
- removed net N$33: JP2.2
- removed net N$34: JP2.1
- removed net N$35: JP1.1
- removed net N$36: JP1.2
- removed net N$37: JP1.3
- removed net N$38: JP1.4
- removed net N$43: JP3.1
- removed net N$44: JP3.2
- removed net N$45: JP3.3
- removed net N$46: JP3.4
- removed net N$47: JP3.5
- removed net N$48: JP3.6
- removed net N$49: JP3.7
- removed net N$50: JP3.8
- net 11: now also JP1.4
- net 12: now also JP1.3
- net 13: now also JP1.2
- net 14: now also JP1.1
- net 5: now also JP2.4
- net 6: now also JP2.5
- net C1: now also JP2.1
- net C2: now also JP3.1
- net C3: now also JP3.2
- net D1: now also JP3.3
- net D2: now also JP3.4
- net D3: now also JP3.5
- net D4: now also JP3.6
- net GND: now also JP2.8
- net NFC1: now also JP2.6
- net NFC2: now also JP2.7
- net SCL: now also JP2.3
- net SDA: now also JP2.2
- net SWDCLK: now also JP3.8
- net SWDIO: now also JP3.7

Commit message: edits
Parts:
- removed R7: 10kΩ, adafruit:R-US_R0402
- added R1: 3.3kΩ, adafruit:R-US_R0402
- C1, C2: value (none) -> 12.5pF
- C3, C4: value (none) -> 10pF
- R3: value 3.3kΩ -> 10kΩ
- R4: value 10kΩ -> 47kΩ
- R5: value 47kΩ -> 2kΩ
- R6: value 2kΩ -> 10kΩ
Connections:
- new net BAT_D3: D3.AA, S1.3
- net 10K: now also R3.2; no longer R4.2
- net D3: no longer D3.AA, S1.3
- net GND: now also R3.1, R4.2, R6.1; no longer R4.1, R6.2, R7.1
- net N$1: now also R2.1; no longer R3.1
- net N$11: now also R1.2; no longer R2.2
- net N$14: now also R4.1; no longer R5.1
- net N$9: now also R5.1; no longer R6.1
- net NC: no longer S1.2
- net NVD: now also R1.1, R6.2; no longer R2.1, R7.2
- net VDD: now also R2.2; no longer R3.2
Other:
- moved on the sheet: R2, R3, R4, R5, R6

Commit message: fixes
Parts:
- added C14: 0.1uF, adafruit:C-USC0402
- added C15: 10uF, adafruit:C-USC0402
- added C16: 4.7uF, adafruit:C-USC0402
Connections:
- removed net 3V3: U5.DVDD
- removed net NC: U5.NC
- new net CPVDD: C14.2, IC1.VDD
- net B+: now also C16.2
- net GND: now also C14.1, C15.1, C16.1, U$1.MP1, U$1.MP2
- net VDD: now also C15.2, U5.DVDD; no longer IC1.VDD
