File: CAD/BT832A.brd (EAGLE design)
At the start: 24.9 x 48 mm, 40 parts, among them IC1 CP2102, U1 MCP73831T-3ACI/OT, U2 BT832, U3 LP5907MFX-3.3/NOPB, U4 LP5907MFX-3.3/NOPB, U5 ADS131M08IPBS, U6 BCM857BS, X1 ABM3B-8.000MHZ-B2-T, X2 FC-12M

Commit message: Update BT832A.brd
Routing:
- net CPRST: track 35.5 -> 36.5 mm
Changed lines of the file:
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@@
 <wire x1="29.15" y1="-18.9576" x2="30.0736" y2="-18.034" width="0.254" layer="1"/>
 <wire x1="27.2796" y1="-10.795" x2="27.2796" y2="-2.8956" width="0.254" layer="1"/>
-<wire x1="27.2796" y1="-2.8956" x2="26.924" y2="-2.54" width="0.254" layer="1"/>
-<wire x1="26.924" y1="-2.54" x2="21.4978" y2="-2.54" width="0.254" layer="1"/>
+<wire x1="27.2796" y1="-2.8956" x2="27.0256" y2="-2.6416" width="0.254" layer="1"/>
+<wire x1="27.0256" y1="-2.6416" x2="19.9738" y2="-2.6416" width="0.254" layer="1"/>
 <wire x1="18.3" y1="2.46813125" x2="18.3" y2="4.414" width="0.254" layer="1"/>
-<wire x1="21.4978" y1="-0.72966875" x2="18.3" y2="2.46813125" width="0.254" layer="1"/>
-<wire x1="21.4978" y1="-2.54" x2="21.4978" y2="-0.72966875" width="0.254" layer="1"/>
+<wire x1="19.9738" y1="0.79433125" x2="18.3" y2="2.46813125" width="0.254" layer="1"/>
+<wire x1="19.9738" y1="-2.6416" x2="19.9738" y2="0.79433125" width="0.254" layer="1"/>
 <wire x1="30.0736" y1="-13.589" x2="27.2796" y2="-10.795" width="0.254" layer="1"/>
 </signal>

Commit message: Update BT832A.brd
Parts:
- moved S1 1.11 mm to (10.4, -15.6)
Routing:
- net D3: track 7.85 -> 8.38 mm
Changed lines of the file:
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@@
 <attribute name="VALUE" x="23.2918" y="-8.8138" size="0.508" layer="27" rot="R270"/>
 </element>
-<element name="S1" library="CL-SB-12B-01T" package="CL-SB-12B" value="CL-SB-12B-01T" x="10.8204" y="-14.5288" smashed="yes" rot="R90">
-<attribute name="AVAILABILITY" value="In Stock" x="10.8204" y="-14.5288" size="1.778" layer="27" rot="R90" display="off"/>
-<attribute name="DESCRIPTION" value=" Slide Switch SPDT Surface Mount " x="10.8204" y="-14.5288" size="1.778" layer="27" rot="R90" display="off"/>
-<attribute name="MF" value="Nidec Copal" x="10.8204" y="-14.5288" size="1.778" layer="27" rot="R90" display="off"/>
-<attribute name="MP" value="CL-SB-12B-01T" x="10.8204" y="-14.5288" size="1.778" layer="27" rot="R90" display="off"/>
-<attribute name="PACKAGE" value="None" x="10.8204" y="-14.5288" size="1.778" layer="27" rot="R90" display="off"/>
-<attribute name="PRICE" value="None" x="10.8204" y="-14.5288" size="1.778" layer="27" rot="R90" display="off"/>
+<element name="S1" library="CL-SB-12B-01T" package="CL-SB-12B" value="CL-SB-12B-01T" x="10.4394" y="-15.5702" smashed="yes" rot="R90">
+<attribute name="AVAILABILITY" value="In Stock" x="10.4394" y="-15.5702" size="1.778" layer="27" rot="R90" display="off"/>
+<attribute name="DESCRIPTION" value=" Slide Switch SPDT Surface Mount " x="10.4394" y="-15.5702" size="1.778" layer="27" rot="R90" display="off"/>
+<attribute name="MF" value="Nidec Copal" x="10.4394" y="-15.5702" size="1.778" layer="27" rot="R90" display="off"/>
+<attribute name="MP" value="CL-SB-12B-01T" x="10.4394" y="-15.5702" size="1.778" layer="27" rot="R90" display="off"/>
+<attribute name="PACKAGE" value="None" x="10.4394" y="-15.5702" size="1.778" layer="27" rot="R90" display="off"/>
+<attribute name="PRICE" value="None" x="10.4394" y="-15.5702" size="1.778" layer="27" rot="R90" display="off"/>
 </element>
 </elements>
@@
 <signal name="NC">
 <contactref element="S1" pad="2"/>
-<wire x1="8.5704" y1="-14.5288" x2="-25.896" y2="1.163" width="0" layer="19" extent="1-16"/>
+<wire x1="8.1894" y1="-15.5702" x2="-25.896" y2="1.163" width="0" layer="19" extent="1-16"/>
 <contactref element="U5" pad="27"/>
 </signal>
@@
 <contactref element="S1" pad="1"/>
 <contactref element="J1" pad="2"/>
-<wire x1="13.986" y1="-21.7" x2="13.986" y2="-17.9444" width="0.508" layer="1"/>
-<wire x1="13.986" y1="-17.9444" x2="13.0704" y2="-17.0288" width="0.508" layer="1"/>
+<wire x1="13.986" y1="-21.7" x2="13.986" y2="-19.3668" width="0.508" layer="1"/>
+<wire x1="13.986" y1="-19.3668" x2="12.6894" y2="-18.0702" width="0.508" layer="1"/>
 <contactref element="U1" pad="3"/>
-<wire x1="13.0704" y1="-17.0288" x2="13.0704" y2="-14.9204" width="0.508" layer="1"/>
-<wire x1="14.859" y1="-13.1318" x2="15.367" y2="-13.1318" width="0.508" layer="1"/>
-<wire x1="13.0704" y1="-14.9204" x2="14.859" y2="-13.1318" width="0.508" layer="1"/>
+<wire x1="12.6894" y1="-18.0702" x2="12.6894" y2="-17.3842" width="0.508" layer="1"/>
+<wire x1="15.367" y1="-13.1318" x2="15.367" y2="-13.589" width="0.508" layer="1"/>
+<wire x1="15.367" y1="-13.589" x2="14.351" y2="-14.605" width="0.508" layer="1"/>
+<wire x1="14.351" y1="-14.605" x2="14.351" y2="-15.7226" width="0.508" layer="1"/>
+<wire x1="14.351" y1="-15.7226" x2="12.6894" y2="-17.3842" width="0.508" layer="1"/>
 </signal>
 <signal name="VIN">
@@
 <contactref element="D3" pad="3"/>
 <contactref element="S1" pad="3"/>
-<wire x1="13.0704" y1="-12.0288" x2="13.0704" y2="-8.0292" width="0.508" layer="1"/>
-<wire x1="13.0704" y1="-8.0292" x2="14.2494" y2="-6.8502" width="0.508" layer="1"/>
-<wire x1="14.2494" y1="-6.8502" x2="16.4338" y2="-6.8502" width="0.508" layer="1"/>
+<wire x1="13.553" y1="-8.6896" x2="13.553" y2="-12.2066" width="0.508" layer="1"/>
+<wire x1="12.6894" y1="-13.0702" x2="13.553" y2="-12.2066" width="0.508" layer="1"/>
+<wire x1="13.553" y1="-8.6896" x2="15.3924" y2="-6.8502" width="0.508" layer="1"/>
+<wire x1="15.3924" y1="-6.8502" x2="16.4338" y2="-6.8502" width="0.508" layer="1"/>
 </signal>
 </signals>

Commit message: Update BT832A.brd
Parts:
- moved C12 1.37 mm to (22.6, -2.39)
- moved C13 0.63 mm to (22.2, -4.95)
- moved R6 0.23 mm to (20.8, -11.3)
Routing:
- net CPRST: track 36.5 -> 35.5 mm
- net VIN: track 14.0 -> 13.5 mm
Changed lines of the file:
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@@
 <attribute name="VALUE" x="25.8826" y="-19.2532" size="0.508" layer="27" rot="R270"/>
 </element>
-<element name="C12" library="adafruit" package="C0402" value="1uF" x="22.3266" y="-1.0414" smashed="yes" rot="R90">
-<attribute name="NAME" x="23.0124" y="0.9906" size="0.508" layer="25" rot="R180"/>
-<attribute name="VALUE" x="21.59" y="-0.9652" size="0.508" layer="27" rot="R90"/>
-</element>
-<element name="C13" library="adafruit" package="C0402" value="1uF" x="22.0726" y="-4.3434" smashed="yes">
-<attribute name="NAME" x="21.1836" y="-3.5814" size="0.508" layer="25"/>
-<attribute name="VALUE" x="24.1554" y="-5.2324" size="0.508" layer="27" rot="R90"/>
+<element name="C12" library="adafruit" package="C0402" value="1uF" x="22.5552" y="-2.3876" smashed="yes" rot="R90">
+<attribute name="NAME" x="23.241" y="-0.3556" size="0.508" layer="25" rot="R180"/>
+<attribute name="VALUE" x="21.8186" y="-2.3114" size="0.508" layer="27" rot="R90"/>
+</element>
+<element name="C13" library="adafruit" package="C0402" value="1uF" x="22.225" y="-4.953" smashed="yes">
+<attribute name="NAME" x="21.336" y="-4.191" size="0.508" layer="25"/>
+<attribute name="VALUE" x="24.3078" y="-5.842" size="0.508" layer="27" rot="R90"/>
 </element>
 <element name="U1" library="MCP73831T-3ACI_OT" package="SOT95P270X145-5N" value="MCP73831T-3ACI/OT" x="16.7386" y="-12.192" smashed="yes">
@@
 <attribute name="VALUE" x="23.7998" y="-18.3642" size="0.508" layer="27" rot="R90"/>
 </element>
-<element name="R6" library="adafruit" library_urn="urn:adsk.eagle:library:420" package="R0402" package3d_urn="urn:adsk.eagle:package:6240564/1" value="2kΩ" x="20.7772" y="-11.4808" smashed="yes">
-<attribute name="NAME" x="22.7838" y="-11.8618" size="0.508" layer="25" rot="R90"/>
-<attribute name="VALUE" x="23.4188" y="-12.1158" size="0.508" layer="27" rot="R90"/>
+<element name="R6" library="adafruit" library_urn="urn:adsk.eagle:library:420" package="R0402" package3d_urn="urn:adsk.eagle:package:6240564/1" value="2kΩ" x="20.7518" y="-11.2522" smashed="yes">
+<attribute name="NAME" x="22.7584" y="-11.6332" size="0.508" layer="25" rot="R90"/>
+<attribute name="VALUE" x="23.3934" y="-11.8872" size="0.508" layer="27" rot="R90"/>
 </element>
 <element name="R7" library="adafruit" library_urn="urn:adsk.eagle:library:420" package="R0603" package3d_urn="urn:adsk.eagle:package:6240565/1" value="10kΩ" x="20.7772" y="-9.5758" smashed="yes" rot="R180">
@@
 <contactref element="C12" pad="2"/>
 <contactref element="IC1" pad="6"/>
-<wire x1="24.2722" y1="-1.0818" x2="23.5818" y2="-0.3914" width="0.254" layer="1"/>
-<wire x1="23.5818" y1="-0.3914" x2="22.3266" y2="-0.3914" width="0.254" layer="1"/>
+<wire x1="24.2722" y1="-1.0818" x2="23.6164" y2="-1.7376" width="0.254" layer="1"/>
+<wire x1="23.6164" y1="-1.7376" x2="22.5552" y2="-1.7376" width="0.254" layer="1"/>
 <contactref element="U2" pad="9"/>
 <contactref element="R3" pad="2"/>
 <wire x1="24.2722" y1="-1.0818" x2="26.05" y2="3.514" width="0" layer="19" extent="1-1"/>
-<wire x1="24.75" y1="0.9652" x2="22.3266" y2="-0.3914" width="0" layer="19" extent="1-1"/>
+<wire x1="24.75" y1="0.9652" x2="22.5552" y2="-1.7376" width="0" layer="19" extent="1-1"/>
 <wire x1="24.8526" y1="-16.6464" x2="24.2722" y2="-1.0818" width="0" layer="19" extent="1-1"/>
 </signal>
@@
 <contactref element="R5" pad="2"/>
 <contactref element="R4" pad="1"/>
-<wire x1="21.6272" y1="-9.5758" x2="21.6272" y2="-11.2808" width="0.254" layer="1"/>
-<wire x1="21.6272" y1="-11.2808" x2="21.4272" y2="-11.4808" width="0.254" layer="1"/>
+<wire x1="21.6272" y1="-9.5758" x2="21.6272" y2="-11.0268" width="0.254" layer="1"/>
+<wire x1="21.6272" y1="-11.0268" x2="21.4018" y2="-11.2522" width="0.254" layer="1"/>
 <contactref element="U1" pad="2"/>
 <contactref element="LED2" pad="C"/>
@@
 <wire x1="-39.1922" y1="8.382" x2="-26.896" y2="1.163" width="0" layer="19" extent="16-16"/>
 <wire x1="15.367" y1="-12.192" x2="-8.636" y2="-15.352" width="0" layer="19" extent="1-16"/>
-<wire x1="21.4272" y1="-11.4808" x2="15.367" y2="-12.192" width="0" layer="19" extent="1-1"/>
-<wire x1="25.0501" y1="-13.5439" x2="21.4272" y2="-11.4808" width="0" layer="19" extent="1-1"/>
+<wire x1="21.4018" y1="-11.2522" x2="15.367" y2="-12.192" width="0" layer="19" extent="1-1"/>
+<wire x1="25.0501" y1="-13.5439" x2="21.4018" y2="-11.2522" width="0" layer="19" extent="1-1"/>
 <wire x1="24.8526" y1="-15.1464" x2="25.0501" y2="-13.5439" width="0" layer="19" extent="1-1"/>
 <wire x1="27.1526" y1="-15.6464" x2="24.8526" y2="-15.1464" width="0" layer="19" extent="1-1"/>
@@
 <wire x1="25.2118" y1="-20.7772" x2="25.1864" y2="-19.558" width="0" layer="19" extent="1-1"/>
 <wire x1="25.938" y1="-24.9164" x2="25.2118" y2="-20.7772" width="0" layer="19" extent="1-1"/>
-<wire x1="21.4226" y1="-4.3434" x2="21.6272" y2="-9.5758" width="0" layer="19" extent="1-1"/>
-<wire x1="22.3266" y1="-1.6914" x2="21.4226" y2="-4.3434" width="0" layer="19" extent="1-1"/>
-<wire x1="27.8892" y1="2.528" x2="21.4226" y2="-4.3434" width="0" layer="19" extent="1-1"/>
+<wire x1="21.575" y1="-4.953" x2="21.6272" y2="-9.5758" width="0" layer="19" extent="1-1"/>
+<wire x1="22.5552" y1="-3.0376" x2="21.575" y2="-4.953" width="0" layer="19" extent="1-1"/>
+<wire x1="27.8892" y1="2.528" x2="21.575" y2="-4.953" width="0" layer="19" extent="1-1"/>
 <wire x1="16.8656" y1="-2.5042" x2="27.8892" y2="2.528" width="0" layer="19" extent="1-1"/>
 <wire x1="12.827" y1="-2.5804" x2="16.8656" y2="-2.5042" width="0" layer="19" extent="1-1"/>
 <wire x1="15.986" y1="-21.7" x2="21.0312" y2="-17.9728" width="0" layer="19" extent="1-1"/>
-<wire x1="26.05" y1="4.614" x2="22.3266" y2="-1.6914" width="0" layer="19" extent="1-1"/>
+<wire x1="26.05" y1="4.614" x2="22.5552" y2="-3.0376" width="0" layer="19" extent="1-1"/>
 <wire x1="21.3" y1="10.414" x2="26.05" y2="4.614" width="0" layer="19" extent="1-1"/>
 <wire x1="19.8" y1="10.414" x2="21.3" y2="10.414" width="0" layer="19" extent="1-1"/>
@@
 <wire x1="29.15" y1="-18.9576" x2="30.0736" y2="-18.034" width="0.254" layer="1"/>
 <wire x1="27.2796" y1="-10.795" x2="27.2796" y2="-2.8956" width="0.254" layer="1"/>
-<wire x1="27.2796" y1="-2.8956" x2="27.0256" y2="-2.6416" width="0.254" layer="1"/>
-<wire x1="27.0256" y1="-2.6416" x2="19.9738" y2="-2.6416" width="0.254" layer="1"/>
-<wire x1="18.3" y1="2.46813125" x2="18.3" y2="4.414" width="0.254" layer="1"/>
-<wire x1="19.9738" y1="0.79433125" x2="18.3" y2="2.46813125" width="0.254" layer="1"/>
-<wire x1="19.9738" y1="-2.6416" x2="19.9738" y2="0.79433125" width="0.254" layer="1"/>
+<wire x1="27.2796" y1="-2.8956" x2="26.7716" y2="-2.3876" width="0.254" layer="1"/>
+<wire x1="26.7716" y1="-2.3876" x2="21.4978" y2="-2.3876" width="0.254" layer="1"/>
+<wire x1="18.3" y1="2.31573125" x2="18.3" y2="4.414" width="0.254" layer="1"/>
+<wire x1="21.4978" y1="-0.88206875" x2="18.3" y2="2.31573125" width="0.254" layer="1"/>
+<wire x1="21.4978" y1="-2.3876" x2="21.4978" y2="-0.88206875" width="0.254" layer="1"/>
 <wire x1="30.0736" y1="-13.589" x2="27.2796" y2="-10.795" width="0.254" layer="1"/>
 </signal>
@@
 <contactref element="U1" pad="5"/>
 <contactref element="R6" pad="1"/>
-<wire x1="18.1102" y1="-11.2522" x2="19.8986" y2="-11.2522" width="0.254" layer="1"/>
-<wire x1="19.8986" y1="-11.2522" x2="20.1272" y2="-11.4808" width="0.254" layer="1"/>
+<wire x1="18.1102" y1="-11.2522" x2="20.1018" y2="-11.2522" width="0.254" layer="1"/>
 </signal>
 <signal name="N$11">
@@
 <wire x1="21.9764" y1="-7.8486" x2="21.9764" y2="-6.4716" width="0.254" layer="1"/>
 <wire x1="21.9764" y1="-6.4716" x2="22.86" y2="-5.588" width="0.254" layer="1"/>
-<wire x1="22.86" y1="-5.588" x2="22.86" y2="-4.4808" width="0.254" layer="1"/>
-<wire x1="22.86" y1="-4.4808" x2="22.7226" y2="-4.3434" width="0.254" layer="1"/>
-<wire x1="22.7226" y1="-4.3434" x2="23.5206" y2="-4.3434" width="0.254" layer="1"/>
-<wire x1="23.5206" y1="-4.3434" x2="24.2722" y2="-3.5918" width="0.254" layer="1"/>
+<wire x1="22.86" y1="-5.588" x2="22.86" y2="-4.968" width="0.254" layer="1"/>
+<wire x1="22.86" y1="-4.968" x2="22.875" y2="-4.953" width="0.254" layer="1"/>
+<wire x1="22.875" y1="-4.953" x2="22.911" y2="-4.953" width="0.254" layer="1"/>
+<wire x1="22.911" y1="-4.953" x2="24.2722" y2="-3.5918" width="0.254" layer="1"/>
 <wire x1="15.4838" y1="-9.0502" x2="16.552" y2="-7.982" width="0.254" layer="1"/>
 <wire x1="16.552" y1="-7.982" x2="17.50673125" y2="-7.982" width="0.254" layer="1"/>

Commit message: edityedits
Parts:
- moved U$2 4.56 mm to (-34.6, -0.91)
- moved SV1 1.84 mm to (-13.6, -0.89)
- moved U4 1.52 mm to (-21.1, -13.7), turned to 180 degrees
Connections:
- removed net N$8: U3.2
- net GND: now also U3.2

Commit message: Update BT832A.brd
Parts:
- moved U3 7.22 mm to (26.5, -9.45), turned to 0 degrees
- moved C12 6.06 mm to (26.4, -7.04), turned to 0 degrees
- moved C1 5.69 mm to (11.7, 0.43)
- moved C2 3.70 mm to (15.7, 0.43)
- moved X2 2.83 mm to (13.7, 0.74), turned to 0 degrees
- moved C13 2.56 mm to (23.4, -7.21), turned to 270 degrees
Routing:
- net VIN: track 13.5 -> 11.7 mm

Commit message: changes
Parts:
- R7: device adafruit:R0603 -> adafruit:R0402
- moved LED2 9.95 mm to (23.6, -7.19), turned to 180 degrees
- moved C2 8.43 mm to (24.1, 0.38)
- moved C1 8.43 mm to (20.1, 0.38)
- moved X2 8.43 mm to (22.1, 0.69)
- moved R3 7.56 mm to (25.8, -6.58), turned to 0 degrees
- moved J1 4.64 mm to (10.5, -24.2), turned to 90 degrees
- moved C13 4.11 mm to (22.8, -11.3), turned to 90 degrees
- moved R7 4.02 mm to (21.3, -13.6), turned to 90 degrees
- moved R5 3.71 mm to (22.4, -21.0)
- moved R4 3.70 mm to (20.7, -21.0)
- moved U6 3.57 mm to (21.4, -17.8)
- moved D1 2.97 mm to (19.7, -10.6)
- moved R2 2.93 mm to (17.3, -17.7)
- moved D2 2.85 mm to (18.0, -20.2)
- moved R6 2.51 mm to (19.9, -13.6), turned to 270 degrees
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Routing:
- net NVD: track 19.0 -> 21.9 mm
- net D3: track 8.38 -> 6.45 mm
- net CPRST: track 35.8 -> 37.4 mm
- net +5V: track 26.7 -> 25.5 mm
- net N$11: track 2.84 -> 1.99 mm
- net N$14: track 11.5 -> 10.7 mm

Commit message: Update BT832A.brd
Routing:
- net XTAL1_1: track 0.00 -> 19.4 mm
- net XTAL2_1: track 0.00 -> 14.4 mm
Changed lines of the file:
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@@
 <contactref element="C2" pad="2"/>
 <contactref element="U2" pad="3"/>
-<wire x1="24.1046" y1="1.031" x2="12.05" y2="9.014" width="0" layer="19" extent="1-1"/>
-<wire x1="22.948" y1="0.6858" x2="24.1046" y2="1.031" width="0" layer="19" extent="1-1"/>
+<wire x1="12.05" y1="9.014" x2="14.3794" y2="9.014" width="0.254" layer="1"/>
+<wire x1="15.9512" y1="7.4422" x2="15.9512" y2="3.6576" width="0.254" layer="1"/>
+<wire x1="15.9512" y1="3.6576" x2="17.1958" y2="2.413" width="0.254" layer="1"/>
+<wire x1="24.1046" y1="1.9812" x2="24.1046" y2="1.031" width="0.254" layer="1"/>
+<wire x1="14.3794" y1="9.014" x2="15.9512" y2="7.4422" width="0.254" layer="1"/>
+<wire x1="17.1958" y1="2.413" x2="23.6728" y2="2.413" width="0.254" layer="1"/>
+<wire x1="23.6728" y1="2.413" x2="24.1046" y2="1.9812" width="0.254" layer="1"/>
+<wire x1="22.948" y1="0.6858" x2="23.2932" y2="1.031" width="0.254" layer="1"/>
+<wire x1="23.2932" y1="1.031" x2="24.1046" y2="1.031" width="0.254" layer="1"/>
 </signal>
 <signal name="XTAL2_1">
@@
 <contactref element="C1" pad="2"/>
 <contactref element="U2" pad="4"/>
-<wire x1="21.248" y1="0.6858" x2="12.05" y2="7.914" width="0" layer="19" extent="1-1"/>
-<wire x1="20.0914" y1="1.031" x2="21.248" y2="0.6858" width="0" layer="19" extent="1-1"/>
+<wire x1="20.0914" y1="1.031" x2="19.1666" y2="1.9558" width="0.254" layer="1"/>
+<wire x1="19.1666" y1="1.9558" x2="17.018" y2="1.9558" width="0.254" layer="1"/>
+<wire x1="17.018" y1="1.9558" x2="15.4686" y2="3.5052" width="0.254" layer="1"/>
+<wire x1="14.8698" y1="7.914" x2="12.05" y2="7.914" width="0.254" layer="1"/>
+<wire x1="15.4686" y1="3.5052" x2="15.4686" y2="7.3152" width="0.254" layer="1"/>
+<wire x1="15.4686" y1="7.3152" x2="14.8698" y2="7.914" width="0.254" layer="1"/>
+<wire x1="21.248" y1="0.6858" x2="20.9028" y2="1.031" width="0.254" layer="1"/>
+<wire x1="20.9028" y1="1.031" x2="20.0914" y2="1.031" width="0.254" layer="1"/>
 </signal>
 <signal name="TXD">
@@
 <wire x1="30.0736" y1="-18.034" x2="30.0736" y2="-13.3604" width="0.254" layer="1"/>
 <wire x1="29.15" y1="-18.9576" x2="30.0736" y2="-18.034" width="0.254" layer="1"/>
-<wire x1="25.8318" y1="-12.192" x2="25.8318" y2="1.4986" width="0.254" layer="1"/>
+<wire x1="25.8318" y1="-12.192" x2="25.8318" y2="0.9144" width="0.254" layer="1"/>
 <wire x1="18.4016" y1="4.414" x2="18.3" y2="4.414" width="0.254" layer="1"/>
-<wire x1="25.8318" y1="1.4986" x2="24.27806875" y2="3.05233125" width="0.254" layer="1"/>
+<wire x1="25.8318" y1="0.9144" x2="23.92246875" y2="2.82373125" width="0.254" layer="1"/>
 <wire x1="30.0736" y1="-13.3604" x2="29.1846" y2="-12.4714" width="0.254" layer="1"/>
 <wire x1="29.1846" y1="-12.4714" x2="26.1112" y2="-12.4714" width="0.254" layer="1"/>
 <wire x1="26.1112" y1="-12.4714" x2="25.8318" y2="-12.192" width="0.254" layer="1"/>
-<wire x1="18.95046875" y1="3.05233125" x2="18.3" y2="3.7028" width="0.254" layer="1"/>
+<wire x1="19.17906875" y1="2.82373125" x2="18.3" y2="3.7028" width="0.254" layer="1"/>
 <wire x1="18.3" y1="3.7028" x2="18.3" y2="4.414" width="0.254" layer="1"/>
-<wire x1="24.27806875" y1="3.05233125" x2="18.95046875" y2="3.05233125" width="0.254" layer="1"/>
+<wire x1="23.92246875" y1="2.82373125" x2="19.17906875" y2="2.82373125" width="0.254" layer="1"/>
 </signal>
 <signal name="N$1">

Commit message: almost there
Parts:
- removed SJ1: (no value), jumper:SJ
- removed U$2: PINHD-1X10, adafruit:1X10-BIG
- added JP2, JP3: (no value), adafruit:1X08-CLEANBIG
- JP1: device adafruit:1X01 -> adafruit:1X08-CLEANBIG
- moved JP1 61.8 mm to (30.2, 8.66), flipped to the top, turned to 270 degrees
- moved C5 52.2 mm to (10.8, 4.34), turned to 90 degrees
- moved C7 50.8 mm to (19.1, -9.68), turned to 270 degrees
- moved C6 50.2 mm to (21.1, 5.82), turned to 270 degrees
- moved C3 43.8 mm to (24.3, 0.56), turned to 180 degrees
- moved C9 43.8 mm to (10.1, 1.14), turned to 90 degrees
- moved U5 41.7 mm to (16.2, 2.82), turned to 90 degrees
- moved X1 41.6 mm to (23.8, 4.34), turned to 90 degrees
- moved C4 40.5 mm to (23.3, 8.92), turned to 0 degrees
- moved C8 39.5 mm to (13.3, -9.70), turned to 270 degrees
- moved U4 37.4 mm to (16.2, -9.91), turned to 0 degrees
- moved SV1 32.8 mm to (18.9, -4.93), turned to 0 degrees
- moved LED2 7.21 mm to (30.0, -10.5)
- moved R3 4.03 mm to (29.4, -8.48), turned to 180 degrees
- moved C12 3.93 mm to (28.9, -10.6), turned to 90 degrees
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Connections:
- removed net REFIN_CAP: C9.2, SJ1.2
- new net N$10: U2.B2
- new net N$12: U2.B3
- new net N$13: U2.6
- new net N$15: U2.5
- new net N$16: U2.D3
- new net N$17: U2.C3
- new net N$19: U2.12
- new net N$20: U2.D2
- new net N$21: U2.13
- new net N$22: U2.C2
- new net N$23: U2.D1
- new net N$24: U2.C1
- new net N$25: U2.1
- new net N$26: U2.2
- new net N$3: U2.C4
- new net N$4: U2.D4
- new net N$5: U2.11
- new net N$6: U2.8
- new net N$7: U2.7
- new net N$8: U2.B4
- net 3V3: no longer U$2.1
- net CS: now also U2.A4; no longer U$2.9
- net DIN: now also U2.B1; no longer U$2.5
- net DOUT: now also U2.A1; no longer U$2.6
- net DRDY: now also U2.A3; no longer U$2.8
- net GND: no longer U$2.2
- net REFIN: now also C9.2; no longer JP1.1, SJ1.1
- net SCLK: now also U2.A2; no longer U$2.7
- net SYNC/RESET: now also U2.A5; no longer U$2.10
Routing:
- net TXD: track 0.00 -> 34.5 mm, vias 0 -> 4
- net RXD: track 0.00 -> 33.0 mm, vias 0 -> 4
- net AVDD: track 0.00 -> 25.0 mm
- net N$17: track 0.00 -> 21.5 mm, vias 0 -> 1
- net VDD: track 1.93 -> 22.3 mm
- net N$22: track 0.00 -> 19.6 mm, vias 0 -> 1
- net N$24: track 0.00 -> 16.8 mm, vias 0 -> 1
- net N$4: track 0.00 -> 16.4 mm, vias 0 -> 1
- net 0P: track 0.00 -> 16.4 mm
- net XTAL1_2: track 0.00 -> 15.6 mm
- net N$16: track 0.00 -> 15.5 mm, vias 0 -> 1
- net N$20: track 0.00 -> 15.4 mm, vias 0 -> 1
- net N$23: track 0.00 -> 13.9 mm, vias 0 -> 1
- net SYNC/RESET: track 0.00 -> 13.0 mm, vias 0 -> 1
- net XTAL2_2: track 0.00 -> 12.1 mm
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- added copper zone on layer 1, net GND
- added copper zone on layer 16, net GND
Other:
- board size 24.9 x 48 mm -> 24.9 x 50 mm
- board text removed: "Old pins (replace)"
