File: CAD/BM832A.brd (EAGLE design)
At the start: 24.9 x 49.9 mm, 44 parts, among them U1 MCP73831T-3ACI/OT, U3 LP5907MFX-3.3/NOPB, U4 LP5907MFX-3.3/NOPB, U5 ADS131M08IPBS, U6 BCM857BS, U7 CP2102N-A02-GQFN20R, U8 BM832, X1 ABM3B-8.000MHZ-B2-T, X2 FC-12M

Commit message: Update BM832A.brd
Routing:
- net GND: track 41.8 -> 57.8 mm, vias 30 -> 31
- net XTAL1_1: track 11.2 -> 14.1 mm
- net RXD: track 33.9 -> 32.2 mm
- net TXD: track 32.7 -> 31.7 mm
- net XTAL2_1: track 9.33 -> 9.96 mm
