File: CAD/BC840M.brd (EAGLE design)
At the start: 25.2 x 38 mm, 34 parts, among them J1 SM02B-SRSS-TB(LF)(SN), U2 BC840M, U3 LP5907MFX-3.3/NOPB, U4 LP5907MFX-3.3/NOPB, U5 ADS131M08IPBS, X1 ABM3B-8.000MHZ-B2-T, X2 FC-12M

Commit message: updated
Parts:
- removed JP4: (no value), pinhead+:2X10_SMT
- added C16, C17, C20, C21, C24, C25, C28, C29: 0.1pF, standardparts:0603
- added JP2: (no value), pinhead+:2X10_SMT
- added R10, R11, R12, R13, R14, R15, R16, R17, R18, R19, R20, R21, R6, R7, R8, R9: 1GOhm, standardparts:0603
- moved LED2 16.0 mm to (32.6, 34.0), turned to 180 degrees
- moved R2 14.1 mm to (31.4, 34.4)
- moved LED1 12.1 mm to (34.0, 34.0), turned to 180 degrees
- moved C7 11.3 mm to (34.9, 62.3)
- moved U4 6.78 mm to (33.9, 60.1), turned to 0 degrees
- moved R5 6.42 mm to (30.0, 34.4), turned to 180 degrees
- moved C11 5.51 mm to (30.0, 35.2), turned to 180 degrees
- moved C15 4.52 mm to (25.7, 46.7), turned to 180 degrees
- moved R3 4.48 mm to (30.0, 36.3), turned to 180 degrees
- moved C6 3.84 mm to (35.8, 48.6), turned to 270 degrees
- moved J1 2.89 mm to (34.3, 38.2), turned to 90 degrees
- moved C10 2.60 mm to (28.0, 38.1)
- moved C4 2.40 mm to (35.7, 42.3), turned to 90 degrees
- moved C14 2.03 mm to (24.9, 37.7), turned to 180 degrees
- moved C2 1.71 mm to (28.4, 56.9)
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- renumbered JP5 to JP3
Connections:
- removed net N$2: U2.H4, U2.H5, U2.H6, U2.H7
- removed net N$3: U2.F5
- removed net N$4: U2.G4, U2.G5, U2.G6
- removed net N$46: U2.F7
- removed net N$47: U2.F6
- removed net N$5: U2.G0
- removed net N$8: U2.A5
- removed net N$9: U2.A4
- new net 0NIN: C16.2, R8.2, U5.30
- new net 0PIN: C16.1, R6.2, U5.29
- new net 1NIN: C17.2, R9.2, U5.31
- new net 1PIN: C17.1, R7.2, U5.32
- new net 2NIN: C20.2, R12.2, U5.2
- new net 2PIN: C20.1, R10.2, U5.1
- new net 3NIN: C21.2, R13.2, U5.3
- new net 3PIN: C21.1, R11.2, U5.4
- new net 4NIN: C24.2, R16.2, U5.6
- new net 4PIN: C24.1, R14.2, U5.5
- new net 5NIN: C25.2, R17.2, U5.7
- new net 5PIN: C25.1, R15.2, U5.8
- new net 6NIN: C28.2, R20.2, U5.10
- new net 6PIN: C28.1, R18.2, U5.9
- new net 7NIN: C29.2, R21.2, U5.11
- new net 7PIN: C29.1, R19.2, U5.12
- net 0N: now also JP1.2, R8.1; no longer U5.30
- net 0P: now also JP1.1, R6.1; no longer U5.29
- net 1N: now also JP1.4, R9.1; no longer U5.31
- net 1P: now also JP1.3, R7.1; no longer U5.32
- net 2N: now also JP1.6, R12.1; no longer U5.2
- net 2P: now also JP1.5, R10.1; no longer U5.1
- net 3N: now also JP1.8, R13.1; no longer U5.3
- net 3P: now also JP1.7, R11.1; no longer U5.4
- net 4N: now also JP1.10, R16.1; no longer U5.6
- net 4P: now also JP1.9, R14.1; no longer U5.5
- net 5N: now also JP1.12, R17.1; no longer U5.7
- net 5P: now also JP1.11, R15.1; no longer U5.8
- net 6N: now also JP1.14, R20.1; no longer U5.10
- net 6P: now also JP1.13, R18.1; no longer U5.9
- net 7N: now also JP1.16, R21.1; no longer U5.11
- net 7P: now also JP1.15, R19.1; no longer U5.12
- net D+: now also U2.A4
- net D-: now also U2.A5
- net GND: now also U2.G0, U2.G4, U2.G5, U2.G6, U2.H4, U2.H5, U2.H6, U2.H7
- net VDD: now also U2.F5
- net XTAL1_1: now also U2.F6
- net XTAL2_1: now also U2.F7
Routing:
- net VIN: track 12.3 -> 47.7 mm, vias 0 -> 1
- net D+: track 0.00 -> 26.2 mm, vias 0 -> 2
- net D-: track 0.00 -> 25.8 mm
- net +5V: track 0.00 -> 18.5 mm, vias 0 -> 2
- net VDD: track 11.2 -> 28.5 mm, vias 0 -> 1
- net 7PIN: track 0.00 -> 12.9 mm
- net BAT: track 0.00 -> 12.5 mm
- net 7NIN: track 0.00 -> 11.1 mm
- net 0PIN: track 0.00 -> 10.3 mm
- net 6NIN: track 0.00 -> 9.67 mm
- net DIN: track 0.00 -> 9.32 mm
- net 0NIN: track 0.00 -> 8.96 mm
- net 6PIN: track 0.00 -> 8.48 mm
- net 4P: track 0.89 -> 8.78 mm
- net DOUT: track 0.00 -> 7.84 mm
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
Commit message: updated
Parts:
- C16, C17, C20, C21, C24, C25, C28, C29: value 0.1pF -> 10pF
- R10, R11, R12, R13, R14, R15, R16, R17, R18, R19, R20, R21, R6, R7, R8, R9: value 1GOhm -> 10MOhm
Changed lines of the file:
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@@
 </element>
 <element name="C6" library="standardparts" package="0201" value="220uF" x="35.773359375" y="48.630840625" smashed="yes" rot="MR270">
-<attribute name="NAME" x="35.341559375" y="46.878240625" size="0.508" layer="26" rot="MR180"/>
+<attribute name="NAME" x="35.544759375" y="46.898559375" size="0.508" layer="26" rot="MR90"/>
 <attribute name="VALUE" x="34.554159375" y="50.967640625" size="0.508" layer="28" rot="MR180"/>
 </element>
@@
 <attribute name="NAME" x="30.6324" y="33.8836" size="0.4064" layer="25" font="vector" rot="R180"/>
 </element>
-<element name="C16" library="standardparts" package="0603" value="0.1pF" x="25.4" y="43.18" smashed="yes" rot="MR90">
+<element name="C16" library="standardparts" package="0603" value="10pF" x="25.4" y="43.18" smashed="yes" rot="MR90">
 <attribute name="NAME" x="26.162" y="42.6974" size="0.4064" layer="26" font="vector" rot="MR90"/>
 </element>
-<element name="R6" library="standardparts" package="0603" value="1GOhm" x="23.3172" y="42.2656" smashed="yes" rot="MR180">
+<element name="R6" library="standardparts" package="0603" value="10MOhm" x="23.3172" y="42.2656" smashed="yes" rot="MR180">
 <attribute name="NAME" x="21.844" y="42.4942" size="0.4064" layer="26" font="vector" rot="MR270"/>
 </element>
-<element name="C17" library="standardparts" package="0603" value="0.1pF" x="25.4" y="45.847" smashed="yes" rot="MR270">
+<element name="C17" library="standardparts" package="0603" value="10pF" x="25.4" y="45.847" smashed="yes" rot="MR270">
 <attribute name="NAME" x="26.2636" y="45.6184" size="0.4064" layer="26" font="vector" rot="MR90"/>
 </element>
-<element name="R7" library="standardparts" package="0603" value="1GOhm" x="23.2918" y="46.6344" smashed="yes" rot="MR180">
+<element name="R7" library="standardparts" package="0603" value="10MOhm" x="23.2918" y="46.6344" smashed="yes" rot="MR180">
 <attribute name="NAME" x="21.844" y="46.6598" size="0.4064" layer="26" font="vector" rot="MR270"/>
 </element>
-<element name="R8" library="standardparts" package="0603" value="1GOhm" x="23.2918" y="43.7134" smashed="yes" rot="MR180">
+<element name="R8" library="standardparts" package="0603" value="10MOhm" x="23.2918" y="43.7134" smashed="yes" rot="MR180">
 <attribute name="NAME" x="21.8694" y="43.8912" size="0.4064" layer="26" font="vector" rot="MR270"/>
 </element>
-<element name="R9" library="standardparts" package="0603" value="1GOhm" x="23.2918" y="45.1866" smashed="yes" rot="MR180">
+<element name="R9" library="standardparts" package="0603" value="10MOhm" x="23.2918" y="45.1866" smashed="yes" rot="MR180">
 <attribute name="NAME" x="21.844" y="45.2628" size="0.4064" layer="26" font="vector" rot="MR270"/>
 </element>
-<element name="C20" library="standardparts" package="0603" value="0.1pF" x="25.3746" y="48.6664" smashed="yes" rot="MR90">
+<element name="C20" library="standardparts" package="0603" value="10pF" x="25.3746" y="48.6664" smashed="yes" rot="MR90">
 <attribute name="NAME" x="26.2128" y="48.2346" size="0.4064" layer="26" font="vector" rot="MR90"/>
 </element>
-<element name="R10" library="standardparts" package="0603" value="1GOhm" x="23.2918" y="48.1076" smashed="yes" rot="MR180">
+<element name="R10" library="standardparts" package="0603" value="10MOhm" x="23.2918" y="48.1076" smashed="yes" rot="MR180">
 <attribute name="NAME" x="21.8186" y="48.6156" size="0.4064" layer="26" font="vector" rot="MR270"/>
 </element>
-<element name="C21" library="standardparts" package="0603" value="0.1pF" x="25.3492" y="51.435" smashed="yes" rot="MR270">
+<element name="C21" library="standardparts" package="0603" value="10pF" x="25.3492" y="51.435" smashed="yes" rot="MR270">
 <attribute name="NAME" x="26.1366" y="51.0032" size="0.4064" layer="26" font="vector" rot="MR90"/>
 </element>
-<element name="R11" library="standardparts" package="0603" value="1GOhm" x="23.3172" y="52.4256" smashed="yes" rot="MR180">
+<element name="R11" library="standardparts" package="0603" value="10MOhm" x="23.3172" y="52.4256" smashed="yes" rot="MR180">
 <attribute name="NAME" x="21.4884" y="51.8922" size="0.4064" layer="26" font="vector" rot="MR90"/>
 </element>
-<element name="R12" library="standardparts" package="0603" value="1GOhm" x="23.2918" y="49.53" smashed="yes" rot="MR180">
+<element name="R12" library="standardparts" package="0603" value="10MOhm" x="23.2918" y="49.53" smashed="yes" rot="MR180">
 <attribute name="NAME" x="21.844" y="50.0126" size="0.4064" layer="26" font="vector" rot="MR270"/>
 </element>
-<element name="R13" library="standardparts" package="0603" value="1GOhm" x="23.3172" y="50.9778" smashed="yes" rot="MR180">
+<element name="R13" library="standardparts" package="0603" value="10MOhm" x="23.3172" y="50.9778" smashed="yes" rot="MR180">
 <attribute name="NAME" x="21.8694" y="51.435" size="0.4064" layer="26" font="vector" rot="MR270"/>
 </element>
-<element name="C24" library="standardparts" package="0603" value="0.1pF" x="25.3238" y="54.5846" smashed="yes" rot="MR90">
+<element name="C24" library="standardparts" package="0603" value="10pF" x="25.3238" y="54.5846" smashed="yes" rot="MR90">
 <attribute name="NAME" x="26.1366" y="54.229" size="0.4064" layer="26" font="vector" rot="MR90"/>
 </element>
-<element name="R14" library="standardparts" package="0603" value="1GOhm" x="23.2918" y="53.8734" smashed="yes" rot="MR180">
+<element name="R14" library="standardparts" package="0603" value="10MOhm" x="23.2918" y="53.8734" smashed="yes" rot="MR180">
 <attribute name="NAME" x="21.4884" y="53.467" size="0.4064" layer="26" font="vector" rot="MR90"/>
 </element>
-<element name="C25" library="standardparts" package="0603" value="0.1pF" x="25.3238" y="57.4294" smashed="yes" rot="MR270">
+<element name="C25" library="standardparts" package="0603" value="10pF" x="25.3238" y="57.4294" smashed="yes" rot="MR270">
 <attribute name="NAME" x="26.162" y="57.023" size="0.4064" layer="26" font="vector" rot="MR90"/>
 </element>
-<element name="R15" library="standardparts" package="0603" value="1GOhm" x="23.2918" y="58.166" smashed="yes" rot="MR180">
+<element name="R15" library="standardparts" package="0603" value="10MOhm" x="23.2918" y="58.166" smashed="yes" rot="MR180">
 <attribute name="NAME" x="21.4376" y="57.7088" size="0.4064" layer="26" font="vector" rot="MR90"/>
 </element>
-<element name="R16" library="standardparts" package="0603" value="1GOhm" x="23.2918" y="55.3212" smashed="yes" rot="MR180">
+<element name="R16" library="standardparts" package="0603" value="10MOhm" x="23.2918" y="55.3212" smashed="yes" rot="MR180">
 <attribute name="NAME" x="21.4884" y="54.8132" size="0.4064" layer="26" font="vector" rot="MR90"/>
 </element>
-<element name="R17" library="standardparts" package="0603" value="1GOhm" x="23.2918" y="56.769" smashed="yes" rot="MR180">
+<element name="R17" library="standardparts" package="0603" value="10MOhm" x="23.2918" y="56.769" smashed="yes" rot="MR180">
 <attribute name="NAME" x="21.4884" y="56.2356" size="0.4064" layer="26" font="vector" rot="MR90"/>
 </element>
-<element name="C28" library="standardparts" package="0603" value="0.1pF" x="25.3238" y="60.325" smashed="yes" rot="MR90">
+<element name="C28" library="standardparts" package="0603" value="10pF" x="25.3238" y="60.325" smashed="yes" rot="MR90">
 <attribute name="NAME" x="26.162" y="59.8678" size="0.4064" layer="26" font="vector" rot="MR90"/>
 </element>
-<element name="R18" library="standardparts" package="0603" value="1GOhm" x="23.2918" y="59.6138" smashed="yes" rot="MR180">
+<element name="R18" library="standardparts" package="0603" value="10MOhm" x="23.2918" y="59.6138" smashed="yes" rot="MR180">
 <attribute name="NAME" x="21.463" y="59.1566" size="0.4064" layer="26" font="vector" rot="MR90"/>
 </element>
-<element name="C29" library="standardparts" package="0603" value="0.1pF" x="25.2984" y="63.1952" smashed="yes" rot="MR270">
+<element name="C29" library="standardparts" package="0603" value="10pF" x="25.2984" y="63.1952" smashed="yes" rot="MR270">
 <attribute name="NAME" x="26.2382" y="62.7888" size="0.4064" layer="26" font="vector" rot="MR90"/>
 </element>
-<element name="R19" library="standardparts" package="0603" value="1GOhm" x="23.2156" y="64.1096" smashed="yes" rot="MR180">
+<element name="R19" library="standardparts" package="0603" value="10MOhm" x="23.2156" y="64.1096" smashed="yes" rot="MR180">
 <attribute name="NAME" x="21.3868" y="63.6778" size="0.4064" layer="26" font="vector" rot="MR90"/>
 </element>
-<element name="R20" library="standardparts" package="0603" value="1GOhm" x="23.2664" y="61.0616" smashed="yes" rot="MR180">
+<element name="R20" library="standardparts" package="0603" value="10MOhm" x="23.2664" y="61.0616" smashed="yes" rot="MR180">
 <attribute name="NAME" x="21.463" y="60.5536" size="0.4064" layer="26" font="vector" rot="MR90"/>
 </element>
-<element name="R21" library="standardparts" package="0603" value="1GOhm" x="23.2664" y="62.5348" smashed="yes" rot="MR180">
+<element name="R21" library="standardparts" package="0603" value="10MOhm" x="23.2664" y="62.5348" smashed="yes" rot="MR180">
 <attribute name="NAME" x="21.463" y="62.0522" size="0.4064" layer="26" font="vector" rot="MR90"/>
 </element>
@@
 <contactref element="U3" pad="2"/>
 <polygon width="0.1524" layer="16">
-<vertex x="13.0764" y="63.439040625"/>
+<vertex x="13.0764" y="64.759840625"/>
 <vertex x="13.0764" y="45.327171875"/>
-<vertex x="13.084084375" y="41.78133125"/>
-<vertex x="27.077753125" y="41.78133125"/>
+<vertex x="13.084359375" y="41.65433125"/>
+<vertex x="26.950753125" y="41.65433125"/>
 <vertex x="31.021503125" y="45.72508125"/>
 <vertex x="31.021503125" y="52.092859375"/>
@@
 <vertex x="33.8836" y="63.422065625"/>
 <vertex x="32.642025" y="63.439040625"/>
+<vertex x="31.321225" y="64.759840625"/>
 </polygon>
 <contactref element="C15" pad="1"/>

Commit message: Update BC840M.brd
Parts:
- moved C20 1.27 mm to (25.3, 47.4)
- moved C21 1.27 mm to (25.2, 50.2)
- moved C29 1.27 mm to (25.2, 61.9)
- moved R11 1.27 mm to (23.2, 51.2)
- moved R13 1.27 mm to (23.2, 49.7)
- moved C16 1.27 mm to (25.3, 41.9)
- moved C17 1.27 mm to (25.3, 44.6)
- moved C24 1.27 mm to (25.2, 53.3)
- moved C25 1.27 mm to (25.2, 56.2)
- moved C28 1.27 mm to (25.2, 59.1)
- moved JP1 1.27 mm to (17.2, 51.7)
- moved R12 1.27 mm to (23.2, 48.3)
- moved R19 1.27 mm to (23.1, 62.8)
- moved R8 1.27 mm to (23.2, 42.4)
- moved R20 1.27 mm to (23.2, 59.8)
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Routing:
- net 0PIN: track 10.3 -> 12.0 mm
- net 2PIN: track 4.84 -> 6.17 mm
- net 0NIN: track 8.96 -> 10.2 mm
- net 6NIN: track 9.67 -> 8.44 mm
- net 5PIN: track 7.64 -> 6.41 mm
- net 7PIN: track 12.9 -> 11.7 mm
- net 7NIN: track 11.1 -> 9.88 mm
- net 6PIN: track 8.48 -> 7.26 mm
- net D+: track 26.2 -> 25.3 mm
- net 1NIN: track 7.76 -> 8.65 mm
- net 2NIN: track 4.14 -> 4.97 mm
- net 5NIN: track 6.64 -> 5.87 mm
- net 3NIN: track 3.93 -> 4.58 mm
- net 4NIN: track 5.96 -> 5.32 mm
- net 1PIN: track 6.31 -> 6.93 mm

Commit message: Update BC840M.brd
Parts:
- moved JP3 0.33 mm to (33.8, 54.2)
Changed lines of the file:
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@@
 <attribute name="VALUE" x="24.20111875" y="39.01948125" size="1.27" layer="27" rot="R90"/>
 </element>
-<element name="JP3" library="pinhead+" package="2X10_SMT" value="" x="33.7566" y="53.8988" smashed="yes" rot="R90">
-<attribute name="NAME" x="35.265359375" y="65.8012375" size="1.27" layer="25" ratio="10" rot="R180"/>
-<attribute name="VALUE" x="40.7416" y="41.1988" size="1.27" layer="27" rot="R90"/>
+<element name="JP3" library="pinhead+" package="2X10_SMT" value="" x="33.7566" y="54.229" smashed="yes" rot="R90">
+<attribute name="NAME" x="35.265359375" y="66.1314375" size="1.27" layer="25" ratio="10" rot="R180"/>
+<attribute name="VALUE" x="40.7416" y="41.529" size="1.27" layer="27" rot="R90"/>
 </element>
 <element name="R1" library="standardparts" package="0201" value="46.4kΩ" x="27.2034" y="38.1254" smashed="yes" rot="R90">
@@
 <wire x1="28.2194" y1="42.0826" x2="29.916" y2="40.386" width="0.254" layer="1"/>
 <wire x1="33.9344" y1="38.989" x2="34.4678" y2="39.5224" width="0.254" layer="1"/>
-<wire x1="34.4678" y1="56.7182" x2="34.8742" y2="57.1246" width="0.254" layer="1"/>
-<wire x1="34.4678" y1="56.7182" x2="34.4678" y2="39.5224" width="0.254" layer="1"/>
-<via x="34.8742" y="57.1246" extent="1-16" drill="0.35"/>
+<wire x1="34.4678" y1="57.6834" x2="34.5694" y2="57.785" width="0.254" layer="1"/>
+<wire x1="34.4678" y1="57.6834" x2="34.4678" y2="39.5224" width="0.254" layer="1"/>
+<via x="34.5694" y="57.785" extent="1-16" drill="0.35"/>
 <wire x1="35.19955625" y1="59.11084375" x2="35.2298" y2="59.0806" width="0.254" layer="16"/>
-<wire x1="35.2298" y1="59.0806" x2="35.2298" y2="57.4802" width="0.254" layer="16"/>
-<wire x1="34.8742" y1="57.1246" x2="35.2298" y2="57.4802" width="0.254" layer="16"/>
+<wire x1="35.2298" y1="59.0806" x2="35.2298" y2="58.4454" width="0.254" layer="16"/>
+<wire x1="34.5694" y1="57.785" x2="35.2298" y2="58.4454" width="0.254" layer="16"/>
 </signal>
 <signal name="N$6">

Commit message: Update BC840M.brd
Parts:
- moved C7 0.70 mm to (34.2, 62.4)
- moved U4 0.70 mm to (33.3, 60.2)
- moved C8 0.70 mm to (31.0, 58.2)
Routing:
- net SCLK: track 6.89 -> 16.5 mm
- net DRDY: track 6.01 -> 15.5 mm
- net DOUT: track 7.84 -> 17.3 mm
- net CS: track 5.28 -> 14.6 mm
- net SYNC/RESET: track 5.09 -> 14.0 mm
- net DIN: track 9.32 -> 18.1 mm
- net GND: track 2.70 -> 5.92 mm, vias 1 -> 2
- net 7PIN: track 11.7 -> 12.9 mm
- net 7NIN: track 9.88 -> 11.0 mm
- net 6NIN: track 8.44 -> 9.51 mm

Commit message: i/o prerouting
Parts:
- moved C1 2.22 mm to (26.6, 55.8), turned to 180 degrees
- moved C29 0.87 mm to (24.6, 61.3)
- moved C2 0.63 mm to (29.0, 56.7)
- moved X2 0.63 mm to (27.1, 57.1)
- moved R18 0.63 mm to (22.6, 58.4)
- moved R20 0.61 mm to (22.6, 59.9)
- moved R21 0.61 mm to (22.6, 61.4)
- moved C28 0.58 mm to (24.8, 58.7)
- moved C20 0.57 mm to (24.7, 47.5)
- moved R19 0.56 mm to (22.6, 62.8)
- moved C16 0.50 mm to (24.8, 42.0)
- moved C17 0.50 mm to (24.8, 44.6)
- moved C24 0.50 mm to (24.7, 53.4)
- moved R12 0.50 mm to (22.7, 48.3)
- moved R14 0.50 mm to (22.7, 52.6)
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Connections:
- net N$10 renamed SWDIO
- net N$11 renamed P104
- net N$12 renamed P101
- net N$13 renamed P25
- net N$14 renamed P19
- net N$15 renamed P17
- net N$16 renamed P22
- net N$17 renamed P15
- net N$18 renamed RESET
- net N$19 renamed VBUS
- net N$20 renamed P7
- net N$21 renamed P12
- net N$22 renamed P107
- net N$23 renamed SWDCLK
- net N$24 renamed P20
- net N$25 renamed P21
- net N$26 renamed P14
- net N$27 renamed P108
- net N$28 renamed P109
- net N$29 renamed P8
- net N$30 renamed P100
- net N$31 renamed P105
- net N$32 renamed P9
- net N$33 renamed P16
- net N$34 renamed P13
- net N$35 renamed P11
- net N$36 renamed P27
- net N$37 renamed P6
- net N$38 renamed P103
- net N$39 renamed P106
- net N$40 renamed P10
- net N$41 renamed P115
- net N$42 renamed P29
- net N$43 renamed P31
- net N$44 renamed P26
- net N$45 renamed P4
- net N$49 renamed P2
- net N$50 renamed P112
- net N$51 renamed P102
- net N$52 renamed P24
- net N$53 renamed P23
- net N$54 renamed P5
- net N$55 renamed P113
- net N$56 renamed P111
- net N$57 renamed P30
- net N$58 renamed P114
- net N$59 renamed P110
- net N$6 renamed VDDH
- net N$60 renamed P28
- net N$61 renamed P3
- net N$7 renamed DCCH
Routing:
- net D+: track 25.3 -> 9.11 mm
- net D-: track 26.1 -> 10.7 mm
- net P31: track 0.00 -> 5.36 mm
- net N$7: track 0.00 -> 4.42 mm, vias 0 -> 1
- net N$2: track 0.00 -> 4.23 mm, vias 0 -> 1
- net N$8: track 0.00 -> 4.12 mm, vias 0 -> 1
- net N$4: track 0.00 -> 3.38 mm, vias 0 -> 1
- net P29: track 0.00 -> 3.27 mm
- net N$6: track 0.00 -> 3.21 mm, vias 0 -> 1
- net P14: track 0.00 -> 3.11 mm
- net P21: track 0.00 -> 3.09 mm
- net P20: track 0.00 -> 3.07 mm
- net P11: track 0.00 -> 2.99 mm
- net P26: track 0.00 -> 2.94 mm
- net P109: track 0.00 -> 2.81 mm
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
Commit message: Update BC840M.brd
Routing:
- net P15: track 2.18 -> 30.2 mm
- net P14: track 3.11 -> 30.4 mm
- net P25: track 0.71 -> 26.5 mm
- net P100: track 0.79 -> 25.3 mm, vias 0 -> 2
- net P22: track 2.23 -> 25.9 mm
- net P17: track 0.79 -> 24.3 mm
- net D+: track 9.11 -> 31.6 mm
- net D-: track 10.7 -> 32.3 mm
- net P101: track 0.71 -> 22.2 mm
- net P104: track 0.84 -> 18.9 mm
- net P21: track 3.09 -> 20.0 mm
- net P107: track 0.82 -> 15.5 mm
- net P4: track 2.39 -> 15.4 mm
- net P108: track 2.23 -> 13.7 mm, vias 0 -> 2
- net SWDIO: track 1.28 -> 12.5 mm, vias 0 -> 2
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Other:
- board text added: "CLKIN"
- board text added: "CLKOUT"

Commit message: updated
Parts:
- added JP4: (no value), pinhead+:2X11_SMT
- moved C2 1.27 mm to (28.1, 55.8), turned to 0 degrees
- moved U$1 0.50 mm to (20.4, 34.9)
- moved C1 0.05 mm to (26.6, 55.8)
Routing:
- net P27: track 8.43 -> 20.5 mm
- net P5: track 2.51 -> 11.7 mm
- net P6: track 10.4 -> 19.3 mm
- net P31: track 5.36 -> 12.6 mm
- net P26: track 13.3 -> 20.1 mm
- net P8: track 7.21 -> 13.8 mm
- net P4: track 15.4 -> 19.1 mm
- net D+: track 31.6 -> 34.1 mm
- net P12: track 10.9 -> 8.46 mm
- net GND: track 7.98 -> 9.98 mm
- net VIN: track 47.4 -> 49.3 mm
