File: CAD/BC840M.sch (EAGLE design)
At the start: 61 parts, among them J1 SM02B-SRSS-TB(LF)(SN), U2 BC840M, U3 LP5907MFX-3.3/NOPB, U4 LP5907MFX-3.3/NOPB, U5 ADS131M08IPBS, X1 ABM3B-8.000MHZ-B2-T, X2 FC-12M

Commit message: latest
Parts:
- added C18, C22: 0.1uF, standardparts:CAPACITOR.0201
- added C19: 10nF, standardparts:CAPACITOR.0201
- added C23: 1uF, standardparts:CAPACITOR.0201
- added CS, DIN, DOUT, DRDY, SCLK: TPTP07R, testpad:TPTP07R
- added LED1, LED2, LED3: (no value), adafruit:LEDCHIPLED_0603
- added NFC1, NFC2: TPTP14SQ, testpad:TPTP14SQ
- added R26, R27, R5: 3.3kΩ, standardparts:RESISTOR.0201
- added U$3: 120Ω/500mAh, spkfncoils:12NH-0402
- C6: value 220uF -> 220nF
Connections:
- net P100 renamed SWO
- removed net P10: U2.E2/P010
- removed net P102: U2.F2/P102
- removed net P103: U2.E0/P103
- removed net P105: U2.D1/P105
- removed net P112: U2.F3/P112
- removed net P115: U2.E3/P115
- removed net P13: U2.D4/P013
- removed net P9: U2.D2/P009
- new net +5V_ISO: C10.2, C18.1, U$2.IN, U$3.1, U2.B5/VBUS
- new net LED1: LED1.A, R5.2
- new net LED2: LED2.A, R26.2
- new net LED3: LED3.A, R27.2
- new net NFC1: NFC2.TP, U2.D2/P009
- new net NFC2: NFC1.TP, U2.E2/P010
- net +5V: now also C19.2, U$3.2; no longer C10.2, U$2.IN, U2.B5/VBUS
- net CS: now also CS.TP, U2.E3/P115
- net DIN: now also DIN.TP, U2.E0/P103
- net DOUT: now also DOUT.TP, U2.F2/P102
- net DRDY: now also DRDY.TP, U2.D1/P105
- net GND: now also C18.2, C19.1, C22.1, C23.1, LED1.C, LED2.C, LED3.C
- net P16: now also R26.1
- net P20: now also R27.1
- net P26: now also R5.1
- net SCLK: now also SCLK.TP, U2.F3/P112
- net SYNC/RESET: now also U2.D4/P013
- net VDD: now also C22.2, C23.2
