File: CAD/BC840M.sch (EAGLE design)
At the start: 90 parts, among them J1 S2B-PH-SM4-TB(LF)(SN), U1 TPD4S012DRYR, U2 BC840M, U3 LP5907MFX-3.3/NOPB, U4 LP5907MFX-3.3/NOPB, U5 ADS131M08IPBS, U6 BQ24072RGTR, U7 DX4R005JJ2R1800, X1 ABM3B-8.000MHZ-B2-T, X2 FC-12M

Commit message: fix
Parts:
- J1: value S2B-PH-SM4-TB(LF)(SN) -> SM02B-SRSS-TB(LF)(SN); device S2B-PH-SM4-TB_LF__SN_:S2B-PH-SM4-TB(LF)(SN) -> SM02B-SRSS-TB_LF__SN_:SM02B-SRSS-TB(LF)(SN)
Changed lines of the file:
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@@
 <part name="U2" library="BC840M" deviceset="BC840M" device=""/>
 <part name="U6" library="BQ24072RGTR" deviceset="BQ24072RGTR" device=""/>
-<part name="J1" library="S2B-PH-SM4-TB_LF__SN_" deviceset="S2B-PH-SM4-TB(LF)(SN)" device=""/>
 <part name="JP1" library="pinhead+" deviceset="PINHD-2X8" device="SMT"/>
 <part name="JP2" library="pinhead+" deviceset="PINHD-2X10" device="SMT"/>
@@
 <part name="C30" library="standardparts" deviceset="CAPACITOR" device=".0201" value="0.1uF"/>
 <part name="C31" library="standardparts" deviceset="CAPACITOR" device=".0402" value="10uF"/>
+<part name="J1" library="SM02B-SRSS-TB_LF__SN_" deviceset="SM02B-SRSS-TB(LF)(SN)" device=""/>
 </parts>
 <sheets>
@@
 <attribute name="VALUE" x="55.7022" y="84.265" size="2.0828" layer="96" ratio="10" rot="SR0"/>
 </instance>
-<instance part="J1" gate="G$1" x="89.1286" y="37.9476" smashed="yes">
-<attribute name="NAME" x="95.85583125" y="34.252" size="1.78541875" layer="95" rot="R90" align="center-left"/>
-<attribute name="VALUE" x="105.7556" y="30.283959375" size="1.784809375" layer="96" rot="R180" align="center-left"/>
-</instance>
 <instance part="JP1" gate="A" x="328.5236" y="120.3706" smashed="yes">
 <attribute name="NAME" x="322.1736" y="131.1656" size="1.778" layer="95"/>
@@
 <attribute name="NAME" x="23.5204" y="75.0824" size="1.016" layer="95" rot="MR0"/>
 <attribute name="VALUE" x="23.5204" y="77.6224" size="1.016" layer="96" rot="R180"/>
+</instance>
+<instance part="J1" gate="G$1" x="84.8868" y="34.163" smashed="yes">
+<attribute name="NAME" x="96.3804" y="39.27216875" size="1.78541875" layer="95" align="center-left"/>
+<attribute name="VALUE" x="96.3776" y="36.721240625" size="1.784809375" layer="96" align="center-left"/>
 </instance>
 </instances>
@@
 <junction x="37.719" y="35.9156"/>
 <pinref part="SUPPLY13" gate="GND" pin="GND"/>
-</segment>
-<segment>
-<wire x1="84.0486" y1="39.2176" x2="80.4672" y2="39.2176" width="0.1524" layer="91"/>
-<wire x1="80.4672" y1="39.2176" x2="80.4672" y2="45.9994" width="0.1524" layer="91"/>
-<pinref part="SUPPLY7" gate="GND" pin="GND"/>
-<wire x1="80.4672" y1="45.9994" x2="75.9714" y2="45.9994" width="0.1524" layer="91"/>
-<pinref part="J1" gate="G$1" pin="1"/>
 </segment>
 <segment>
@@
 <label x="22.7076" y="68.6562" size="1.778" layer="95"/>
 </segment>
+<segment>
+<pinref part="J1" gate="G$1" pin="1"/>
+<wire x1="84.8868" y1="39.243" x2="80.4926" y2="39.243" width="0.1524" layer="91"/>
+<wire x1="80.4926" y1="39.243" x2="80.4672" y2="45.9994" width="0.1524" layer="91"/>
+<pinref part="SUPPLY7" gate="GND" pin="GND"/>
+<wire x1="80.4672" y1="45.9994" x2="75.9714" y2="45.9994" width="0.1524" layer="91"/>
+</segment>
 </net>
 <net name="CLKIN" class="0">
@@
 </segment>
 <segment>
-<pinref part="J1" gate="G$1" pin="2"/>
-<wire x1="84.0486" y1="36.6776" x2="77.8764" y2="36.6522" width="0.1524" layer="91"/>
+<wire x1="84.0486" y1="36.703" x2="77.8764" y2="36.6522" width="0.1524" layer="91"/>
 <wire x1="77.8764" y1="36.6522" x2="77.8764" y2="36.6776" width="0.1524" layer="91"/>
 <label x="77.851" y="35.179" size="1.778" layer="95" rot="R180"/>
-</segment>
-<segment>
+<pinref part="J1" gate="G$1" pin="2"/>
+<wire x1="84.8868" y1="36.703" x2="84.0486" y2="36.703" width="0.1524" layer="91"/>
+</segment>
+<segment>
