File: CAD/CP2012_20Pin/BT832A.brd (EAGLE design)
At the start: 24.9 x 49.9 mm, 44 parts, among them U1 MCP73831T-3ACI/OT, U2 BT832, U3 LP5907MFX-3.3/NOPB, U4 LP5907MFX-3.3/NOPB, U5 ADS131M08IPBS, U6 BCM857BS, U7 CP2102N-A02-GQFN20R, X1 ABM3B-8.000MHZ-B2-T, X2 FC-12M

Commit message: edits
Parts:
- moved D1 0.25 mm to (19.7, -10.6)
Other:
- outline, holes or cut-outs redrawn
Changed lines of the file:
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@@
 <dimension x1="31.496" y1="-29.083" x2="29.464" y2="20.828" x3="34.5186" y3="-4.1275" textsize="1.778" layer="47" dtype="vertical"/>
 <text x="18.5928" y="0.508" size="0.3048" layer="22" rot="MR0">TOP</text>
+<wire x1="20.828" y1="-28.194" x2="20.828" y2="-27.432" width="0.1016" layer="20"/>
+<wire x1="20.828" y1="-27.432" x2="21.082" y2="-27.178" width="0.1016" layer="20" curve="-90"/>
+<wire x1="21.082" y1="-27.178" x2="21.336" y2="-27.178" width="0.1016" layer="20"/>
+<wire x1="21.336" y1="-27.178" x2="21.59" y2="-27.432" width="0.1016" layer="20" curve="-90"/>
+<wire x1="21.59" y1="-27.432" x2="21.59" y2="-28.194" width="0.1016" layer="20"/>
+<wire x1="21.59" y1="-28.194" x2="21.336" y2="-28.448" width="0.1016" layer="20" curve="-90"/>
+<wire x1="21.336" y1="-28.448" x2="21.082" y2="-28.448" width="0.1016" layer="20"/>
+<wire x1="21.082" y1="-28.448" x2="20.828" y2="-28.194" width="0.1016" layer="20" curve="-90"/>
+<wire x1="27.686" y1="-27.432" x2="27.94" y2="-27.178" width="0.1016" layer="20" curve="-90"/>
+<wire x1="27.94" y1="-27.178" x2="28.194" y2="-27.178" width="0.1016" layer="20"/>
+<wire x1="28.194" y1="-27.178" x2="28.448" y2="-27.432" width="0.1016" layer="20" curve="-90"/>
+<wire x1="28.448" y1="-27.432" x2="28.448" y2="-28.194" width="0.1016" layer="20"/>
+<wire x1="28.448" y1="-28.194" x2="28.194" y2="-28.448" width="0.1016" layer="20" curve="-90"/>
+<wire x1="28.194" y1="-28.448" x2="27.94" y2="-28.448" width="0.1016" layer="20"/>
+<wire x1="27.94" y1="-28.448" x2="27.686" y2="-28.194" width="0.1016" layer="20" curve="-90"/>
+<wire x1="27.686" y1="-28.194" x2="27.686" y2="-27.432" width="0.1016" layer="20"/>
+<wire x1="26.924" y1="-25.273" x2="27.432" y2="-25.273" width="0.1016" layer="20"/>
+<wire x1="27.432" y1="-25.273" x2="27.686" y2="-25.019" width="0.1016" layer="20" curve="90"/>
+<wire x1="27.686" y1="-25.019" x2="27.686" y2="-24.765" width="0.1016" layer="20"/>
+<wire x1="27.686" y1="-24.765" x2="27.432" y2="-24.511" width="0.1016" layer="20" curve="90"/>
+<wire x1="27.432" y1="-24.511" x2="26.924" y2="-24.511" width="0.1016" layer="20"/>
+<wire x1="26.924" y1="-24.511" x2="26.67" y2="-24.765" width="0.1016" layer="20" curve="90"/>
+<wire x1="26.67" y1="-24.765" x2="26.67" y2="-25.019" width="0.1016" layer="20"/>
+<wire x1="26.67" y1="-25.019" x2="26.924" y2="-25.273" width="0.1016" layer="20" curve="90"/>
+<wire x1="21.844" y1="-25.273" x2="22.352" y2="-25.273" width="0.1016" layer="20"/>
+<wire x1="22.352" y1="-25.273" x2="22.606" y2="-25.019" width="0.1016" layer="20" curve="90"/>
+<wire x1="22.606" y1="-25.019" x2="22.606" y2="-24.765" width="0.1016" layer="20"/>
+<wire x1="22.606" y1="-24.765" x2="22.352" y2="-24.511" width="0.1016" layer="20" curve="90"/>
+<wire x1="22.352" y1="-24.511" x2="21.844" y2="-24.511" width="0.1016" layer="20"/>
+<wire x1="21.844" y1="-24.511" x2="21.59" y2="-24.765" width="0.1016" layer="20" curve="90"/>
+<wire x1="21.59" y1="-24.765" x2="21.59" y2="-25.019" width="0.1016" layer="20"/>
+<wire x1="21.59" y1="-25.019" x2="21.844" y2="-25.273" width="0.1016" layer="20" curve="90"/>
+<rectangle x1="20.574" y1="-28.702" x2="21.971" y2="-26.924" layer="29"/>
+<rectangle x1="21.336" y1="-25.527" x2="22.987" y2="-24.257" layer="29"/>
+<rectangle x1="26.289" y1="-25.527" x2="27.94" y2="-24.257" layer="29"/>
+<rectangle x1="27.305" y1="-28.702" x2="28.702" y2="-26.924" layer="29"/>
+<rectangle x1="21.4376" y1="-25.4762" x2="22.8346" y2="-24.3078" layer="31"/>
+<rectangle x1="26.4414" y1="-25.4762" x2="27.8384" y2="-24.3078" layer="31"/>
+<rectangle x1="27.3558" y1="-28.6258" x2="28.6512" y2="-26.9494" layer="31"/>
+<rectangle x1="20.6248" y1="-28.6258" x2="21.9202" y2="-26.9494" layer="31"/>
 </plain>
 <attributes>
@@
 <attribute name="VALUE" x="14.36021875" y="-17.563490625" size="0.381" layer="27" ratio="10" rot="SR90"/>
 </element>
-<element name="D1" library="diode" library_urn="urn:adsk.eagle:library:210" package="SOD323_ST" package3d_urn="urn:adsk.eagle:package:43461/1" value="BAT60J" x="19.8628" y="-10.4648" smashed="yes" rot="R180">
-<attribute name="NAME" x="20.4968" y="-9.1828" size="0.508" layer="25" rot="R180"/>
-<attribute name="POPULARITY" value="7" x="19.8628" y="-10.4648" size="1.778" layer="27" rot="R180" display="off"/>
+<element name="D1" library="diode" library_urn="urn:adsk.eagle:library:210" package="SOD323_ST" package3d_urn="urn:adsk.eagle:package:43461/1" value="BAT60J" x="19.6596" y="-10.6172" smashed="yes" rot="R180">
+<attribute name="NAME" x="20.2936" y="-9.3352" size="0.508" layer="25" rot="R180"/>
+<attribute name="POPULARITY" value="7" x="19.6596" y="-10.6172" size="1.778" layer="27" rot="R180" display="off"/>
 </element>
 <element name="D2" library="diode" library_urn="urn:adsk.eagle:library:210" package="SOT23" package3d_urn="urn:adsk.eagle:package:43389/2" value="BAS40-06" x="18.0594" y="-20.4978" smashed="yes" rot="R270">
@@
 <contactref element="D1" pad="A"/>
 <contactref element="R6" pad="2"/>
-<wire x1="18.6128" y1="-10.4648" x2="18.052" y2="-10.4648" width="0.254" layer="1"/>
-<wire x1="18.052" y1="-10.4648" x2="17.079" y2="-11.4378" width="0.254" layer="1"/>
+<wire x1="18.4096" y1="-10.6172" x2="17.8996" y2="-10.6172" width="0.254" layer="1"/>
+<wire x1="17.8996" y1="-10.6172" x2="17.079" y2="-11.4378" width="0.254" layer="1"/>
 <wire x1="17.079" y1="-11.4378" x2="17.079" y2="-11.7426" width="0.254" layer="1"/>
 <wire x1="21.2852" y1="-13.3454" x2="21.2852" y2="-13.3326" width="0.254" layer="1"/>
@@
 <contactref element="C7" pad="1"/>
 <contactref element="C13" pad="2"/>
-<wire x1="22.7838" y1="-10.6276" x2="22.758509375" y2="-10.4648" width="0.254" layer="1"/>
-<wire x1="21.1128" y1="-10.4648" x2="22.758509375" y2="-10.4648" width="0.254" layer="1"/>
+<wire x1="22.7838" y1="-10.6276" x2="22.782184375" y2="-10.6172" width="0.254" layer="1"/>
+<wire x1="20.9096" y1="-10.6172" x2="22.782184375" y2="-10.6172" width="0.254" layer="1"/>
 <wire x1="24.6276" y1="-9.7688" x2="23.3576" y2="-9.7688" width="0.254" layer="1"/>
 <wire x1="23.3576" y1="-9.7688" x2="22.7838" y2="-10.3426" width="0.254" layer="1"/>
@@
 <wire x1="16.07644375" y1="-10.668" x2="15.179" y2="-11.555803125" width="0.254" layer="1"/>
 <wire x1="15.179" y1="-11.7426" x2="15.179" y2="-11.555803125" width="0.254" layer="1"/>
-<wire x1="21.1128" y1="-9.5758" x2="21.1128" y2="-10.4648" width="0.254" layer="1"/>
+<wire x1="21.1128" y1="-9.5758" x2="21.1128" y2="-10.414" width="0.254" layer="1"/>
+<wire x1="21.1128" y1="-10.414" x2="20.9096" y2="-10.6172" width="0.254" layer="1"/>
 <wire x1="21.0366" y1="-9.652" x2="17.8562" y2="-9.652" width="0.254" layer="1"/>
 <wire x1="21.0366" y1="-9.652" x2="21.1128" y2="-9.5758" width="0.254" layer="1"/>
