File: CAD/CP2102_24Pin/BT832A.brd (EAGLE design)
At the start: 24.9 x 49.9 mm, 44 parts, among them IC1 CP2102, U1 MCP73831T-3ACI/OT, U2 BT832, U3 LP5907MFX-3.3/NOPB, U4 LP5907MFX-3.3/NOPB, U5 ADS131M08IPBS, U6 BCM857BS, X1 ABM3B-8.000MHZ-B2-T, X2 FC-12M

Commit message: edits
Other:
- outline, holes or cut-outs redrawn
Changed lines of the file:
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@@
 <dimension x1="31.496" y1="-29.083" x2="29.464" y2="20.828" x3="34.5186" y3="-4.1275" textsize="1.778" layer="47" dtype="vertical"/>
 <text x="18.5928" y="0.508" size="0.3048" layer="22" rot="MR0">TOP</text>
+<wire x1="20.828" y1="-28.1686" x2="20.828" y2="-27.3812" width="0.1524" layer="20"/>
+<wire x1="20.828" y1="-27.3812" x2="21.0566" y2="-27.1526" width="0.1524" layer="20" curve="-90"/>
+<wire x1="21.0566" y1="-27.1526" x2="21.2852" y2="-27.1526" width="0.1524" layer="20"/>
+<wire x1="21.2852" y1="-27.1526" x2="21.5646" y2="-27.432" width="0.1524" layer="20" curve="-90"/>
+<wire x1="21.5646" y1="-27.432" x2="21.5646" y2="-28.1686" width="0.1524" layer="20"/>
+<wire x1="21.5646" y1="-28.1686" x2="21.2852" y2="-28.448" width="0.1524" layer="20" curve="-90"/>
+<wire x1="21.2852" y1="-28.448" x2="21.1074" y2="-28.448" width="0.1524" layer="20"/>
+<wire x1="21.1074" y1="-28.448" x2="20.828" y2="-28.1686" width="0.1524" layer="20" curve="-90"/>
+<wire x1="21.6408" y1="-25.019" x2="21.6408" y2="-24.7396" width="0.1524" layer="20"/>
+<wire x1="21.6408" y1="-24.7396" x2="21.8694" y2="-24.511" width="0.1524" layer="20" curve="-90"/>
+<wire x1="21.8694" y1="-24.511" x2="22.4282" y2="-24.511" width="0.1524" layer="20"/>
+<wire x1="22.4282" y1="-24.511" x2="22.6568" y2="-24.7396" width="0.1524" layer="20" curve="-90"/>
+<wire x1="22.6568" y1="-24.7396" x2="22.6568" y2="-25.0444" width="0.1524" layer="20"/>
+<wire x1="22.6568" y1="-25.0444" x2="22.4282" y2="-25.273" width="0.1524" layer="20" curve="-90"/>
+<wire x1="22.4282" y1="-25.273" x2="21.8948" y2="-25.273" width="0.1524" layer="20"/>
+<wire x1="21.8948" y1="-25.273" x2="21.6408" y2="-25.019" width="0.1524" layer="20" curve="-90"/>
+<wire x1="26.6446" y1="-25.019" x2="26.6446" y2="-24.7396" width="0.1524" layer="20"/>
+<wire x1="26.6446" y1="-24.7396" x2="26.8732" y2="-24.511" width="0.1524" layer="20" curve="-90"/>
+<wire x1="26.8732" y1="-24.511" x2="27.432" y2="-24.511" width="0.1524" layer="20"/>
+<wire x1="27.432" y1="-24.511" x2="27.6606" y2="-24.7396" width="0.1524" layer="20" curve="-90"/>
+<wire x1="27.6606" y1="-24.7396" x2="27.6606" y2="-25.0444" width="0.1524" layer="20"/>
+<wire x1="27.6606" y1="-25.0444" x2="27.432" y2="-25.273" width="0.1524" layer="20" curve="-90"/>
+<wire x1="27.432" y1="-25.273" x2="26.8986" y2="-25.273" width="0.1524" layer="20"/>
+<wire x1="26.8986" y1="-25.273" x2="26.6446" y2="-25.019" width="0.1524" layer="20" curve="-90"/>
+<wire x1="27.7114" y1="-28.1432" x2="27.7114" y2="-27.3558" width="0.1524" layer="20"/>
+<wire x1="27.7114" y1="-27.3558" x2="27.94" y2="-27.1272" width="0.1524" layer="20" curve="-90"/>
+<wire x1="27.94" y1="-27.1272" x2="28.1686" y2="-27.1272" width="0.1524" layer="20"/>
+<wire x1="28.1686" y1="-27.1272" x2="28.448" y2="-27.4066" width="0.1524" layer="20" curve="-90"/>
+<wire x1="28.448" y1="-27.4066" x2="28.448" y2="-28.1432" width="0.1524" layer="20"/>
+<wire x1="28.448" y1="-28.1432" x2="28.1686" y2="-28.4226" width="0.1524" layer="20" curve="-90"/>
+<wire x1="28.1686" y1="-28.4226" x2="27.9908" y2="-28.4226" width="0.1524" layer="20"/>
+<wire x1="27.9908" y1="-28.4226" x2="27.7114" y2="-28.1432" width="0.1524" layer="20" curve="-90"/>
 </plain>
 <attributes>
