File: CAD/BT832_OLD/BT832_CP2102_24Pin/BT832A.sch (EAGLE design)
At the start: 44 parts, among them IC1 CP2102, U1 MCP73831T-3ACI/OT, U2 BT832, U3 LP5907MFX-3.3/NOPB, U4 LP5907MFX-3.3/NOPB, U5 ADS131M08IPBS, U6 BCM857BS, X1 ABM3B-8.000MHZ-B2-T, X2 FC-12M

Commit message: added missing voltage divider (doesn't fix the battery charger circuit)
Parts:
- added R7: 24kΩ, adafruit:R-US_R0402
- added R8: 47kΩ, adafruit:R-US_R0402
Connections:
- new net VBUS: IC1.VBUS, R7.2, R8.2
- net +5V: now also R7.1; no longer IC1.VBUS
- net GND: now also R8.1
Other:
- note added: "Page 20 (oops) https://www.silabs.com/documents/public/data-sheets/CP2102-9.pdf"
Changed lines of the file:
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@@
 <part name="SUPPLY3" library="supply2" library_urn="urn:adsk.eagle:library:372" deviceset="GND" device=""/>
 <part name="P+2" library="supply1" library_urn="urn:adsk.eagle:library:371" deviceset="+5V" device=""/>
-<part name="P+3" library="supply1" library_urn="urn:adsk.eagle:library:371" deviceset="+5V" device=""/>
 <part name="C12" library="adafruit" deviceset="C-US" device="C0402" value="1uF"/>
 <part name="C13" library="adafruit" deviceset="C-US" device="C0402" value="1uF"/>
@@
 <part name="C17" library="adafruit" library_urn="urn:adsk.eagle:library:420" deviceset="C-US" device="C0402" package3d_urn="urn:adsk.eagle:package:6240340/1" value="4.7uF"/>
 <part name="SUPPLY15" library="supply2" library_urn="urn:adsk.eagle:library:372" deviceset="GND" device=""/>
+<part name="R7" library="adafruit" library_urn="urn:adsk.eagle:library:420" deviceset="R-US_" device="R0402" package3d_urn="urn:adsk.eagle:package:6240564/1" value="24kΩ"/>
+<part name="R8" library="adafruit" library_urn="urn:adsk.eagle:library:420" deviceset="R-US_" device="R0402" package3d_urn="urn:adsk.eagle:package:6240564/1" value="47kΩ"/>
+<part name="SUPPLY16" library="supply2" library_urn="urn:adsk.eagle:library:372" deviceset="GND" device=""/>
 </parts>
 <sheets>
@@
 Battery/Power Management
 Power Switches</text>
+<text x="178.308" y="38.354" size="1.6764" layer="97">Page 20 (oops)
+https://www.silabs.com/documents/public/data-sheets/CP2102-9.pdf</text>
 </plain>
 <instances>
@@
 <attribute name="VALUE" x="145.542" y="80.01" size="1.778" layer="96" rot="R180"/>
 </instance>
-<instance part="P+3" gate="1" x="163.322" y="80.01" smashed="yes" rot="R90">
-<attribute name="VALUE" x="168.402" y="78.74" size="1.778" layer="96" rot="R180"/>
-</instance>
 <instance part="C12" gate="G$1" x="100.076" y="115.57" smashed="yes" rot="R180">
 <attribute name="NAME" x="99.06" y="114.935" size="1.778" layer="95" rot="R180"/>
@@
 </instance>
 <instance part="SUPPLY15" gate="GND" x="80.01" y="35.306" smashed="yes"/>
+<instance part="R7" gate="G$1" x="189.484" y="25.4" smashed="yes" rot="R90">
+<attribute name="NAME" x="187.2234" y="23.622" size="1.778" layer="95" rot="R90"/>
+<attribute name="VALUE" x="192.786" y="21.59" size="1.778" layer="96" rot="R90"/>
+</instance>
+<instance part="R8" gate="G$1" x="180.594" y="25.146" smashed="yes" rot="R90">
+<attribute name="NAME" x="178.3334" y="23.368" size="1.778" layer="95" rot="R90"/>
+<attribute name="VALUE" x="183.896" y="21.336" size="1.778" layer="96" rot="R90"/>
+</instance>
+<instance part="SUPPLY16" gate="GND" x="180.594" y="15.494" smashed="yes">
+<attribute name="VALUE" x="178.689" y="12.319" size="1.778" layer="96"/>
+</instance>
 </instances>
 <busses>
@@
 <wire x1="75.184" y1="39.878" x2="80.01" y2="39.878" width="0.1524" layer="91"/>
 </segment>
+<segment>
+<pinref part="R8" gate="G$1" pin="1"/>
+<wire x1="180.594" y1="20.066" x2="180.594" y2="18.034" width="0.1524" layer="91"/>
+<label x="181.102" y="17.018" size="1.778" layer="95"/>
+<pinref part="SUPPLY16" gate="GND" pin="GND"/>
+</segment>
 </net>
 <net name="XTAL2_2" class="0">
@@
 </segment>
 <segment>
-<pinref part="IC1" gate="G$1" pin="VBUS"/>
-<wire x1="170.942" y1="80.01" x2="165.862" y2="80.01" width="0.1524" layer="91"/>
-<pinref part="P+3" gate="1" pin="+5V"/>
-</segment>
-<segment>
 <pinref part="D2" gate="G$1" pin="AA"/>
 <wire x1="62.23" y1="29.718" x2="62.23" y2="25.654" width="0.1524" layer="91"/>
@@
 <wire x1="49.022" y1="59.944" x2="49.022" y2="63.246" width="0.1524" layer="91"/>
 <pinref part="P+5" gate="1" pin="+5V"/>
+</segment>
+<segment>
+<pinref part="R7" gate="G$1" pin="1"/>
+<wire x1="189.484" y1="20.32" x2="189.484" y2="17.78" width="0.1524" layer="91"/>
+<label x="190.5" y="17.526" size="1.778" layer="95"/>
 </segment>
 </net>
@@
 </segment>
 </net>
+<net name="VBUS" class="0">
+<segment>
+<pinref part="R7" gate="G$1" pin="2"/>
+<wire x1="189.484" y1="30.48" x2="189.484" y2="33.274" width="0.1524" layer="91"/>
+<label x="189.484" y="35.306" size="1.778" layer="95"/>
+</segment>
+<segment>
+<pinref part="R8" gate="G$1" pin="2"/>
+<wire x1="180.594" y1="30.226" x2="180.594" y2="33.02" width="0.1524" layer="91"/>
+<label x="179.578" y="35.052" size="1.778" layer="95"/>
+</segment>
+<segment>
+<pinref part="IC1" gate="G$1" pin="VBUS"/>
+<wire x1="170.942" y1="80.01" x2="165.862" y2="80.01" width="0.1524" layer="91"/>
+<label x="165.1" y="77.216" size="1.778" layer="95"/>
+</segment>
+</net>
