File: CAD/BC40M/BC40M_nrf53.brd (EAGLE design)
At the start: 25.5 x 40 mm, 92 parts, among them J1 SM02B-SRSS-TB(LF)(SN), U1 TPD4S012DRYR, U2 BC840M, U3 LP5907MFX-3.3/NOPB, U4 LP5907MFX-3.3/NOPB, U5 ADS131M08IPBS, U6 BQ24072RGTR, U7 DX4R005JJ2R1800, X1 ABM3B-8.000MHZ-B2-T, X2 FC-12M, X3 1365-20

Commit message: added revisions and alt configurations
Parts:
- removed C30: 0.1uF, standardparts:0201
- removed C31: 10uF, standardparts:0402
- removed CS, DIN, DOUT, DRDY, SCLK, SYNC: TPTP07R, testpad:TP07R
- removed JP1: (no value), pinhead+:2X08_SMT
- removed JP2, JP3: (no value), pinhead+:2X10_SMT
- removed LED3: (no value), adafruit:CHIPLED_0603
- removed R10, R11, R12, R13, R14, R15, R16, R17, R18, R19, R20, R21, R6, R7, R8, R9: 1MOhm, standardparts:0603
- removed SJ1, SJ2: (no value), jumper:SJ
- removed U$1: BC40M, BC40M-V0-lib2:BC40M
- removed U7: DX4R005JJ2R1800, DX4R005JJ2R1800:DX4R005JJ2R1800
- removed X2: FC-12M, crystal:FC-12M
- removed X3: 1365-20, con-leotronics:1365-20
- added HDR1, HDR2: 1365-20, con-leotronics:1365-20
- added MCU: BC40M, BC40M-V0-lib2:BC40M
- added X5: 1365-16, con-leotronics:1365-16
- C1, C2: value 12.5pF -> 10pF
- C12: value 1uF -> 4.7uF
- C13: value 1uF -> 100pF
- C14: value 4.7uF -> 100pF
- C15: value 10uF -> 100pF; device standardparts:0402 -> standardparts:0201
- C16, C17, C20: device standardparts:0603 -> standardparts:0201
- C18: value 0.1uF -> 100pF
- C19: value 10nF -> 100pF
- C21, C28: value 100pF -> 0.1uF; device standardparts:0603 -> standardparts:0201
- C22: value 0.1uF -> 10nF
- C23: value 1uF -> 0.1uF
- C24: value 100pF -> 1uF; device standardparts:0603 -> standardparts:0201
- C25: value 100pF -> 4.7uF; device standardparts:0603 -> standardparts:0201
- C29: value 100pF -> 10uF; device standardparts:0603 -> standardparts:0402
- C3: value 10pF -> 1uF
- C4: value 10pF -> 220nF
- C6: value 220nF -> 1uF
- C9: value 4.7uF -> 10uF; device standardparts:0201 -> standardparts:0402
- LED1: value (none) -> GM5WA94310A; device adafruit:CHIPLED_0603 -> led:GM5WA94310A
- R1: value 10kΩ -> 3.3kΩ
- R2: value 100kΩ -> 3.3kΩ
- R22: value 0Ω -> 348kΩ; device standardparts:0805 -> standardparts:0201
- R23: value 348kΩ -> 750kΩ; device standardparts:0603 -> standardparts:0201
- R24: value 750kΩ -> 100kΩ; device standardparts:0603 -> standardparts:0201
- R27: value 3.3kΩ -> 10kΩ
- R3: value 1.18kΩ -> 3.3kΩ; device standardparts:0603 -> standardparts:0201
- R4: value 1.13kΩ -> 1.18kΩ; device standardparts:0603 -> standardparts:0201
- R5: value 3.3kΩ -> 1.13kΩ
- U1: value TPD4S012DRYR -> LP5907MFX-3.3/NOPB; device TPD4S012DRYR:PSON50P145X100X60-6N -> LP5907MFX-3.3_NOPB:SOT95P280X145-5N
- U2: value BC840M -> DX4R005JJ2R1800; device BC840M:BC840M -> DX4R005JJ2R1800:DX4R005JJ2R1800
- U4: value LP5907MFX-3.3/NOPB -> ADS131M08IPBS; device LP5907MFX-3.3_NOPB:SOT95P280X145-5N -> ADS131M08IPBS:QFP50P700X700X120-32N
- U5: value ADS131M08IPBS -> BQ24072RGTR; device ADS131M08IPBS:QFP50P700X700X120-32N -> BQ24072RGTR:QFN50P300X300X100-17N
- U6: value BQ24072RGTR -> TPD4S012DRYR; device BQ24072RGTR:QFN50P300X300X100-17N -> TPD4S012DRYR:PSON50P145X100X60-6N
- moved LED1 36.2 mm to (32.3, 67.4), turned to 90 degrees
- moved R3 32.7 mm to (35.2, 66.8), turned to 90 degrees
- moved R1 31.4 mm to (34.9, 65.7), turned to 180 degrees
- moved R27 25.6 mm to (27.6, 43.0), turned to 270 degrees
- moved J1 20.6 mm to (15.6, 44.3), turned to 270 degrees
- moved C19 20.5 mm to (23.4, 56.0), flipped to the bottom, turned to 270 degrees
- moved C29 19.6 mm to (31.3, 42.9), flipped to the top, turned to 90 degrees
- moved C27 19.4 mm to (26.8, 56.1), turned to 0 degrees
- moved C26 19.3 mm to (26.7, 55.4), turned to 0 degrees
- moved U2 18.5 mm to (20.3, 40.0), turned to 90 degrees
- moved C9 18.3 mm to (29.5, 48.6), turned to 90 degrees
- moved R26 18.1 mm to (15.6, 65.4)
- moved LED2 18.1 mm to (14.5, 65.9), turned to 180 degrees
- moved C18 17.9 mm to (23.3, 53.9), flipped to the bottom, turned to 270 degrees
- moved R2 17.7 mm to (36.5, 66.5), turned to 90 degrees
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Connections:
- net LED2 renamed LED5
- removed net 0NIN: C16.2, R8.2, U5.30
- removed net 0PIN: C16.1, R6.2, U5.29
- removed net 1NIN: C17.2, R9.2, U5.31
- removed net 1PIN: C17.1, R7.2, U5.32
- removed net 2NIN: C20.2, R12.2, U5.2
- removed net 2PIN: C20.1, R10.2, U5.1
- removed net 3NIN: C21.2, R13.2, U5.3
- removed net 3PIN: C21.1, R11.2, U5.4
- removed net 4NIN: C24.2, R16.2, U5.6
- removed net 4PIN: C24.1, R14.2, U5.5
- removed net 5NIN: C25.2, R17.2, U5.7
- removed net 5PIN: C25.1, R15.2, U5.8
- removed net 6NIN: C28.2, R20.2, U5.10
- removed net 6PIN: C28.1, R18.2, U5.9
- removed net 7NIN: C29.2, R21.2, U5.11
- removed net 7PIN: C29.1, R19.2, U5.12
- removed net AVDD1: SJ2.1, U4.5
- removed net DCCH: U2.A6
- removed net LED1: LED1.A, R5.2
- removed net LED3: LED3.A, R27.2
- removed net P101: JP2.8, U2.A0
- removed net P107: JP2.14, U2.C0
- removed net P108: JP2.13, U2.C5
- removed net P11: JP2.7, U2.D5
- removed net P2: JP3.14, U2.F4
- removed net P23: JP3.13, U2.F0
- removed net P25: JP2.4, U2.A1
- removed net P26: R5.1, U2.E6
- removed net P28: JP3.2, U2.H1
- removed net P3: JP3.9, U2.H0
- removed net P31: JP3.12, U2.E5
- removed net P5: JP3.10, U2.G7
- removed net P7: JP2.11, U2.B6
- removed net P8: JP2.5, U2.C7
- removed net SWO: JP2.20, U2.D0
- removed net XTAL1_1: C2.2, U2.F6, X2.2
- removed net XTAL2_1: C1.2, U2.F7, X2.1
- new net N$1: LED1.2, R3.2
- new net N$2: LED1.3, R2.2
- new net N$3: LED1.1, R1.2
- new net P102: HDR1.16, MCU.C5
- new net P103: HDR1.5, MCU.E6
- new net P105: HDR1.12, MCU.A6
- new net P10_MISO: HDR2.1, MCU.G7
- new net P115: HDR2.19, MCU.H4
- new net P13: HDR1.10, MCU.A5
- new net P18: HDR1.11, MCU.B3
- new net P25_AIN4: HDR2.6, MCU.B0
- new net P26_AIN5: HDR1.1, MCU.C1
- new net P27_AIN6: HDR2.8, MCU.C0
- new net P28_AIN7: HDR2.4, MCU.F1
- new net P4_AIN0: HDR1.17, MCU.D5
- new net P5_AIN1: HDR1.15, MCU.D4
- new net P6_AIN2: HDR1.19, MCU.D7
- new net P7_AIN3: HDR1.20, MCU.B6
- new net P9_MOSI: HDR2.2, MCU.C4
- net +5V: now also C22.2, C25.2, C28.2, C29.2, U2.1, U6.6; no longer C19.2, C30.2, C31.2, C9.2, U1.6, U7.1
- net +5V_ISO: now also C21.1, MCU.F5, U5.13; no longer C18.1, U2.B5, U6.13
- net 0N: now also C13.2, U4.30, X5.2; no longer JP1.2, R8.1
- net 0P: now also C13.1, U4.29, X5.1; no longer JP1.1, R6.1
- net 1N: now also C14.2, U4.31, X5.4; no longer JP1.4, R9.1
- net 1P: now also C14.1, U4.32, X5.3; no longer JP1.3, R7.1
- net 2N: now also C15.2, U4.2, X5.6; no longer JP1.6, R12.1
- net 2P: now also C15.1, U4.1, X5.5; no longer JP1.5, R10.1
- net 3N: now also C16.2, U4.3, X5.8; no longer JP1.8, R13.1
- net 3P: now also C16.1, U4.4, X5.7; no longer JP1.7, R11.1
- net 4N: now also C17.2, U4.6, X5.10; no longer JP1.10, R16.1
- net 4P: now also C17.1, U4.5, X5.9; no longer JP1.9, R14.1
- net 5N: now also C18.2, U4.7, X5.12; no longer JP1.12, R17.1
- net 5P: now also C18.1, U4.8, X5.11; no longer JP1.11, R15.1
- net 6N: now also C19.2, U4.10, X5.14; no longer JP1.14, R20.1
- net 6P: now also C19.1, U4.9, X5.13; no longer JP1.13, R18.1
- net 7N: now also C20.2, U4.11, X5.16; no longer JP1.16, R21.1
- net 7P: now also C20.1, U4.12, X5.15; no longer JP1.15, R19.1
- net AVDD: now also C3.2, C6.1, U3.5, U4.15; no longer C5.2, C8.1, SJ1.2, SJ2.2, U5.15
- net BAT: now also C12.2, R22.1, U5.2, U5.3; no longer C14.2, R23.1, U6.2, U6.3
- net CAP: now also C4.1, U4.24; no longer C6.1, U5.24
- net CHG: now also MCU.C7, U5.9; no longer U2.D6, U6.9
- net CLKIN: now also C1.1, U4.23; no longer C3.1, U5.23
- net CLKOUT: now also C2.1, HDR2.20, U4.22; no longer C4.1, JP3.1, U5.22
- net CS: now also MCU.E4, U4.17; no longer CS.TP, U2.E3, U5.17
- net CUR_DETECT: now also MCU.E7, R22.2, R23.1; no longer R23.2, R24.1, U2.E7
- net D+: now also MCU.H5, U2.3, U6.1; no longer U1.1, U2.A4, U7.3
- net D-: now also MCU.G5, U2.2, U6.2; no longer U1.2, U2.A5, U7.2
- net DIN: now also HDR2.17, MCU.F2, U4.21; no longer DIN.TP, JP3.19, U2.E0, U5.21
- net DOUT: now also HDR2.15, MCU.F3, U4.20; no longer DOUT.TP, JP3.17, U2.F2, U5.20
- net DRDY: now also MCU.E3, U4.18; no longer DRDY.TP, U2.D1, U5.18
- net GND: now also C1.2, C2.2, C21.2, C24.1, C25.1, C28.1, C29.1, C3.1, C5.2, C7.1, C8.1, HDR2.16, LED1.4, LED1.5, LED1.6, MCU.D3, MCU.E0, MCU.F0, MCU.F4, MCU.G0, MCU.H0, MCU.H1, MCU.H7, R23.2, R27.1, R5.1, U1.2, U2.5, U2.MP1, U2.MP2, U4.13, U4.25, U4.28, U5.15, U5.4, U5.6, U5.8; no longer C1.1, C13.1, C14.1, C15.1, C18.2, C19.1, C2.1, C3.2, C30.1, C31.1, C5.1, C7.2, C8.2, JP3.5, LED1.C, LED3.C, R1.1, R22.1, R22.2, R24.2, R3.1, R30.2, U1.4, U2.G0, U2.G4, U2.G5, U2.G6, U2.H4, U2.H5, U2.H6, U2.H7, U4.2, U5.13, U5.25, U5.28, U6.15, U6.6, U6.8, U7.5, U7.MP1, U7.MP2
- net ID: now also U2.4; no longer U7.4
- net ILM: now also R4.2, U5.12; no longer R3.2, U6.12
- net ISET: now also R5.2, U5.16; no longer R4.2, U6.16
- net NFC1: now also MCU.F7; no longer U2.D2
- net NFC2: now also MCU.C6; no longer U2.E2
- net P104: now also HDR1.2, MCU.A1; no longer JP2.10, U2.B0
- net P106: now also HDR1.14, MCU.A7; no longer JP3.11, U2.E1
- net P109: now also MCU.A0, R26.1; no longer JP2.15, U2.C6
- net P110: now also HDR2.9, MCU.G2; no longer JP3.18, U2.H2
- net P111: now also HDR2.3, MCU.H2; no longer JP3.4, U2.G2
- net P113: now also HDR2.5, MCU.G3; no longer JP3.6, U2.G3
- net P114: now also HDR2.7, MCU.H3; no longer JP3.8, U2.H3
- net P12: now also HDR1.18, MCU.B7; no longer JP2.9, U2.B7
- net P14: now also HDR1.13, MCU.B4; no longer JP2.1, U2.C4
- net P15: now also HDR1.8, MCU.A4; no longer JP2.2, U2.B3
- net P16: now also HDR1.3, MCU.B5; no longer R26.1, U2.D3
- net P17: now also HDR1.6, MCU.A3; no longer JP2.3, U2.A3
- net P19: now also MCU.C3, R3.1; no longer JP2.19, U2.A2
- net P20: now also HDR1.4, MCU.A2; no longer R27.1, U2.C2
- net P21: now also MCU.C2, R1.1; no longer JP2.12, U2.C3
- net P22: now also HDR1.9, MCU.B2; no longer JP2.6, U2.B2
- net P24: now also HDR1.7, MCU.B1; no longer JP3.20, U2.F1
- net P29: now also MCU.E1, R2.1; no longer JP3.16, U2.E4
- net P30: now also HDR2.11, MCU.G1; no longer JP3.7, U2.G1
- net PGOOD: now also MCU.D6, U5.7; no longer U2.D7, U6.7
- net RESET: now also HDR2.14, MCU.D2, R24.1; no longer JP2.17, R2.1, U2.B4
- net SCLK: now also HDR2.13, MCU.E2, U4.19; no longer JP3.15, SCLK.TP, U2.F3, U5.19
- net SWDCLK: now also HDR2.10, MCU.D1; no longer JP2.18, U2.C1
- net SWDIO: now also HDR2.12, MCU.D0; no longer JP2.16, U2.B1
- net SYNC/RESET: now also MCU.E5, U4.16; no longer SYNC.TP, U2.D4, U5.16
- net TMR: now also U5.14; no longer U6.14
- net TS: now also R27.2, U5.1; no longer R1.2, U6.1
- net VDD: now also C7.2, C9.2, HDR2.18, MCU.G4, R30.2, U1.5, U4.26; no longer C12.2, C15.2, C22.2, JP3.3, R31.2, SJ1.1, U2.F5, U3.5, U5.26
- net VDDH: now also MCU.F6, R24.2; no longer R2.2, U2.A7
- net VIN: now also C24.2, C5.1, C8.2, R31.2, U1.1, U1.3; no longer C13.2, C7.1, U4.1, U4.3
- net VSWITCH: now also U5.10, U5.11, U5.5; no longer U6.10, U6.11, U6.5
Routing:
- net +5V_ISO: track 68.2 -> 24.0 mm, vias 4 -> 2
- net GND: track 174.9 -> 217.7 mm, vias 30 -> 38
- net P26: track 31.2 -> 0.00 mm, vias 2 -> 0
- net P15: track 31.7 -> 3.20 mm
- net P28: track 28.5 -> 0.00 mm
- net P25: track 27.9 -> 0.00 mm
- net RESET: track 30.0 -> 55.3 mm
- net P111: track 27.7 -> 3.61 mm
- net P101: track 23.3 -> 0.00 mm
- net P17: track 26.1 -> 3.00 mm
- net P4_AIN0: track 0.00 -> 23.1 mm, vias 0 -> 2
- net P5_AIN1: track 0.00 -> 20.7 mm, vias 0 -> 2
- net P104: track 22.9 -> 2.63 mm
- net P27_AIN6: track 0.00 -> 19.7 mm
- net P25_AIN4: track 0.00 -> 19.5 mm
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Other:
- board size 25.5 x 40 mm -> 26.3 x 32.9 mm
- board text added: "0+"
- board text added: "0-"
- board text added: "10/MISO"
- board text added: "103"
- board text added: "115"
- board text added: "13"
- board text added: "14 | 106"
- board text added: "16"
- board text added: "18 | 105"
- board text added: "20"
- board text added: "26"
- board text added: "27"
- board text added: "3.3V"
- board text added: "4 | 12"
- board text added: "5 | 102"
- board text added: "6"
- board text added: "7+"
- board text added: "7-"
- board text added: "9/MOSI"
- board text added: "BC40M + ADS131M08 Joshua Brewster Bojan Jovanovich AGPL v3 License"
- board text added: "G"
- board text added: "MCU"
- board text added: "P10"
- board text added: "P102"
- board text added: "P103"
- board text added: "P104"
- board text added: "P105"
- board text added: "P106"
- board text added: "P110"
- board text added: "P111"
- board text added: "P113"
- board text added: "P114"
- board text added: "P115"
- board text added: "P12"
- board text added: "P13"
- board text added: "P14"
- board text added: "P15"
- board text added: "P16"
- board text added: "P17"
- board text added: "P18"
- board text added: "P20"
- board text added: "P22"
- board text added: "P24"
- board text added: "P25"
- board text added: "P26"
- board text added: "P27"
- board text added: "P28"
- board text added: "P30"
- board text added: "P4"
- board text added: "P5"
- board text added: "P6"
- board text added: "P7"
- board text added: "P9"
- board text added: "RST"
- board text added: "SWCLK"
- board text added: "V"
- board text removed: "101"
- board text removed: "106"
- board text removed: "107"
- board text removed: "108"
- board text removed: "109"
- board text removed: "11"
- board text removed: "12"
- board text removed: "14"
- board text removed: "19"
- board text removed: "2"
- board text removed: "21"
- board text removed: "23"
- board text removed: "29"
- board text removed: "3"
- board text removed: "31"
- board text removed: "5"
- board text removed: "8"
- board text removed: "8.192MHz"
- board text removed: "BC840M"
- board text removed: "BC840M + ADS131M08 JOSHUA BREWSTER JACOB TINKHAUSER BOJAN JOVANOVICH AGPL v3 LICENSE"
- board text removed: "R2"
- board text removed: "S1"
- board text removed: "SWD CLK"
- board text removed: "SWD IO"
- board text removed: "TOP"
