File: CAD/BC840M/BC840M.brd (EAGLE design)
At the start: 25.5 x 40 mm, 90 parts, among them J1 SM02B-SRSS-TB(LF)(SN), U1 TPD4S012DRYR, U2 BC840M, U3 LP5907MFX-3.3/NOPB, U4 LP5907MFX-3.3/NOPB, U5 ADS131M08IPBS, U6 BQ24072RGTR, U7 DX4R005JJ2R1800, X1 ABM3B-8.000MHZ-B2-T, X2 FC-12M

Commit message: added revisions and alt configurations
Parts:
- removed R10, R11, R12, R13, R14, R15, R16, R17, R18, R19, R20, R21, R6, R7, R8, R9: 1MOhm, standardparts:0603
- moved C29 2.40 mm to (22.2, 60.9)
- moved C24 0.52 mm to (24.3, 53.4)
- moved C28 0.52 mm to (24.2, 58.7)
- moved C25 0.50 mm to (24.3, 56.0)
- moved C17 0.31 mm to (24.7, 44.9)
- moved R28 0.05 mm to (22.6, 48.0)
Connections:
- removed net 0NIN: C16.2, R8.2, U5.30
- removed net 0PIN: C16.1, R6.2, U5.29
- removed net 1NIN: C17.2, R9.2, U5.31
- removed net 1PIN: C17.1, R7.2, U5.32
- removed net 2NIN: C20.2, R12.2, U5.2
- removed net 2PIN: C20.1, R10.2, U5.1
- removed net 3NIN: C21.2, R13.2, U5.3
- removed net 3PIN: C21.1, R11.2, U5.4
- removed net 4NIN: C24.2, R16.2, U5.6
- removed net 4PIN: C24.1, R14.2, U5.5
- removed net 5NIN: C25.2, R17.2, U5.7
- removed net 5PIN: C25.1, R15.2, U5.8
- removed net 6NIN: C28.2, R20.2, U5.10
- removed net 6PIN: C28.1, R18.2, U5.9
- removed net 7NIN: C29.2, R21.2, U5.11
- removed net 7PIN: C29.1, R19.2, U5.12
- net 0N: now also C16.2, U5.30; no longer R8.1
- net 0P: now also C16.1, U5.29; no longer R6.1
- net 1N: now also C17.2, U5.31; no longer R9.1
- net 1P: now also C17.1, U5.32; no longer R7.1
- net 2N: now also C20.2, U5.2; no longer R12.1
- net 2P: now also C20.1, U5.1; no longer R10.1
- net 3N: now also C21.2, U5.3; no longer R13.1
- net 3P: now also C21.1, U5.4; no longer R11.1
- net 4N: now also C24.2, U5.6; no longer R16.1
- net 4P: now also C24.1, U5.5; no longer R14.1
- net 5N: now also C25.2, U5.7; no longer R17.1
- net 5P: now also C25.1, U5.8; no longer R15.1
- net 6N: now also C28.2, U5.10; no longer R20.1
- net 6P: now also C28.1, U5.9; no longer R18.1
- net 7N: now also C29.2, U5.11; no longer R21.1
- net 7P: now also C29.1, U5.12; no longer R19.1
Routing:
- net 0P: track 8.69 -> 22.7 mm
- net 7N: track 1.95 -> 15.0 mm
- net 0PIN: track 12.9 -> 0.00 mm
- net 7P: track 8.40 -> 21.3 mm
- net 7PIN: track 12.7 -> 0.00 mm
- net 0N: track 1.92 -> 14.3 mm
- net 7NIN: track 11.2 -> 0.00 mm
- net 6N: track 2.51 -> 13.3 mm
- net 0NIN: track 10.7 -> 0.00 mm
- net 1N: track 2.39 -> 12.8 mm
- net 6NIN: track 9.84 -> 0.00 mm
- net 1NIN: track 9.09 -> 0.00 mm
- net 6P: track 8.78 -> 17.8 mm
- net 1P: track 8.72 -> 17.3 mm
- net 6PIN: track 8.31 -> 0.00 mm
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