File: CAD/BC840M/BC840M.sch (EAGLE design)
At the start: 90 parts, among them J1 SM02B-SRSS-TB(LF)(SN), U1 TPD4S012DRYR, U2 BC840M, U3 LP5907MFX-3.3/NOPB, U4 LP5907MFX-3.3/NOPB, U5 ADS131M08IPBS, U6 BQ24072RGTR, U7 DX4R005JJ2R1800, X1 ABM3B-8.000MHZ-B2-T, X2 FC-12M

Commit message: design corrections
Connections:
- net GND: no longer U5.REFIN
Changed lines of the file:
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@@
-</segment>
-<segment>
-<pinref part="U5" gate="G$1" pin="REFIN"/>
-<wire x1="393.319" y1="111.4298" x2="395.859" y2="111.4298" width="0.1524" layer="91"/>
-<label x="396.621" y="111.1758" size="1.778" layer="95"/>
 </segment>
 <segment>

Commit message: added revisions and alt configurations
Parts:
- removed R10, R11, R12, R13, R14, R15, R16, R17, R18, R19, R20, R21, R6, R7, R8, R9: 1MOhm, standardparts:RESISTOR.0603
Connections:
- removed net 0NIN: C16.2, R8.2, U5.AN0N
- removed net 0PIN: C16.1, R6.2, U5.AN0P
- removed net 1NIN: C17.2, R9.2, U5.AN1N
- removed net 1PIN: C17.1, R7.2, U5.AN1P
- removed net 2NIN: C20.2, R12.2, U5.AIN2N
- removed net 2PIN: C20.1, R10.2, U5.AIN2P
- removed net 3NIN: C21.2, R13.2, U5.AIN3N
- removed net 3PIN: C21.1, R11.2, U5.AIN3P
- removed net 4NIN: C24.2, R16.2, U5.AIN4N
- removed net 4PIN: C24.1, R14.2, U5.AIN4P
- removed net 5NIN: C25.2, R17.2, U5.AIN5N
- removed net 5PIN: C25.1, R15.2, U5.AIN5P
- removed net 6NIN: C28.2, R20.2, U5.AIN6N
- removed net 6PIN: C28.1, R18.2, U5.AIN6P
- removed net 7NIN: C29.2, R21.2, U5.AIN7N
- removed net 7PIN: C29.1, R19.2, U5.AIN7P
- net 0N: now also C16.2, U5.AN0N; no longer R8.1
- net 0P: now also C16.1, U5.AN0P; no longer R6.1
- net 1N: now also C17.2, U5.AN1N; no longer R9.1
- net 1P: now also C17.1, U5.AN1P; no longer R7.1
- net 2N: now also C20.2, U5.AIN2N; no longer R12.1
- net 2P: now also C20.1, U5.AIN2P; no longer R10.1
- net 3N: now also C21.2, U5.AIN3N; no longer R13.1
- net 3P: now also C21.1, U5.AIN3P; no longer R11.1
- net 4N: now also C24.2, U5.AIN4N; no longer R16.1
- net 4P: now also C24.1, U5.AIN4P; no longer R14.1
- net 5N: now also C25.2, U5.AIN5N; no longer R17.1
- net 5P: now also C25.1, U5.AIN5P; no longer R15.1
- net 6N: now also C28.2, U5.AIN6N; no longer R20.1
- net 6P: now also C28.1, U5.AIN6P; no longer R18.1
- net 7N: now also C29.2, U5.AIN7N; no longer R21.1
- net 7P: now also C29.1, U5.AIN7P; no longer R19.1
