File: CAD/BC840M/BC840M_1.25mm_headers.sch (EAGLE design)
At the start: 62 parts, among them J1 SM02B-SRSS-TB(LF)(SN), U1 LP5907MFX-3.3/NOPB, U2 DX4R005JJ2R1800, U3 LP5907MFX-3.3/NOPB, U4 ADS131M08IPBS, U5 BQ24072RGTR, U6 TPD4S012DRYR, X1 ABM3B-8.000MHZ-B2-T, X5 1365-16

Commit message: added revisions and alt configurations
Parts:
- removed HDR1, HDR2: 1365-20, con-leotronics:1365-20
- removed MCU: BC40M, BC40M-V0-lib2:BC40M
- removed R22: 348kΩ, standardparts:RESISTOR.0201
- removed R23: 750kΩ, standardparts:RESISTOR.0201
- removed R24: 100kΩ, standardparts:RESISTOR.0201
- removed R25: 0Ω, standardparts:RESISTOR.0805
- removed R26: 3.3kΩ, standardparts:RESISTOR.0201
- removed R27: 10kΩ, standardparts:RESISTOR.0201
- removed R28, R29: 10kΩ, standardparts:RESISTOR.0402
- removed R30, R31: 100kΩ, standardparts:RESISTOR.0402
- added C30: 0.1uF, standardparts:CAPACITOR.0201
- added C31: 10uF, standardparts:CAPACITOR.0402
- added CS, DIN, DOUT, DRDY, SCLK, SYNC: TPTP07R, testpad:TPTP07R
- added LED3: (no value), adafruit:LEDCHIPLED_0603
- added R10, R11: 3.3kΩ, standardparts:RESISTOR.0201
- added R12, R13: 10kΩ, standardparts:RESISTOR.0402
- added R14, R15: 100kΩ, standardparts:RESISTOR.0402
- added R6, R9: 0Ω, standardparts:RESISTOR.0805
- added R7: 348kΩ, standardparts:RESISTOR.0201
- added R8: 750kΩ, standardparts:RESISTOR.0201
- added U7: DX4R005JJ2R1800, DX4R005JJ2R1800:DX4R005JJ2R1800
- added X2: FC-12M, crystal:FC-12M
- added X3, X4: 1365-20, con-leotronics:1365-20
- C1, C2: value 10pF -> 12.5pF
- C12: value 4.7uF -> 1uF
- C13: value 100pF -> 1uF
- C14: value 100pF -> 4.7uF
- C15: value 100pF -> 10uF; device standardparts:CAPACITOR.0201 -> standardparts:CAPACITOR.0402
- C18: value 100pF -> 0.1uF
- C19: value 100pF -> 10nF
- C21, C28: value 0.1uF -> 100pF
- C22: value 10nF -> 0.1uF
- C23: value 0.1uF -> 1uF
- C24: value 1uF -> 100pF
- C25: value 4.7uF -> 100pF
- C29: value 10uF -> 100pF; device standardparts:CAPACITOR.0402 -> standardparts:CAPACITOR.0201
- C3: value 1uF -> 10pF
- C4: value 220nF -> 10pF
- C6: value 1uF -> 220nF
- C9: value 10uF -> 4.7uF; device standardparts:CAPACITOR.0402 -> standardparts:CAPACITOR.0201
- LED1: value GM5WA94310A -> (none); device led:GM5WA94310A -> adafruit:LEDCHIPLED_0603
- R1: value 3.3kΩ -> 10kΩ
- R2: value 3.3kΩ -> 100kΩ
- R3: value 3.3kΩ -> 1.18kΩ; SPICEPREFIX (none) -> R
- R4: value 1.18kΩ -> 1.13kΩ; SPICEPREFIX R -> (none)
- R5: value 1.13kΩ -> 3.3kΩ
- U1: value LP5907MFX-3.3/NOPB -> TPD4S012DRYR; device LP5907MFX-3.3_NOPB:LP5907MFX-3.3/NOPB -> TPD4S012DRYR:TPD4S012DRYR
- U2: value DX4R005JJ2R1800 -> BC840M; device DX4R005JJ2R1800:DX4R005JJ2R1800 -> BC840M:BC840M
- U4: value ADS131M08IPBS -> LP5907MFX-3.3/NOPB; device ADS131M08IPBS:ADS131M08IPBS -> LP5907MFX-3.3_NOPB:LP5907MFX-3.3/NOPB
- U5: value BQ24072RGTR -> ADS131M08IPBS; device BQ24072RGTR:BQ24072RGTR -> ADS131M08IPBS:ADS131M08IPBS
- U6: value TPD4S012DRYR -> BQ24072RGTR; device TPD4S012DRYR:TPD4S012DRYR -> BQ24072RGTR:BQ24072RGTR
Connections:
- removed net LED5: LED2.A, R26.2
- removed net N$1: LED1R.A, R3.2
- removed net N$2: LED1G.A, R2.2
- removed net N$3: LED1B.A, R1.2
- removed net P102: HDR1-16.S, MCU.C5/P102/I2C
- removed net P103: HDR1-5.S, MCU.E6/P103/I2C
- removed net P105: HDR1-12.S, MCU.A6/P105
- removed net P10_MISO: HDR2-1.S, MCU.G7/P010/MISO
- removed net P115: HDR2-19.S, MCU.H4/P115
- removed net P13: HDR1-10.S, MCU.A5/013/QSPI0
- removed net P18: HDR1-11.S, MCU.B3/P018/QSPI_CS
- removed net P25_AIN4: HDR2-6.S, MCU.B0/P025/AIN4
- removed net P26_AIN5: HDR1-1.S, MCU.C1/P026/AIN5
- removed net P27_AIN6: HDR2-8.S, MCU.C0/P027/AIN6
- removed net P28_AIN7: HDR2-4.S, MCU.F1/P028/AIN7
- removed net P4_AIN0: HDR1-17.S, MCU.D5/P004/AIN0
- removed net P5_AIN1: HDR1-15.S, MCU.D4/P005/AIN1
- removed net P6_AIN2: HDR1-19.S, MCU.D7/P006/AIN2
- removed net P7_AIN3: HDR1-20.S, MCU.B6/P007/AIN3
- removed net P9_MOSI: HDR2-2.S, MCU.C4/P9/MOSI
- new net DCCH: U2.A6/DCCH
- new net LED1: LED1.A, R5.2
- new net LED2: LED2.A, R10.2
- new net LED3: LED3.A, R11.2
- new net P101: U2.A0/P101, X3-13.S
- new net P107: U2.C0/P107, X3-7.S
- new net P108: U2.C5/P108, X3-8.S
- new net P11: U2.D5/P011, X3-18.S
- new net P2: U2.F4/P002, X4-11.S
- new net P23: U2.F0/P023, X4-8.S
- new net P25: U2.A1/P025, X3-17.S
- new net P26: R5.1, U2.E6/P026
- new net P28: U2.H1/P028, X4-3.S
- new net P3: U2.H0/P003, X4-1.S
- new net P31: U2.E5/P031, X4-17.S
- new net P5: U2.G7/P005, X4-19.S
- new net P7: U2.B6/P007, X3-16.S
- new net P8: U2.C7/P008, X3-14.S
- new net SWO: U2.D0/P100, X3-3.S
- new net XTAL1_1: C2.2, U2.F6/P000, X2.2
- new net XTAL2_1: C1.2, U2.F7/P001, X2.1
- net +5V: now also C19.2, C30.2, C31.2, C9.2, U1.VBUS, U7.1; no longer C22.2, C25.2, C28.2, C29.2, U2.1, U6.VBUS
- net +5V_ISO: now also C18.1, U2.B5/VBUS, U6.IN; no longer C21.1, MCU.F5/VBUS, U5.IN
- net 0N: now also C16.2, U5.AN0N; no longer C13.2, U4.AN0N
- net 0P: now also C16.1, U5.AN0P; no longer C13.1, U4.AN0P
- net 1N: now also C17.2, U5.AN1N; no longer C14.2, U4.AN1N
- net 1P: now also C17.1, U5.AN1P; no longer C14.1, U4.AN1P
- net 2N: now also C20.2, U5.AIN2N; no longer C15.2, U4.AIN2N
- net 2P: now also C20.1, U5.AIN2P; no longer C15.1, U4.AIN2P
- net 3N: now also C21.2, U5.AIN3N; no longer C16.2, U4.AIN3N
- net 3P: now also C21.1, U5.AIN3P; no longer C16.1, U4.AIN3P
- net 4N: now also C24.2, U5.AIN4N; no longer C17.2, U4.AIN4N
- net 4P: now also C24.1, U5.AIN4P; no longer C17.1, U4.AIN4P
- net 5N: now also C25.2, U5.AIN5N; no longer C18.2, U4.AIN5N
- net 5P: now also C25.1, U5.AIN5P; no longer C18.1, U4.AIN5P
- net 6N: now also C28.2, U5.AIN6N; no longer C19.2, U4.AIN6N
- net 6P: now also C28.1, U5.AIN6P; no longer C19.1, U4.AIN6P
- net 7N: now also C29.2, U5.AIN7N; no longer C20.2, U4.AIN7N
- net 7P: now also C29.1, U5.AIN7P; no longer C20.1, U4.AIN7P
- net AVDD: now also C5.2, C8.1, U4.OUT, U5.AVDD; no longer C3.2, C6.1, U3.OUT, U4.AVDD
- net BAT: now also C14.2, R7.1, U6.BAT@2, U6.BAT@3; no longer C12.2, R22.1, U5.BAT@2, U5.BAT@3
- net CAP: now also C6.1, U5.CAP; no longer C4.1, U4.CAP
- net CHG: now also R13.2, U2.D6/P027, U6.!CHG; no longer MCU.C7/P008, R29.2, U5.!CHG
- net CLKIN: now also C3.1, U5.XTAL1; no longer C1.1, U4.XTAL1
- net CLKOUT: now also C4.1, U5.XTAL2, X4-20.S; no longer C2.1, HDR2-20.S, U4.XTAL2
- net CS: now also CS.TP, R15.1, U2.E3/P115, U5.CS; no longer MCU.E4/P101, R31.1, U4.CS
- net CUR_DETECT: now also R7.2, R8.1, U2.E7/P004; no longer MCU.E7/P011, R22.2, R23.1
- net D+: now also U1.D+, U2.A4/D+, U7.3; no longer MCU.H5/D+, U2.3, U6.D+
- net D-: now also U1.D-, U2.A5/D-, U7.2; no longer MCU.G5/D-, U2.2, U6.D-
- net DIN: now also DIN.TP, U2.E0/P103, U5.DIN, X4-2.S; no longer HDR2-17.S, MCU.F2/P108, U4.DIN
- net DOUT: now also DOUT.TP, R14.1, U2.F2/P102, U5.DOUT, X4-4.S; no longer HDR2-15.S, MCU.F3/P112, R30.1, U4.DOUT
- net DRDY: now also DRDY.TP, U2.D1/P105, U5.DRDY; no longer MCU.E3/P031, U4.DRDY
- net GND: now also C1.1, C13.1, C14.1, C15.1, C18.2, C19.1, C2.1, C3.2, C30.1, C31.1, C5.1, C7.2, C8.2, LED1.C, LED3.C, R1.1, R14.2, R3.1, R6.1, R6.2, R8.2, U2.G0/VSS, U2.G4/VSS, U2.G5/VSS, U2.G6/VSS, U2.H4/VSS, U2.H5/VSS, U2.H6/VSS, U2.H7/VSS, U4.GND, U5.AGND, U5.AGND-1, U5.DGND, U6.!CE, U6.EN1, U6.TD, U6.VSS, U7.5, U7.MP1, U7.MP2, X4-16.S; no longer C1.2, C2.2, C21.2, C24.1, C25.1, C28.1, C29.1, C3.1, C5.2, C7.1, C8.1, HDR2-16.S, LED1B.C, LED1G.C, LED1R.C, MCU.D3/VSS, MCU.E0/GND, MCU.F0/GND, MCU.F4/GND, MCU.G0/VSS, MCU.H0/GND, MCU.H1/GND, MCU.H7/VSS, R23.2, R27.1, R5.1, U2.5, U2.MP1, U2.MP2, U4.AGND, U4.AGND-1, U4.DGND, U5.!CE, U5.EN1, U5.TD, U5.VSS, U6.GND
- net ID: now also U7.4; no longer U2.4
- net ILM: now also R3.2, U6.ILIM; no longer R4.2, U5.ILIM
- net ISET: now also R4.2, U6.ISET; no longer R5.2, U5.ISET
- net NFC1: now also U2.D2/P009; no longer MCU.F7/P002/NFC1
- net NFC2: now also U2.E2/P010; no longer MCU.C6/NFC2
- net P104: now also U2.B0/P104, X3-11.S; no longer HDR1-2.S, MCU.A1/P104
- net P106: now also U2.E1/P106, X4-10.S; no longer HDR1-14.S, MCU.A7/P106
- net P109: now also U2.C6/P109, X3-20.S; no longer MCU.A0/P109, R26.1
- net P110: now also U2.H2/P110, X4-5.S; no longer HDR2-9.S, MCU.G2/P110
- net P111: now also U2.G2/P111, X4-15.S; no longer HDR2-3.S, MCU.H2/P111
- net P113: now also U2.G3/P113, X4-13.S; no longer HDR2-5.S, MCU.G3/P113
- net P114: now also U2.H3/P114, X4-7.S; no longer HDR2-7.S, MCU.H3/P114
- net P12: now also U2.B7/P012, X3-12.S; no longer HDR1-18.S, MCU.B7/P012/SPI_DCX
- net P14: now also U2.C4/P014, X3-10.S; no longer HDR1-13.S, MCU.B4/P014/QSPI1
- net P15: now also U2.B3/P015, X3-19.S; no longer HDR1-8.S, MCU.A4/015/QSPI2
- net P16: now also R10.1, U2.D3/P016; no longer HDR1-3.S, MCU.B5/P016/QSPI3
- net P17: now also U2.A3/P017, X3-4.S; no longer HDR1-6.S, MCU.A3/P017/QSPI_CLK
- net P19: now also U2.A2/P019, X3-2.S; no longer MCU.C3/P019, R3.1
- net P20: now also R11.1, U2.C2/P020; no longer HDR1-4.S, MCU.A2/P020
- net P21: now also U2.C3/P021, X3-9.S; no longer MCU.C2/P021, R1.1
- net P22: now also U2.B2/P022, X3-15.S; no longer HDR1-9.S, MCU.B2/P022
- net P24: now also U2.F1/P024, X4-12.S; no longer HDR1-7.S, MCU.B1/P024
- net P29: now also U2.E4/P029, X4-9.S; no longer MCU.E1/P029, R2.1
- net P30: now also U2.G1/P030, X4-14.S; no longer HDR2-11.S, MCU.G1/P030
- net PGOOD: now also R12.2, U2.D7/P006, U6.!PGOOD; no longer MCU.D6/P023, R28.2, U5.!PGOOD
- net RESET: now also R2.1, U2.B4/P018/RESET, X3-6.S; no longer HDR2-14.S, MCU.D2/RESET, R24.1
- net SCLK: now also SCLK.TP, U2.F3/P112, U5.SCLK, X4-6.S; no longer HDR2-13.S, MCU.E2/P107, U4.SCLK
- net SWDCLK: now also U2.C1/SWDCLK, X3-5.S; no longer HDR2-10.S, MCU.D1/SWDCLK
- net SWDIO: now also U2.B1/SWDIO, X3-1.S; no longer HDR2-12.S, MCU.D0/SWDIO
- net SYNC/RESET: now also SYNC.TP, U2.D4/P013, U5.SYNC/RESET; no longer MCU.E5/P100, U4.SYNC/RESET
- net TMR: now also U6.TMR; no longer U5.TMR
- net TS: now also R1.2, U6.TS; no longer R27.2, U5.TS
- net VDD: now also C12.2, C15.2, C22.2, R15.2, R9.2, U2.F5/VDD, U3.OUT, U5.DVDD, X4-18.S; no longer C7.2, C9.2, HDR2-18.S, MCU.G4/VDD, R25.2, R30.2, U1.OUT, U4.DVDD
- net VDDH: now also R12.1, R13.1, R2.2, R9.1, U2.A7/VDDH; no longer MCU.F6/VDDH, R24.2, R25.1, R28.1, R29.1
- net VIN: now also C13.2, C7.1, U4.EN, U4.IN; no longer C24.2, C5.1, C8.2, R31.2, U1.EN, U1.IN
- net VSWITCH: now also U6.EN2, U6.OUT@10, U6.OUT@11; no longer U5.EN2, U5.OUT@10, U5.OUT@11
Other:
- note added: "830050789"
- note added: "BC840M"
- note removed: "BC40M"
- note removed: "L1MC-RGB0028000MP0 (OR OTHER)"
- note removed: "Low Pass Filters"
- moved on the sheet: C1, C10, C11, C12, C13, C14, C15, C16, C17, C18, C19, C2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
