File: CAD/BM833/BM833.brd (EAGLE design)
At the start: 33.4 x 25.1 mm, 64 parts, among them J1 SM02B-SRSS-TB(LF)(SN), U1 TPD4S012DRYR, U2 BM833, U3 LP5907MFX-3.3/NOPB, U4 LP5907MFX-3.3/NOPB, U5 ADS131M08IPBS, U6 BQ24072RGTR, U7 DX4R005JJ2R1800, X1 ABM3B-8.000MHZ-B2-T, X2 FC-12M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

Commit message: -
Parts:
- moved NFC2 1.94 mm to (18.2, 63.1)
- moved NFC1 1.92 mm to (19.8, 63.1)
- moved R31 1.74 mm to (27.0, 53.5)
- moved C4 1.16 mm to (28.6, 52.9)
- moved U4 0.19 mm to (25.1, 56.2)
Connections:
- removed net N$24: U2.1, U2.13, U2.15, U2.18, U2.19, U2.2, U2.3, U2.30, U2.4, U2.45, U2.5
- removed net P18: U2.40
- net GND: now also U2.1, U2.13, U2.15, U2.18, U2.19, U2.2, U2.3, U2.30, U2.4, U2.45, U2.5
- net RESET: now also U2.40
Routing:
- net GND: track 149.6 -> 165.2 mm
- net P12: track 14.3 -> 1.78 mm
- net P109: track 12.3 -> 1.78 mm
- net NFC2: track 9.87 -> 0.08 mm, vias 1 -> 0
- net NFC1: track 9.20 -> 0.00 mm, vias 1 -> 0
- net +5V_ISO: track 11.3 -> 20.3 mm, vias 0 -> 2
- net DOUT: track 24.6 -> 16.3 mm
- net P4_AIN2: track 10.8 -> 3.90 mm
- net P31_AIN7: track 27.7 -> 22.2 mm
- net VIN: track 22.0 -> 16.7 mm, vias 3 -> 2
- net P30_AIN6: track 23.9 -> 18.6 mm, vias 2 -> 1
- net P113: track 9.93 -> 4.93 mm
- net RESET: track 5.45 -> 10.4 mm
- net P114: track 8.31 -> 3.38 mm
- net D+: track 24.2 -> 28.8 mm
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Other:
- board text removed: "TOP"
