File: CAD/Sensors/Photodiodes/LightSensorCircuitSMT.sch (EAGLE design)
At the start: 46 parts, among them IC1 CP2102, U1 MCP73831T-3ACI/OT, U2 BT832, U3 LP5907MFX-3.3/NOPB, U4 LP5907MFX-3.3/NOPB, U5 ADS131M08IPBS, U6 BCM857BS, X1 ABM3B-8.000MHZ-B2-T, X2 FC-12M

Commit message: Copy the content of CAD folder from main branch
Parts:
- removed C10: 1.0uF, adafruit:C-USC0402
- removed C11, C14: 0.1uF, adafruit:C-USC0402
- removed C12, C13, C5, C7, C8: 1uF, adafruit:C-USC0402
- removed C15: 10uF, adafruit:C-USC0402
- removed C16, C17: 4.7uF, adafruit:C-USC0402
- removed C6: 220uF, adafruit:C-USC0402
- removed C9: 100uF, adafruit:C-USC0402
- removed D3: BAS40-06, diode:BAS40-06
- removed IC1: CP2102, silabs:CP2102
- removed JP1, JP2, JP3: (no value), adafruit:PINHD-1X8CLEANBIG
- removed R6: 10kΩ, adafruit:R-US_R0402
- removed R7: 24kΩ, adafruit:R-US_R0402
- removed R8: 47kΩ, adafruit:R-US_R0402
- removed S1: CL-SB-12B-01T, CL-SB-12B-01T:CL-SB-12B-01T
- removed SV1: (no value), con-lsta:FE08-2
- removed U$1: DX4R005JJ2R1800, DX4R005JJ2R1800:DX4R005JJ2R1800
- removed U2: BT832, BT832:BT832
- removed U3, U4: LP5907MFX-3.3/NOPB, LP5907MFX-3.3_NOPB:LP5907MFX-3.3/NOPB
- removed U5: ADS131M08IPBS, ADS131M08IPBS:ADS131M08IPBS
- removed U6: BCM857BS, BCM857BS:BCM857BS
- removed X1: ABM3B-8.000MHZ-B2-T, Crystals_Oscillators:ABM3B-8.000MHZ-B2-T
- removed X2: FC-12M, crystal:FC-12M
- added LED3: (no value), adafruit:LEDCHIPLED_1206
- C1, C2: value 12.5pF -> 500pF; device adafruit:C-USC0402 -> adafruit:C-USC0603
- C3, C4: value 10pF -> 0.1uF; device adafruit:C-USC0402 -> adafruit:C-USC0603
- D1: value BAT60J -> BPW_34_S-Z; device diode:BAT60J -> BPW_34_S-Z:BPW_34_S-Z
- D2: value BAS40-06 -> BPW_34_S-Z; device diode:BAS40-06 -> BPW_34_S-Z:BPW_34_S-Z
- J1: device SparkFun-Connectors:JST_2MM_MALE -> SparkFun-Connectors:CONN_05X2NO_SILK
- LED1, LED2: device adafruit:LEDCHIP-LED0603 -> adafruit:LEDCHIPLED_1206
- R1, R2: value 3.3kΩ -> 100k; device adafruit:R-US_R0402 -> adafruit:R-US_R0603
- R3: value 10kΩ -> (none); device adafruit:R-US_R0402 -> adafruit:R-US_R0603
- R4: value 47kΩ -> (none); device adafruit:R-US_R0402 -> adafruit:R-US_R0603
- R5: value 2kΩ -> (none); device adafruit:R-US_R0402 -> adafruit:R-US_R0603
- U1: value MCP73831T-3ACI/OT -> OPA1S2385IDRCR; device MCP73831T-3ACI_OT:MCP73831T-3ACI/OT -> OPA1S2385IDRCR:OPA1S2385IDRCR
Connections:
- removed net +5V: C10.2, C11.2, D2.AA, IC1.REGIN, R7.1, U$1.1, U6.E1
- removed net 0N: SV1.1, U5.AN0N
- removed net 0P: SV1.2, U5.AN0P
- removed net 10K: R3.2, U6.B1, U6.B2, U6.C1
- removed net 11: JP1.4, U2.P13
- removed net 12: JP1.3, U2.P18
- removed net 13: JP1.2, U2.P20
- removed net 14: JP1.1, U2.P21/RESET
- removed net 1N: SV1.3, U5.AN1N
- removed net 1P: SV1.4, U5.AN1P
- removed net 2N: SV1.5, U5.AIN2N
- removed net 2P: SV1.6, U5.AIN2P
- removed net 3N: SV1.7, U5.AIN3N
- removed net 3P: SV1.8, U5.AIN3P
- removed net 4N: SV1.9, U5.AIN4N
- removed net 4P: SV1.10, U5.AIN4P
- removed net 5: JP2.4, U2.P02/AIN0
- removed net 5N: SV1.11, U5.AIN5N
- removed net 5P: SV1.12, U5.AIN5P
- removed net 6: JP2.5, U2.P03/AIN1
- removed net 6N: SV1.13, U5.AIN6N
- removed net 6P: SV1.14, U5.AIN6P
- removed net 7N: SV1.15, U5.AIN7N
- removed net 7P: SV1.16, U5.AIN7P
- removed net AVDD: C5.2, C8.1, U4.OUT, U5.AVDD
- removed net B+: C16.2, J1.+, S1.1, U1.VBAT
- removed net BAT_D3: D3.AA, S1.3
- removed net C1: JP2.1, U2.P24
- removed net C2: JP3.1, U2.P22
- removed net C3: JP3.2, U2.P17
- removed net CAP: C6.1, U5.CAP
- removed net CPRST: IC1.!RST, U2.P08
- removed net CPVDD: C14.2, IC1.VDD
- removed net CS: U2.P05, U5.CS
- removed net D+: IC1.D+, U$1.3
- removed net D-: IC1.D-, U$1.2
- removed net D1: JP3.3, U2.P23
- removed net D2: JP3.4, U2.P19
- removed net D3: JP3.5, U2.P16
- removed net D4: JP3.6, U2.P14
- removed net DIN: U2.P25, U5.DIN
- removed net DOUT: U2.P28, U5.DOUT
- removed net DRDY: U2.P04, U5.DRDY
- removed net GND: C1.1, C10.1, C11.1, C12.1, C13.1, C14.1, C15.1, C16.1, C17.1, C2.1, C3.2, C4.2, C5.1, C6.2, C7.2, C8.2, C9.1, IC1.GND, IC1.GND@EXP, IC1.GND@M, J1.-, JP1.5, JP2.8, LED2.C, R3.1, R4.2, R5.2, R6.1, R8.1, U$1.5, U$1.MP1, U$1.MP2, U1.VSS, U2.GND, U3.GND, U4.GND, U5.AGND, U5.AGND-1, U5.DGND, X1.2, X1.4
- removed net ID: U$1.4
- removed net N$1: LED2.A, R2.1
- removed net N$11: LED1.A, R1.2
- removed net N$14: D2.K2, R4.1, U6.C2
- removed net N$18: LED1.C, U1.STAT
- removed net N$9: R5.1, U1.PROG
- removed net NFC1: JP2.6, U2.P009/NFC1
- removed net NFC2: JP2.7, U2.P010/NFC2
- removed net NVD: C17.2, D1.A, D2.K1, D3.K2, R1.1, R6.2, U1.VDD, U6.E2
- removed net REFIN: C9.2, U5.REFIN
- removed net RXD: IC1.RXD, JP1.7, U2.P12
- removed net SCL: JP2.3, U2.P27/SCL
- removed net SCLK: U2.P29, U5.SCLK
- removed net SDA: JP2.2, U2.P26/SDA
- removed net SWDCLK: JP3.8, U2.SWDCLK
- removed net SWDIO: JP3.7, U2.SWDIO
- removed net SYNC/RESET: U2.P07, U5.SYNC/RESET
- removed net TXD: IC1.TXD, JP1.8, U2.P11
- removed net VBUS: IC1.VBUS, R7.2, R8.2
- removed net VDD: C12.2, C15.2, JP1.6, R2.2, U2.VDD, U3.OUT, U5.DVDD
- removed net VIN: C13.2, C7.1, D1.C, D3.K1, U3.EN, U3.IN, U4.EN, U4.IN
- removed net XTAL1_1: C2.2, U2.P00/XL1, X2.2
- removed net XTAL1_2: C3.1, U5.XTAL1, X1.1
- removed net XTAL2_1: C1.2, U2.P01/XL2, X2.1
- removed net XTAL2_2: C4.1, U5.XTAL2, X1.3
- new net +INA: C1.2, C3.2, D1.C, R1.1, U1.+INA
- new net +INB: C2.2, C4.2, D2.C, R2.1, U1.+INB
- new net AGND: C3.1, C4.1, D1.A, D2.A, J1.3, U1.-INA, U1.-INB, U1.EPAD, U1.V-
- new net INS: J1.2, U1.INS
- new net LED1: J1.10, R5.2
- new net LED2: J1.8, R4.2
- new net LED3: J1.6, R3.2
- new net LEDR1: LED1.A, R5.1
- new net LEDR2: LED2.A, R4.1
- new net LEDR3: LED3.A, R3.1
- new net LED_GND: J1.9, LED1.C, LED2.C, LED3.C
- new net OUTA: C1.1, J1.1, R1.2, U1.OUTA
- new net OUTB: C2.1, J1.7, R2.2, U1.OUTB
- new net SWITCHB: J1.4, U1.SC
- new net V+: J1.5, U1.V+
Other:
- note removed: "830050789"
- note removed: "ADS131M08 Circuitry"
- note removed: "BT832A/AF Circuitry See BlueNor_BT832 Datasheet Page 17 for recommendations"
- note removed: "Battery Charger/Switcher System (See LOLIN32 Schematic)"
- note removed: "LFXTAL061486Reel"
- note removed: "MicroUSB"
- note removed: "Page 20 (oops) https://www.silabs.com/documents/public/data-sheets/CP2102-9.pdf"
- note removed: "TODO: Add 2.2uF caps between + and - inputs (at least for EEG)"
- note removed: "TODO: All necessary passives to add from datasheet Hook up USB-UART (break out UART pins too) Indicators Battery/Power Management Power Switches"
