File: CAD/Sensors/Photodiodes/LightSensorCircuitNoAmp_BTSeriesHookup.brd (EAGLE design)
At the start: 111 x 22.7 mm, 15 parts, among them J1 62202021121, J2 FTSH-108-02-LM-D-ES

Commit message: fix
Parts:
- moved J1 0.08 mm to (-36.2, 18.9), flipped to the bottom, turned to 270 degrees
Connections:
- removed net LED1_P12: J1.9, R5.2, SV1.8
- removed net LED3_P11: J1.3, R3.2, SV1.4
- new net LED1_P11: J1.3, R5.2, SV1.8
- new net LED3_P12: J1.9, R3.2, SV1.4
Routing:
- net LED1_P12: track 63.4 -> 0.00 mm
- net LED1_P11: track 0.00 -> 62.9 mm
- net LED3_P12: track 0.00 -> 61.6 mm
- net LED3_P11: track 61.1 -> 0.00 mm
- net GND: track 172.5 -> 171.2 mm
- net V+: track 97.6 -> 98.8 mm, vias 0 -> 1
- net LED2_P13: track 61.9 -> 62.5 mm
