File: CAD/Sensors/Photodiodes/LightSensorCircuitNoAmp_BTSeriesHookup.brd (EAGLE design)
At the start: 111 x 22.7 mm, 15 parts, among them J1 62202021121, J2 FTSH-108-02-LM-D-ES

Commit message: edit
Parts:
- added C3, C4: (no value), adafruit:C025-025X050
- added D3, D4: BPW34S, BPW34S:DIO_BPW34S
- added H1, H2, H3, H4, H5, H6: MOUNT-HOLE3.6, holes:3,6
- added LED4, LED5, LED6, LED7, LED8, LED9: (no value), adafruit:CHIPLED_1206
- added R10, R11, R12, R13, R6, R7, R8, R9: (no value), adafruit:0204/5
- added SV2, SV3: (no value), con-lsta:FE09
- added SV4: (no value), con-lsta:FE05-1
- SV1: device con-lstb:MA04-2 -> con-lstb:MA05-2
- moved R4 268.5 mm to (283.9, 81.8)
- moved R3 239.8 mm to (253.9, 81.8)
- moved LED3 170.7 mm to (223.7, 87.4)
- moved LED2 170.6 mm to (223.7, 89.5)
- moved LED1 170.5 mm to (223.7, 91.5)
- moved C2 156.4 mm to (193.9, 84.2)
- moved D2 155.3 mm to (193.9, 89.4), turned to 270 degrees
- moved R2 154.4 mm to (193.8, 81.6)
- moved C1 145.0 mm to (164.0, 84.2)
- moved D1 143.9 mm to (164.0, 89.5), turned to 270 degrees
- moved R1 142.9 mm to (164.0, 81.7)
- moved R5 122.2 mm to (127.7, 88.9)
- moved SV1 121.4 mm to (113.1, 92.9)
- moved J2 116.5 mm to (103.4, 87.1)
- moved J1 110.8 mm to (54.0, 83.3)
Connections:
- removed net LED1_P11: J1.3, R5.2, SV1.8
- removed net LED2_P13: J1.5, R4.2, SV1.6
- removed net LED3_P12: J1.9, R3.2, SV1.4
- new net 10: R13.2, SV4.2
- new net 11: SV4.3
- new net 12: SV4.4
- new net 13: SV4.5
- new net 14: SV3.9
- new net 15: SV3.8
- new net 2: R5.2, SV2.3
- new net 26: SV3.7
- new net 27: SV3.6
- new net 28: SV3.5
- new net 29: SV3.4
- new net 3: R6.2, SV2.4
- new net 4: R7.2, SV2.5
- new net 4+: J2.10, SV1.10
- new net 4-: J2.09, SV1.9
- new net 5: R8.2, SV2.6
- new net 5+: J2.12, SV1.8
- new net 5-: J2.11, SV1.7
- new net 5V: SV3.1
- new net 6: R9.2, SV2.7
- new net 6+: J2.14, SV1.6
- new net 6-: J2.13, SV1.5
- new net 7: R10.2, SV2.8
- new net 7+: J2.16, SV1.4
- new net 7-: J2.15, SV1.3
- new net 8: R11.2, SV2.9
- new net 9: R12.2, SV4.1
- new net C: C3.1, D3.A, J2.06, R3.2
- new net D: C4.1, D4.A, J2.08, R4.2
- new net LEDR4: LED4.A, R8.1
- new net LEDR5: LED5.A, R9.1
- new net LEDR6: LED6.A, R10.1
- new net LEDR7: LED7.A, R11.1
- new net LEDR8: LED8.A, R12.1
- new net LEDR9: LED9.A, R13.1
- new net RP_RX: J1.18, SV2.2
- new net RP_TX: J1.17, SV2.1
- net A: now also J2.02; no longer J2.04, SV1.3
- net B: now also J2.04; no longer J2.02, SV1.5
- net GND: now also C3.2, C4.2, LED4.C, LED5.C, LED6.C, LED7.C, LED8.C, LED9.C, R3.1, R4.1, SV3.2; no longer J2.09, J2.11, J2.13, J2.15, SV1.7
- net LEDR2: now also R6.1; no longer R4.1
- net LEDR3: now also R7.1; no longer R3.1
- net V+: now also D3.C, D4.C, SV3.3
Routing:
- net GND: track 171.2 -> 577.3 mm, vias 2 -> 5
- net D: track 0.00 -> 214.1 mm
- net V+: track 98.8 -> 283.5 mm, vias 1 -> 2
- net C: track 0.00 -> 179.2 mm
- net LEDR7: track 0.00 -> 162.3 mm
- net LEDR8: track 0.00 -> 157.6 mm
- net LEDR9: track 0.00 -> 153.7 mm
- net 9: track 0.00 -> 132.3 mm, vias 0 -> 1
- net 8: track 0.00 -> 132.0 mm
- net 10: track 0.00 -> 131.5 mm, vias 0 -> 1
- net 7: track 0.00 -> 130.9 mm
- net 6: track 0.00 -> 110.6 mm
- net 5: track 0.00 -> 108.3 mm
- net 4: track 0.00 -> 106.9 mm
- net 3: track 0.00 -> 104.6 mm
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- removed copper zone on layer 1, net GND
Other:
- board size 111 x 22.7 mm -> 288.6 x 33.2 mm
- board text added: "L3 L2 L1"
- board text added: "L6 L5 L4"
- board text added: "L7"
- board text added: "L8 L9"
- board text added: "RX TX"
- board text added: "TX RX"
- board text removed: "LONG"
- board text removed: "SHORT"
