File: CAD/Sensors/Photodiodes/LightSensorCircuitNoAmp_BTSeriesHookup.sch (EAGLE design)
At the start: 15 parts, among them J1 62202021121, J2 FTSH-108-02-LM-D-ES

Commit message: fix
Connections:
- removed net LED1_P12: J1.9, R5.2, SV1.8
- removed net LED3_P11: J1.3, R3.2, SV1.4
- new net LED1_P11: J1.3, R5.2, SV1.8
- new net LED3_P12: J1.9, R3.2, SV1.4
Changed lines of the file:
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@@
-</segment>
-</net>
-<net name="LED3_P11" class="0">
-<segment>
-<pinref part="J1" gate="G$1" pin="3"/>
-<wire x1="22.098" y1="4.064" x2="23.876" y2="4.064" width="0.1524" layer="91"/>
-<label x="24.638" y="3.81" size="1.778" layer="95"/>
-</segment>
-<segment>
-<pinref part="R3" gate="G$1" pin="2"/>
-<wire x1="245.11" y1="45.72" x2="241.3" y2="45.72" width="0.1524" layer="91"/>
-<label x="236.22" y="43.18" size="1.778" layer="95"/>
-</segment>
-<segment>
-<wire x1="96.012" y1="5.08" x2="93.472" y2="5.08" width="0.1524" layer="91"/>
-<label x="85.852" y="5.08" size="1.778" layer="95"/>
-<pinref part="SV1" gate="G$1" pin="4"/>
 </segment>
 </net>
@@
 </segment>
 </net>
-<net name="LED1_P12" class="0">
+<net name="LED1_P11" class="0">
+<segment>
+<wire x1="96.012" y1="10.16" x2="93.472" y2="10.16" width="0.1524" layer="91"/>
+<label x="85.852" y="10.16" size="1.778" layer="95"/>
+<pinref part="SV1" gate="G$1" pin="8"/>
+</segment>
+<segment>
+<pinref part="J1" gate="G$1" pin="3"/>
+<wire x1="22.098" y1="4.064" x2="23.876" y2="4.064" width="0.1524" layer="91"/>
+<label x="24.638" y="3.81" size="1.778" layer="95"/>
+</segment>
+<segment>
+<pinref part="R5" gate="G$1" pin="2"/>
+<wire x1="245.11" y1="29.21" x2="241.3" y2="29.21" width="0.1524" layer="91"/>
+<label x="236.22" y="26.67" size="1.778" layer="95"/>
+</segment>
+</net>
+<net name="LED3_P12" class="0">
+<segment>
+<wire x1="96.012" y1="5.08" x2="93.472" y2="5.08" width="0.1524" layer="91"/>
+<label x="85.852" y="5.08" size="1.778" layer="95"/>
+<pinref part="SV1" gate="G$1" pin="4"/>
+</segment>
 <segment>
 <pinref part="J1" gate="G$1" pin="9"/>
@@
 </segment>
 <segment>
-<pinref part="R5" gate="G$1" pin="2"/>
-<wire x1="245.11" y1="29.21" x2="241.3" y2="29.21" width="0.1524" layer="91"/>
-<label x="236.22" y="26.67" size="1.778" layer="95"/>
-</segment>
-<segment>
-<wire x1="96.012" y1="10.16" x2="93.472" y2="10.16" width="0.1524" layer="91"/>
-<label x="85.852" y="10.16" size="1.778" layer="95"/>
-<pinref part="SV1" gate="G$1" pin="8"/>
+<pinref part="R3" gate="G$1" pin="2"/>
+<wire x1="245.11" y1="45.72" x2="241.3" y2="45.72" width="0.1524" layer="91"/>
+<label x="236.22" y="43.18" size="1.778" layer="95"/>
 </segment>
 </net>

Commit message: edit
Parts:
- added C3, C4: (no value), adafruit:C-US025-025X050
- added D3, D4: BPW34S, BPW34S:BPW34S
- added H1, H2, H3, H4, H5, H6: MOUNT-HOLE3.6, holes:MOUNT-HOLE3.6
- added LED4, LED5, LED6, LED7, LED8, LED9: (no value), adafruit:LEDCHIPLED_1206
- added R10, R11, R12, R13, R6, R7, R8, R9: (no value), adafruit:R-US_0204/5
- added SV2, SV3: (no value), con-lsta:FE09-1
- added SV4: (no value), con-lsta:FE05-1
- SV1: device con-lstb:MA04-2 -> con-lstb:MA05-2
Connections:
- removed net LED1_P11: J1.3, R5.2, SV1.8
- removed net LED2_P13: J1.5, R4.2, SV1.6
- removed net LED3_P12: J1.9, R3.2, SV1.4
- new net 10: R13.2, SV4.2
- new net 11: SV4.3
- new net 12: SV4.4
- new net 13: SV4.5
- new net 14: SV3.9
- new net 15: SV3.8
- new net 2: R5.2, SV2.3
- new net 26: SV3.7
- new net 27: SV3.6
- new net 28: SV3.5
- new net 29: SV3.4
- new net 3: R6.2, SV2.4
- new net 4: R7.2, SV2.5
- new net 4+: J2.10, SV1.10
- new net 4-: J2.09, SV1.9
- new net 5: R8.2, SV2.6
- new net 5+: J2.12, SV1.8
- new net 5-: J2.11, SV1.7
- new net 5V: SV3.1
- new net 6: R9.2, SV2.7
- new net 6+: J2.14, SV1.6
- new net 6-: J2.13, SV1.5
- new net 7: R10.2, SV2.8
- new net 7+: J2.16, SV1.4
- new net 7-: J2.15, SV1.3
- new net 8: R11.2, SV2.9
- new net 9: R12.2, SV4.1
- new net C: C3.1, D3.A, J2.06, R3.2
- new net D: C4.1, D4.A, J2.08, R4.2
- new net LEDR4: LED4.A, R8.1
- new net LEDR5: LED5.A, R9.1
- new net LEDR6: LED6.A, R10.1
- new net LEDR7: LED7.A, R11.1
- new net LEDR8: LED8.A, R12.1
- new net LEDR9: LED9.A, R13.1
- new net RP_RX: J1.18, SV2.2
- new net RP_TX: J1.17, SV2.1
- net A: now also J2.02; no longer J2.04, SV1.3
- net B: now also J2.04; no longer J2.02, SV1.5
- net GND: now also C3.2, C4.2, LED4.C, LED5.C, LED6.C, LED7.C, LED8.C, LED9.C, R3.1, R4.1, SV3.2; no longer J2.09, J2.11, J2.13, J2.15, SV1.7
- net LEDR2: now also R6.1; no longer R4.1
- net LEDR3: now also R7.1; no longer R3.1
- net V+: now also D3.C, D4.C, SV3.3
Other:
- moved on the sheet: C2, D2, LED1, LED2, LED3, R2, R3, R4, R5
