File: CAD/Sensors/Photodiodes/lightamp.brd (EAGLE design)
At the start: 17 x 13 mm, 6 parts, among them U1 OPA381AIDGKR

Commit message: clarity
Parts:
- C1: value 2.2pF -> 220pF
Changed lines of the file:
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@@
 <?xml version="1.0" encoding="utf-8"?>
 <!DOCTYPE eagle SYSTEM "eagle.dtd">
-<eagle version="9.6.2">
+<eagle version="9.5.1">
 <drawing>
 <settings>
@@
 <attribute name="VALUE" x="17.48310625" y="16.752140625" size="0.762" layer="27" rot="R180"/>
 </element>
-<element name="C1" library="adafruit" library_urn="urn:adsk.eagle:library:420" package="C025-025X050" package3d_urn="urn:adsk.eagle:package:6240323/1" value="2.2pF" x="22.118325" y="12.293603125" smashed="yes" rot="R90">
+<element name="C1" library="adafruit" library_urn="urn:adsk.eagle:library:420" package="C025-025X050" package3d_urn="urn:adsk.eagle:package:6240323/1" value="220pF" x="22.118325" y="12.293603125" smashed="yes" rot="R90">
 <attribute name="NAME" x="23.0606625" y="16.060421875" size="0.9906" layer="25" ratio="10" rot="R180"/>
 <attribute name="VALUE" x="20.83054375" y="8.70456875" size="0.8128" layer="27" ratio="10"/>
