File: CAD/Sensors/Photodiodes/lightampSMT.sch (EAGLE design)
At the start: 6 parts, among them U1 OPA381AIDGKR

Commit message: clarity
Parts:
- C1: value 2.2pF -> 220pF
Other:
- moved on the sheet: C1, C3, D1, R1
