File: CAD/Sensors/Breakouts/FNIRS_Carrier/FNIRS_Carrier_BT_Series.brd (EAGLE design)
At the start: 119.4 x 37.7 mm, 36 parts, among them J1 62202021121, J2 62202021121, J6 FTSH-108-02-LM-D-ES, J7 FTSH-108-02-LM-D-ES, J8 FTSH-108-02-LM-D-ES, X1 TSW-108-07-G-S

Commit message: latest
Parts:
- moved SV1 2.03 mm to (-63.0, 60.4)
- moved C8 0.84 mm to (-68.7, 70.2)
- moved C2 0.84 mm to (-68.7, 53.5)
- moved C4 0.84 mm to (-68.7, 59.0)
- moved C5 0.84 mm to (-68.7, 61.7)
- moved C1 0.84 mm to (-68.7, 50.7)
- moved C3 0.84 mm to (-68.7, 56.2)
- moved C6 0.84 mm to (-68.7, 64.5)
- moved C7 0.84 mm to (-68.7, 67.4)
Routing:
- net GND: track 389.6 -> 383.0 mm
- net AOUT9_0P2: track 30.0 -> 28.5 mm
- net AOUT15_6P2: track 39.5 -> 38.0 mm
- net AOUT14_5P2: track 39.2 -> 37.8 mm
- net AOUT11_2P2: track 37.6 -> 36.1 mm
- net AOUT10_1P2: track 34.2 -> 32.7 mm
- net AOUT16_7P2: track 39.7 -> 38.2 mm
- net AOUT12_3P2: track 41.5 -> 40.0 mm
- net AOUT13_4P2: track 39.4 -> 37.9 mm
